File: STM32H7_Board.kicad_pcb (KiCad board)
At the start: 4 copper layers, 100 x 60 mm, 153 parts, among them IC1 SDRAM_IS42S16320F-7TL, IC3 LED_Driver_TPS61165DBVR, IC5 STM32H7S3I8T6 LQFP 176, J10 SWDB, J11 UART1_HDR, J19 BOOT0_Jumper, J2 I2S_OR_LJ_OUT, J22 USB_C_Receptacle_USB2.0_16P, J27 Molex-52437-2471, J28 Camera_STROBE, J3 UART2_HDR, J32 1.5V_Option_Header, J4 I/O_HDR1, J5 IM2_Jumper, J6 IM1_Jumper, J7 I2C1_Headers, J8 IM0_Jumper, J9 User Button Jumper, Q1 MOSFET_SI2333DDS-T1-BE3, U2 NAND_MT29F2G16ABAEAWP-AITE, U7 USBLC6-2SC6, Y1 Oscillator_ASE-50.000MHZ-L-R-T

Commit message: Update
Parts:
- removed C1: 10u, Capacitor_SMD:C_0805_2012Metric
- removed C11, C13, C68: 4u7, Capacitor_SMD:C_0805_2012Metric
- removed C43: 1u, Capacitor_SMD:C_0805_2012Metric
- removed C62: 22u, Capacitor_SMD:C_0805_2012Metric
- removed J9: User Button Jumper, Connector_PinHeader_2.54mm:PinHeader_1x02_P2.54mm_Vertical
- removed L2: 1u DFE252012P-1R0M=P2, Inductor_SMD:L_1008_2520Metric
- C10, C21, C23, C24, C25, C39, C4, C42, C44, C45, C47, C51, C53, C54, C63, C66, C67, L10, L11, L3, L4, LD1, Q1, R1, R11, R12, R6, Z1: moved to B.Cu
- FB5: footprint Capacitor_SMD:C_0805_2012Metric_Pad1.18x1.45mm_HandSolder -> Capacitor_SMD:C_0805_2012Metric
- J11, J3, J7: footprint Connector_PinHeader_2.54mm:PinHeader_2x03_P2.54mm_Horizontal -> Personal_Project:PinHeader_2x03_P2.54mm_Horizontal_Court
- moved L1 179.4 mm to (175.6, 78.5), turned to 90 degrees
- moved D3 174.6 mm to (181.7, 80.5), turned to 180 degrees
- moved J8 174.3 mm to (181.3, 65.4)
- moved C52 166.8 mm to (177.9, 73.9)
- moved J6 166.8 mm to (185.5, 65.4)
- moved IC3 165.6 mm to (181.2, 77.2)
- moved R10 164.2 mm to (187.4, 77.2), turned to -90 degrees
- moved J5 159.3 mm to (189.9, 65.3)
- moved C40 155.7 mm to (185.1, 77.2), turned to -90 degrees
- moved C30 150.1 mm to (185.7, 81.0), turned to -90 degrees
- moved FFC1 147.3 mm to (191.2, 93.5), turned to 90 degrees
- moved C41 146.1 mm to (182.7, 104.8), turned to -90 degrees
- moved C33 141.5 mm to (185.1, 104.8), turned to -90 degrees
- moved J4 134.6 mm to (125.2, 67.8), turned to 90 degrees
- moved J11 128.5 mm to (118.2, 121.9), turned to -90 degrees
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Connections:
- C22 pad 2: SMPS_GND -> GND
- C65 pad 2: /Interface_Headers/USR_BTN_J -> /Interface_Headers/USR_BTN
- IC5 pad 118: SMPS_GND -> GND
- IC5 pad 143: /Interface_Headers/USB_D2-_DI -> /Interface_Headers/USB_DI_D2-
- IC5 pad 144: /Interface_Headers/USB_D2+_DI -> /Interface_Headers/USB_DI_D2+
- IC5 pad 32: AGND -> GND
- IC5 pad 33: AGND -> GND
- LD1 pad 16: /Power_Management/VREFDDR -> unconnected-(LD1-VREFDDR-Pad16)
- LD1 pad 21: LD6+ -> unconnected-(LD1-LDO6OUT-Pad21)
- LD1 pad 34: BST_5V2+ -> /Power_Management/BST_5V2+
- LD1 pad 35: /Power_Management/VBUSOTG -> unconnected-(LD1-VBUSOTG-Pad35)
- LD1 pad 39: LD4+ -> unconnected-(LD1-LDO4OUT-Pad39)
- U7 pad 1: /Interface_Headers/USB_D2-_DI -> /Interface_Headers/USB_DI_D2+
- U7 pad 3: /Interface_Headers/USB_D2+_DI -> /Interface_Headers/USB_DI_D2-
- U7 pad 4: /Interface_Headers/USB_D2+ -> /Interface_Headers/USB_D2-
- U7 pad 6: /Interface_Headers/USB_D2- -> /Interface_Headers/USB_D2+
- U8 pad 1: /Interface_Headers/USR_BTN_J -> /Interface_Headers/USR_BTN
- U8 pad 2: /Interface_Headers/USR_BTN_J -> /Interface_Headers/USR_BTN
Routing:
- net GND: track 0.00 -> 121.2 mm, vias 0 -> 24
- net PWR_D+: track 0.00 -> 108.8 mm, vias 0 -> 11
- net /Interface_Headers/USB_DI_D2+: track 0.00 -> 42.3 mm
- net /Interface_Headers/USB_DI_D2-: track 0.00 -> 40.9 mm
- net 3V3_BK3+: track 0.00 -> 37.2 mm, vias 0 -> 4
- net 3V3_BK4+: track 0.00 -> 22.3 mm
- net USB_VBUS+: track 0.00 -> 19.5 mm, vias 0 -> 3
- net BK1+: track 0.00 -> 18.4 mm, vias 0 -> 1
- net 1V5_BK2+: track 0.00 -> 15.4 mm, vias 0 -> 1
- net /Interface_Headers/USB_D2+: track 0.00 -> 13.7 mm
- net /Interface_Headers/USB_D2-: track 0.00 -> 13.2 mm
- net /Power_Management/VLX1: track 0.00 -> 13.0 mm
- net Net-(J22-CC1): track 0.00 -> 12.3 mm
- net /Power_Management/VLX4: track 0.00 -> 11.3 mm
- net /Power_Management/VLX2: track 0.00 -> 11.2 mm
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- added copper zone on B.Cu, net /Power_Management/MOSFET_PWR
- added copper zone on B.Cu, net /Power_Management/PWR+
- added copper zone on B.Cu, net /Power_Management/PWR+_PP
- added copper zone on F.Cu, net PWR_D+
- added copper zone on F.Cu, net USB_VBUS+
Other:
- board size 100 x 60 mm -> 100 x 69.9 mm

Commit message: Update
Parts:
- removed C113: 100n, Capacitor_SMD:C_0805_2012Metric
- removed C116: 1u, Capacitor_SMD:C_0805_2012Metric
- removed C119, C63: 4u7, Capacitor_SMD:C_0805_2012Metric
- removed FB5: BEAD(FCM1608KF-601T03)_600Ohm@100MHz1, Capacitor_SMD:C_0805_2012Metric
- moved C15 46.9 mm to (230.2, 114.0), turned to 90 degrees
- moved J19 45.1 mm to (147.3, 119.7), turned to -90 degrees
- moved C16 44.3 mm to (228.2, 114.0), turned to 90 degrees
- moved C50 40.4 mm to (227.2, 133.9), turned to -90 degrees
- moved C18 39.2 mm to (224.2, 114.0), turned to 90 degrees
- moved C20 34.2 mm to (220.2, 114.0), turned to 90 degrees
- moved C55 33.3 mm to (222.2, 133.0), turned to -90 degrees
- moved IC1 29.3 mm to (220.0, 124.1), turned to -90 degrees
- moved C48 22.3 mm to (210.2, 115.0), turned to 90 degrees
- moved C35 12.2 mm to (244.0, 68.6)
- moved J32 12.2 mm to (255.8, 64.7)
- moved C29 12.2 mm to (251.9, 63.9)
- moved J27 12.2 mm to (254.8, 53.6)
- moved C27 12.2 mm to (259.9, 65.3)
- moved FB3 12.2 mm to (259.4, 69.3)
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Connections:
- net Net-(J11-Pin_3) renamed /Interface_Headers/UART1_TX/RX_R
- net Net-(J3-Pin_3) renamed /Interface_Headers/UART2_TX/RX_R
- C104 pad 2: SMPS_GND -> GND
- C106 pad 1: 1V8_LD3+ -> 3V3_BK3+
- C107 pad 1: 1V8_LD3+ -> 3V3_BK3+
- C110 pad 1: 1V8_LD3+ -> 3V3_BK3+
- C111 pad 2: /STM32H7S3I8T6/VDD33USB -> 3V3_BK3+
- C112 pad 1: 1V8_LD3+ -> 3V3_BK3+
- C57 pad 2: SMPS_GND -> GND
- C9 pad 2: SMPS_GND -> GND
- IC5 pad 140: /STM32H7S3I8T6/USB_OTG_HS_VBUS_FR -> 3V3_BK3+
- IC5 pad 141: /STM32H7S3I8T6/VDD33USB -> 3V3_BK3+
- IC5 pad 167: SMPS_GND -> GND
- IC5 pad 60: SMPS_GND -> GND
- IC5 pad 63: 1V8_LD3+ -> 3V3_BK3+
- IC5 pad 69: 1V8_LD3+ -> 3V3_BK3+
- IC5 pad 75: 1V8_LD3+ -> 3V3_BK3+
- IC5 pad 81: 1V8_LD3+ -> 3V3_BK3+
- IC5 pad 98: SMPS_GND -> GND
- LD1 pad 23: LD1+ -> /Power_Management/LD1+
Routing:
- net 3V3_BK3+: track 37.2 -> 178.6 mm, vias 4 -> 24
- net BK1+: track 18.4 -> 91.0 mm, vias 1 -> 5
- net /Interface_Headers/SWCLK: track 2.27 -> 61.5 mm, vias 1 -> 0
- net PWR_D+: track 108.8 -> 57.5 mm, vias 11 -> 8
- net /Interface_Headers/SWDIO: track 2.44 -> 53.0 mm, vias 1 -> 0
- net /Camera_Interface/CAMERA_SDA: track 7.34 -> 34.7 mm
- net /Camera_Interface/CAMERA_SCL: track 9.78 -> 34.1 mm
- net /Power_Management/INTN: track 6.17 -> 26.5 mm, vias 0 -> 1
- net /Interface_Headers/I2S2_SDI/O: track 0.00 -> 18.6 mm, vias 0 -> 2
- net 3V3_BK4+: track 22.3 -> 7.44 mm, vias 0 -> 1
- net GND: track 121.2 -> 135.0 mm, vias 24 -> 39
- net /STM32H7S3I8T6/USB_OTG_HS_VBUS_FR: track 9.49 -> 0.00 mm
- net 1V5_BK2+: track 15.4 -> 6.37 mm
- net /Interface_Headers/I/O_HDR5: track 0.00 -> 9.02 mm
- net /DCMIPP_D9: track 0.00 -> 8.20 mm, vias 0 -> 1
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- added copper zone on B.Cu, net /Power_Management/VLX1
- added copper zone on B.Cu, net /Power_Management/VLX2
- added copper zone on B.Cu, net /Power_Management/VLX3
- added copper zone on B.Cu, net /Power_Management/VLX4
- added copper zone on B.Cu, net 1V5_BK2+
- added copper zone on B.Cu, net 3V3_BK3+
- added copper zone on In2.Cu, net 3V3_BK3+
- added copper zone on B.Cu, net 3V3_BK4+
- added copper zone on B.Cu, net BK1+
- added copper zone on B.Cu, net PWR_D+

Commit message: Update
Routing:
- net GND: vias 39 -> 35
Changed lines of the file:
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@@
 		(tags "capacitor")
 		(property "Reference" "C111"
-			(at -3.8 0.1 360)
+			(at -3.8 0.1 0)
 			(layer "F.SilkS")
 			(effects
@@
 		)
 		(property "Value" "1u"
-			(at 0 1.68 360)
+			(at 0 1.68 0)
 			(layer "F.Fab")
 			(effects
@@
 		)
 		(fp_text user "${REFERENCE}"
-			(at 0 0 360)
+			(at 0 0 0)
 			(layer "F.Fab")
 			(effects
@@
 		(tags "Through hole pin header THT 1x03 2.54mm single row")
 		(property "Reference" "J8"
-			(at 0 -2.33 360)
+			(at 0 -2.33 0)
 			(layer "F.SilkS")
 			(effects
@@
 		)
 		(property "Value" "IM0_Jumper"
-			(at 0 7.41 360)
+			(at 0 7.41 0)
 			(layer "F.Fab")
 			(effects
@@
 		)
 		(fp_text user "${REFERENCE}"
-			(at 0 2.54 360)
+			(at 0 2.54 0)
 			(layer "F.Fab")
 			(effects
@@
 		(tags "Through hole pin header THT 1x03 2.54mm single row")
 		(property "Reference" "J5"
-			(at 0 -2.33 360)
+			(at 0 -2.33 0)
 			(layer "F.SilkS")
 			(effects
@@
 		)
 		(property "Value" "IM2_Jumper"
-			(at 0 7.41 360)
+			(at 0 7.41 0)
 			(layer "F.Fab")
 			(effects
@@
 		(tags "Through hole pin header THT 1x03 2.54mm single row")
 		(property "Reference" "J6"
-			(at 0 -2.33 360)
+			(at 0 -2.33 0)
 			(layer "F.SilkS")
 			(effects
@@
 		)
 		(property "Value" "IM1_Jumper"
-			(at 0 7.41 360)
+			(at 0 7.41 0)
 			(layer "F.Fab")
 			(effects
@@
 	)
 	(via
-		(at 102.1 66.2)
-		(size 0.7)
-		(drill 0.3)
-		(layers "F.Cu" "B.Cu")
-		(free yes)
-		(net 1)
-	)
-	(via
 		(at 116.95 98.725)
 		(size 0.7)
@@
 	)
 	(via
-		(at 102.1 68)
-		(size 0.7)
-		(drill 0.3)
-		(layers "F.Cu" "B.Cu")
-		(free yes)
-		(net 1)
-	)
-	(via
-		(at 102.1 64.3)
-		(size 0.7)
-		(drill 0.3)
-		(layers "F.Cu" "B.Cu")
-		(free yes)
-		(net 1)
-	)
-	(via
 		(at 121.05 107.2)
 		(size 0.7)
@@
 		(size 0.7)
 		(drill 0.3)
-		(layers "F.Cu" "B.Cu")
-		(free yes)
-		(net 1)
-	)
-	(via
-		(at 102.1 62.4)
-		(size 0.7)
-		(drill 0.3)

Commit message: Update
Parts:
- removed C100, C12, C26, C28, C31, C32, C56: 100n, Capacitor_SMD:C_0805_2012Metric
- removed C34, C53, C67: 4u7, Capacitor_SMD:C_0805_2012Metric
- removed C42, C51: 10u, Capacitor_SMD:C_0805_2012Metric
- removed C44, C66, C96: 1u, Capacitor_SMD:C_0805_2012Metric
- removed FB2: 2508051217Y3 0805 (2012 Metric), Inductor_SMD:L_0805_2012Metric
- removed FB4: Part # MI0805K601R-10, Capacitor_SMD:C_0805_2012Metric
- added J1: BTB_10132798-062100LF, Personal_Project:BTB_AMPHENOL_10132798-062100LF, B.Cu at (130.5, 95.1)
- added R5: 4k7, Resistor_SMD:R_0805_2012Metric_1, F.Cu at (240.7, 159.3)
- Y1: value Oscillator_ASE-50.000MHZ-L-R-T -> ECS-3225SMV-240-FP-TR
- moved U1 149.0 mm to (247.4, 89.5)
- moved U8 149.0 mm to (247.6, 93.9)
- moved C17 114.7 mm to (241.5, 163.4)
- moved C19 114.7 mm to (267.5, 162.4)
- moved C46 114.7 mm to (267.5, 164.4)
- moved C49 114.7 mm to (267.5, 166.4)
- moved U2 114.7 mm to (254.2, 164.2)
- moved C30 88.5 mm to (243.5, 14.0)
- moved C41 88.5 mm to (240.5, 37.7)
- moved D3 88.5 mm to (239.5, 13.4)
- moved C40 88.5 mm to (242.9, 10.1)
- moved C52 88.5 mm to (235.7, 6.85)
- moved IC3 88.5 mm to (239.1, 10.1)
- moved R10 88.5 mm to (245.2, 10.1)
- moved C33 88.5 mm to (242.9, 37.7)
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Connections:
- net /STM32H7S3I8T6/PM0 renamed /STM32H7S3I8T6/PM0_UCPD1_CC1
- net /STM32H7S3I8T6/PM1 renamed /STM32H7S3I8T6/PM1_UCPD1_CC2
- net BK1+ renamed 1V2_BK1+
- C101 pad 1: 3V3_BK3+ -> 3V3_BK4+
- C102 pad 1: 3V3_BK3+ -> 3V3_BK4+
- C103 pad 1: 3V3_BK3+ -> 3V3_BK4+
- C105 pad 1: 3V3_BK3+ -> 3V3_BK4+
- C106 pad 1: 3V3_BK3+ -> 3V3_BK4+
- C107 pad 1: 3V3_BK3+ -> 3V3_BK4+
- C108 pad 1: 3V3_BK3+ -> 3V3_BK4+
- C109 pad 2: 3V3_BK3+ -> 3V3_BK4+
- C110 pad 1: 3V3_BK3+ -> 3V3_BK4+
- C111 pad 2: 3V3_BK3+ -> 3V3_BK4+
- C112 pad 1: 3V3_BK3+ -> 3V3_BK4+
- C114 pad 1: 3V3_BK3+ -> 3V3_BK4+
- C115 pad 1: 3V3_BK3+ -> 3V3_BK4+
- C120 pad 1: 3V3_BK3+ -> 3V3_BK4+
- C121 pad 1: 3V3_BK3+ -> 3V3_BK4+
- C122 pad 1: 3V3_BK3+ -> 3V3_BK4+
- C29 pad 1: 2V8_LD5+ -> 2V8_BK3+
- C35 pad 1: 2V8_LD5+ -> 2V8_BK3+
- C47 pad 1: 3V3_BK3+ -> 2V8_BK3+
- C86 pad 1: 3V3_BK3+ -> 3V3_BK4+
- C88 pad 1: 3V3_BK3+ -> 3V3_BK4+
- C90 pad 2: 3V3_BK3+ -> 3V3_BK4+
- C91 pad 1: 3V3_BK3+ -> 3V3_BK4+
- C93 pad 1: 3V3_BK3+ -> 3V3_BK4+
- C95 pad 1: 3V3_BK3+ -> 3V3_BK4+
- C98 pad 1: 3V3_BK3+ -> 3V3_BK4+
- FB1 pad 1: 3V3_BK3+ -> 3V3_BK4+
- FB3 pad 2: 2V8_LD5+ -> 2V8_BK3+
- FPC1 pad 13: /SDMMC1_D1 -> /PP1_XSPIM_P1_IO1
- FPC1 pad 16: /SDMMC1_D2 -> /PP2_XSPIM_P1_IO2
- FPC1 pad 19: /SDMMC1_D3 -> /PP3_XSPIM_P1_IO3
- FPC1 pad 2: /Interface_Headers/SDMMC1_CK -> /Interface_Headers/QSPI_CLK
- FPC1 pad 5: /Interface_Headers/SDMMC1_CMD -> /Interface_Headers/QSPI_CS
- FPC1 pad 8: /SDMMC1_D0 -> /PP0_XSPIM_P1_IO0
- IC5 pad 1: 3V3_BK3+ -> 3V3_BK4+
- IC5 pad 100: 3V3_BK3+ -> 3V3_BK4+
- IC5 pad 105: /SDMMC1_D0 -> /DCMIPP_D2
- IC5 pad 106: /SDMMC1_D1 -> /DCMIPP_D3
- IC5 pad 107: 3V3_BK3+ -> 3V3_BK4+
- IC5 pad 12: 3V3_BK3+ -> 3V3_BK4+
- IC5 pad 120: 3V3_BK3+ -> 3V3_BK4+
- IC5 pad 121: /SDMMC1_D2 -> /Power_Management/INTN
- IC5 pad 122: /SDMMC1_D3 -> /Power_Management/PWRCTRL
- IC5 pad 123: /Interface_Headers/SDMMC1_CK -> /Interface_Headers/I2S2_CK
- IC5 pad 126: /Interface_Headers/SDMMC1_CMD -> /Power_Management/WAKEUP
- IC5 pad 133: 3V3_BK3+ -> 3V3_BK4+
- IC5 pad 138: /STM32H7S3I8T6/PM2 -> /Power_Management/PONKEYN
- IC5 pad 140: 3V3_BK3+ -> 3V3_BK4+
- IC5 pad 141: 3V3_BK3+ -> 3V3_BK4+
- IC5 pad 145: 3V3_BK3+ -> 3V3_BK4+
- IC5 pad 146: /STM32H7S3I8T6/PM8 -> /Interface_Headers/I/O_HDR9
- IC5 pad 147: /STM32H7S3I8T6/PM9 -> /Interface_Headers/I/O_HDR8
- IC5 pad 148: 3V3_BK3+ -> 3V3_BK4+
- IC5 pad 150: /STM32H7S3I8T6/PM11 -> /Interface_Headers/I/O_HDR0
- IC5 pad 151: /Interface_Headers/SPI_MISO -> /STM32H7S3I8T6/PM14
- IC5 pad 152: /Interface_Headers/I/O_HDR8 -> /STM32H7S3I8T6/PM13
- IC5 pad 155: /Power_Management/PONKEYN -> /STM32H7S3I8T6/PD6
- IC5 pad 157: 3V3_BK3+ -> 3V3_BK4+
- IC5 pad 164: /Interface_Headers/I2S2_SDI/O -> /Interface_Headers/I2S1_SDI/O
- IC5 pad 165: /Power_Management/WAKEUP -> /Interface_Headers/I2S2_SDI/O
- IC5 pad 169: 3V3_BK3+ -> 3V3_BK4+
- IC5 pad 170: /DCMIPP_D2 -> /FMC_D9
- IC5 pad 171: /DCMIPP_D3 -> /FMC_D10
- IC5 pad 172: /Interface_Headers/I/O_HDR6 -> /FMC_D11
- IC5 pad 173: /Camera_Interface/CAMERA_SCL -> /Interface_Headers/UART1_TX/RX
- IC5 pad 175: /Interface_Headers/I/O_HDR9 -> /Camera_Interface/CAMERA_SCL
- IC5 pad 19: /Interface_Headers/SPI_CLK -> /Interface_Headers/UART2_TX/RX
- IC5 pad 2: /Power_Management/PWRCTRL -> /STM32H7S3I8T6/PC13
- IC5 pad 21: /Interface_Headers/SPI_MOSI -> /Camera_Interface/STROBE
- IC5 pad 27: 3V3_BK3+ -> 3V3_BK4+
- IC5 pad 41: 3V3_BK3+ -> 3V3_BK4+
- IC5 pad 45: /Interface_Headers/I2S1_SDI/O -> /Memory/FMC_INT
- IC5 pad 48: /Interface_Headers/I2S2_CK -> /LCD_Interface/LCD_TE
- IC5 pad 5: 3V3_BK3+ -> 3V3_BK4+
- IC5 pad 51: 3V3_BK3+ -> 3V3_BK4+
- IC5 pad 53: /Interface_Headers/I/O_HDR7 -> /Interface_Headers/I/O_HDR4
- IC5 pad 58: 3V3_BK3+ -> 3V3_BK4+
- IC5 pad 62: /Interface_Headers/I/O_HDR2 -> /Camera_Interface/PWDN
- IC5 pad 63: 3V3_BK3+ -> 3V3_BK4+
- IC5 pad 65: /LCD_Interface/LCD_TE -> /Interface_Headers/I/O_HDR6
- IC5 pad 66: /Interface_Headers/SPI_CS -> /PP2_XSPIM_P1_IO2
- IC5 pad 67: /Interface_Headers/I/O_HDR0 -> /PP3_XSPIM_P1_IO3
- IC5 pad 69: 3V3_BK3+ -> 3V3_BK4+
- IC5 pad 71: /Interface_Headers/I/O_HDR4 -> /Interface_Headers/QSPI_CLK
- IC5 pad 72: /STM32H7S3I8T6/PP5 -> /Interface_Headers/I/O_HDR7
- IC5 pad 73: /Camera_Interface/STROBE -> /PP0_XSPIM_P1_IO0
- IC5 pad 75: 3V3_BK3+ -> 3V3_BK4+
- IC5 pad 79: /Camera_Interface/PWDN -> /PP1_XSPIM_P1_IO1
- IC5 pad 81: 3V3_BK3+ -> 3V3_BK4+
- IC5 pad 82: /Interface_Headers/I/O_HDR1 -> /Interface_Headers/QSPI_CS
- IC5 pad 87: 3V3_BK3+ -> 3V3_BK4+
- IC5 pad 90: /Memory/FMC_INT -> /STM32H7S3I8T6/PD13
- IC5 pad 91: /FMC_D11 -> /Interface_Headers/I/O_HDR1
- IC5 pad 92: /FMC_D10 -> /Interface_Headers/I/O_HDR2
- IC5 pad 93: /FMC_D9 -> /Interface_Headers/SPI_CS
- IC5 pad 94: /Interface_Headers/UART2_TX/RX -> /Interface_Headers/SPI_CLK
- IC5 pad 95: /Interface_Headers/UART1_TX/RX -> /Interface_Headers/SPI_MISO
- IC5 pad 96: /Power_Management/INTN -> /Interface_Headers/SPI_MOSI
- J19 pad 1: 3V3_BK3+ -> 3V3_BK4+
- J27 pad 11: 2V8_LD5+ -> 2V8_BK3+
- L3 pad 2: 3V3_BK3+ -> 2V8_BK3+
- LD1 pad 13: PWR_D+ -> unconnected-(LD1-LDO3IN-Pad13)
- LD1 pad 14: 1V8_LD3+ -> unconnected-(LD1-LDO3OUT-Pad14)
- LD1 pad 18: 3V3_LD2+ -> unconnected-(LD1-LDO2OUT-Pad18)
- LD1 pad 19: PWR_D+ -> unconnected-(LD1-LDO25IN-Pad19)
- LD1 pad 20: 2V8_LD5+ -> unconnected-(LD1-LDO5OUT-Pad20)
- LD1 pad 22: PWR_D+ -> unconnected-(LD1-LDO16IN-Pad22)
- LD1 pad 23: /Power_Management/LD1+ -> unconnected-(LD1-LDO1OUT-Pad23)
- LD1 pad 31: 3V3_BK3+ -> 2V8_BK3+
- LD1 pad 42: 3V3_BK3+ -> 3V3_BK4+
- OS1 pad 4: 2V8_LD5+ -> 2V8_BK3+
- OS3 pad 4: 3V3_BK3+ -> 3V3_BK4+
- R11 pad 1: 3V3_BK3+ -> 3V3_BK4+
- R12 pad 1: 3V3_BK3+ -> 3V3_BK4+
- R6 pad 1: 3V3_BK3+ -> 3V3_BK4+
- Y1 pad 4: 3V3_BK3+ -> 3V3_BK4+
Routing:
- net 3V3_BK3+: track 178.6 -> 0.00 mm, vias 24 -> 0
- net 3V3_BK4+: track 7.44 -> 146.7 mm, vias 1 -> 16
- net GND: track 135.0 -> 230.2 mm, vias 35 -> 66
- net /FMC_NE1: track 4.31 -> 69.4 mm, vias 1 -> 0
- net /DCMIPP_D6: track 2.25 -> 61.1 mm, vias 1 -> 0
- net 1V2_BK1+: track 91.0 -> 32.6 mm
- net /DCMIPP_D4: track 2.00 -> 58.6 mm, vias 1 -> 0
- net /Memory/FMC_SDCLK: track 3.01 -> 56.1 mm, vias 1 -> 0
- net /Memory/FMC_NBL0: track 3.16 -> 52.6 mm, vias 1 -> 0
- net /Memory/FMC_NCE: track 3.00 -> 50.1 mm, vias 1 -> 0
- net /FMC_D8: track 3.52 -> 49.4 mm, vias 1 -> 0
- net /FMC_A8: track 2.76 -> 44.3 mm, vias 1 -> 0
- net /Memory/FMC_BA1: track 0.00 -> 40.2 mm
- net /FMC_A9: track 4.31 -> 42.7 mm, vias 1 -> 0
- net /Memory/FMC_BA0: track 0.00 -> 38.3 mm
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- added copper zone on B.Cu, net 2V8_BK3+
- removed copper zone on B.Cu, net /Power_Management/VLX2
- removed copper zone on B.Cu, net 1V5_BK2+
- removed copper zone on B.Cu, net 3V3_BK3+
- removed copper zone on In2.Cu, net 3V3_BK3+
Other:
- board size 100 x 69.9 mm -> 100 x 50 mm
- board text added: "USB-C"

Commit message: Update
Parts:
- removed C106, C107, C110, C112, C41: 100n, Capacitor_SMD:C_0805_2012Metric
- removed C30: 1u, Capacitor_SMD:C_0805_2012Metric
- removed C33, C52: 4u7, Capacitor_SMD:C_0805_2012Metric
- removed C40: 220n, Capacitor_SMD:C_0805_2012Metric
- removed D3: MBR0540T1G, Personal_Project:MBR0540T3G_SOD3716X135N
- removed DI1: Diode_PESD5V0U2BT-Q, Package_TO_SOT_SMD:SOT-23
- removed FFC1: FFC_ZF5S-40-02-T-WT, Personal_Project:FFC_ZF5S-40-02-T-WT
- removed FPC1: FPC_0545482072, Personal_Project:FPC_0545482072
- removed FPC2, FPC5, FPC6: FPC_0545481072, Personal_Project:FPC_0545481072
- removed IC3: LED_Driver_TPS61165DBVR, Personal_Project:LEDDriver_TPS61165DBVR_SOT95P280X145-6N
- removed J10: SWDB, Connector_PinHeader_2.54mm:PinHeader_2x04_P2.54mm_Horizontal
- removed J11: UART1_HDR, Personal_Project:PinHeader_2x03_P2.54mm_Horizontal_Court
- removed J19: BOOT0_Jumper, Connector_PinHeader_2.54mm:PinHeader_1x03_P2.54mm_Vertical
- removed J28: Camera_STROBE, Connector_PinHeader_2.54mm:PinHeader_1x02_P2.54mm_Vertical
- removed J32: 1.5V_Option_Header, Connector_PinHeader_2.54mm:PinHeader_1x02_P2.54mm_Vertical
- removed J4: I/O_HDR1, Connector_PinHeader_2.54mm:PinHeader_2x10_P2.54mm_Horizontal
- removed J5: IM2_Jumper, Connector_PinHeader_2.54mm:PinHeader_1x03_P2.54mm_Vertical
- removed J6: IM1_Jumper, Connector_PinHeader_2.54mm:PinHeader_1x03_P2.54mm_Vertical
- removed J7: I2C1_Headers, Personal_Project:PinHeader_2x03_P2.54mm_Horizontal_Court
- removed J8: IM0_Jumper, Connector_PinHeader_2.54mm:PinHeader_1x03_P2.54mm_Vertical
- removed L1: Inductor_VLCF5020T-100M1R1-1, Personal_Project:Inductor_VLCF5020
- removed R10: 1R8, Resistor_SMD:R_0805_2012Metric_1
- removed R13, R2: 10k, Resistor_SMD:R_0805_2012Metric
- removed R22: 1k, Resistor_SMD:R_0805_2012Metric_1
- removed R3, R4: 33R, Resistor_SMD:R_0805_2012Metric
- added C1: 1uF, Capacitor_SMD:C_0805_2012Metric, B.Cu at (104.8, 94.4)
- added CN1: 100n, Resistor_SMD:R_Array_Concave_4x0603, F.Cu at (140.9, 77.3)
- added J9: BTB_10132798-062100LF, Personal_Project:BTB_AMPHENOL_10132798-062100LF, F.Cu at (185.8, 108.5)
- added R8: 2k2, Resistor_SMD:R_0805_2012Metric, F.Cu at (195.4, 63.4)
- added R9: 2k2, Resistor_SMD:R_0805_2012Metric, F.Cu at (195.4, 66.3)
- added RN1: 33R, Resistor_SMD:R_Array_Convex_4x0402, F.Cu at (162.6, 102.1)
- added RN10: 33R, Resistor_SMD:R_Array_Convex_4x0402, F.Cu at (129.5, 101.9)
- added RN11: 33R, Resistor_SMD:R_Array_Convex_4x0402, F.Cu at (194.7, 60.1)
- added RN12: 33R, Resistor_SMD:R_Array_Convex_4x0402, F.Cu at (197.8, 60.1)
- added RN13: 33R, Resistor_SMD:R_Array_Convex_4x0402, F.Cu at (200.8, 60.1)
- added RN14: 33R, Resistor_SMD:R_Array_Convex_4x0402, F.Cu at (142.4, 113.0)
- added RN2: 33R, Resistor_SMD:R_Array_Convex_4x0402, F.Cu at (156.9, 114.0)
- added RN3: 33R, Resistor_SMD:R_Array_Convex_4x0402, F.Cu at (147.1, 111.8)
- added RN4: 33R, Resistor_SMD:R_Array_Convex_4x0402, F.Cu at (152.3, 78.1)
- added RN5: 33R, Resistor_SMD:R_Array_Convex_4x0402, F.Cu at (165.7, 98.0)
- added RN6: 33R, Resistor_SMD:R_Array_Convex_4x0402, F.Cu at (165.8, 90.8)
- added RN7: 33R, Resistor_SMD:R_Array_Convex_4x0402, F.Cu at (161.4, 86.2)
- added RN8: 33R, Resistor_SMD:R_Array_Convex_4x0402, F.Cu at (158.1, 79.7)
- added RN9: 33R, Resistor_SMD:R_Array_Convex_4x0402, F.Cu at (129.5, 104.7)
- added U3: ~, Personal_Project:Button_KMR231GLFS, B.Cu at (101.2, 96.2)
- C15, C16, C17, C18, C19, C20, C46, C48, C49, C50, C55: footprint Capacitor_SMD:C_0805_2012Metric -> Capacitor_SMD:C_0603_1608Metric
- J27: moved to B.Cu
- J3: value UART2_HDR -> SWDB; footprint Personal_Project:PinHeader_2x03_P2.54mm_Horizontal_Court -> Connector_PinHeader_2.54mm:PinHeader_2x04_P2.54mm_Horizontal
- R21: value 22R -> 51R
- moved J27 87.7 mm to (169.1, 72.2), turned to 0 degrees
- moved C17 83.9 mm to (216.0, 83.5), turned to 90 degrees
- moved R5 79.4 mm to (220.1, 82.7), turned to -90 degrees
- moved C49 78.8 mm to (213.0, 109.5), turned to -90 degrees
- moved U2 78.4 mm to (215.2, 96.2), turned to -90 degrees
- moved C46 76.0 mm to (215.0, 109.5), turned to -90 degrees
- moved C19 73.2 mm to (217.0, 109.5), turned to -90 degrees
- moved C35 72.1 mm to (172.3, 61.0)
- moved R7 72.1 mm to (177.2, 56.9)
- moved C27 72.1 mm to (188.2, 57.6)
- moved C29 72.1 mm to (180.3, 56.2)
- moved FB3 72.1 mm to (187.8, 61.6)
- moved OS1 72.1 mm to (176.1, 60.9)
- moved J3 60.7 mm to (107.5, 87.9), turned to 180 degrees
- moved C64 52.9 mm to (241.8, 82.3)
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Connections:
- IC5 pad 10: /FMC_D15 -> /STM32H7S3I8T6/FMC_D15_R
- IC5 pad 102: /DCMIPP_D9 -> /STM32H7S3I8T6/PD15
- IC5 pad 116: /Interface_Headers/I2S2_WS -> /STM32H7S3I8T6/PA15_I2S6_WS
- IC5 pad 121: /Power_Management/INTN -> /STM32H7S3I8T6/PC10_I2S3_CK
- IC5 pad 122: /Power_Management/PWRCTRL -> /STM32H7S3I8T6/PC11_I2S3_SDI
- IC5 pad 123: /Interface_Headers/I2S2_CK -> /STM32H7S3I8T6/PC12_I2S6_CK
- IC5 pad 124: /FMC_A6 -> /STM32H7S3I8T6/FMC_A6_R
- IC5 pad 125: /FMC_A7 -> /STM32H7S3I8T6/FMC_A7_R
- IC5 pad 127: /Memory/FMC_SDNWE -> /STM32H7S3I8T6/FMC_SDNWE_R
- IC5 pad 128: /Memory/FMC_SDNRAS -> /STM32H7S3I8T6/FMC_SDNRAS_R
- IC5 pad 129: /Memory/FMC_SDNCAS -> /STM32H7S3I8T6/FMC_SDNCAS_R
- IC5 pad 130: /Memory/FMC_SDNE0 -> /STM32H7S3I8T6/FMC_SDNE0_R
- IC5 pad 131: /Memory/FMC_SDCKE0 -> /STM32H7S3I8T6/FMC_SDCKE0_R
- IC5 pad 138: /Power_Management/PONKEYN -> /Power_Management/PWRCTRL
- IC5 pad 139: /STM32H7S3I8T6/PM3 -> /Power_Management/INTN
- IC5 pad 146: /Interface_Headers/I/O_HDR9 -> /STM32H7S3I8T6/PM8
- IC5 pad 147: /Interface_Headers/I/O_HDR8 -> /STM32H7S3I8T6/PM9
- IC5 pad 150: /Interface_Headers/I/O_HDR0 -> /STM32H7S3I8T6/PM11
- IC5 pad 154: /Memory/FMC_NCE -> /STM32H7S3I8T6/FMC_NCE_R
- IC5 pad 155: /STM32H7S3I8T6/PD6 -> /STM32H7S3I8T6/PD6_FMC_NE3_R
- IC5 pad 156: /FMC_D8 -> /STM32H7S3I8T6/FMC_D8_R
- IC5 pad 158: /FMC_A8 -> Net-(IC5-PF0)
- IC5 pad 159: /FMC_A9 -> Net-(IC5-PF1)
- IC5 pad 160: /FMC_A10 -> Net-(IC5-PF2)
- IC5 pad 161: /FMC_A11 -> Net-(IC5-PF3)
- IC5 pad 162: /DCMIPP_D8 -> /STM32H7S3I8T6/PF4
- IC5 pad 164: /Interface_Headers/I2S1_SDI/O -> /STM32H7S3I8T6/PB4
- IC5 pad 165: /Interface_Headers/I2S2_SDI/O -> /STM32H7S3I8T6/PB5_I2S6_SDO
- IC5 pad 17: /Memory/FMC_CLE -> Net-(IC5-PF5)
- IC5 pad 170: /FMC_D9 -> Net-(IC5-PE0)
- IC5 pad 171: /FMC_D10 -> Net-(IC5-PE1)
- IC5 pad 172: /FMC_D11 -> Net-(IC5-PE2)
- IC5 pad 173: /Interface_Headers/UART1_TX/RX -> /STM32H7S3I8T6/PB6_UART5_TX
- IC5 pad 175: /Camera_Interface/CAMERA_SCL -> /Power_Management/SCL_STPMIC1
- IC5 pad 176: /Camera_Interface/CAMERA_SDA -> /Power_Management/SDA_STPMIC1
- IC5 pad 18: /Memory/FMC_ALE -> Net-(IC5-PF6)
- IC5 pad 19: /Interface_Headers/UART2_TX/RX -> /STM32H7S3I8T6/PF7_UART7_TX
- IC5 pad 20: /Camera_Interface/DCMIPP_PIXCLK -> Net-(IC5-PF8)
- IC5 pad 21: /Camera_Interface/STROBE -> Net-(IC5-PF9)
- IC5 pad 28: /Memory/FMC_NBL1 -> /STM32H7S3I8T6/FMC_NBL1_R
- IC5 pad 29: /FMC_A0 -> /STM32H7S3I8T6/FMC_A0_R
- IC5 pad 30: /FMC_A1 -> /STM32H7S3I8T6/FMC_A1_R
- IC5 pad 31: /FMC_A2 -> /STM32H7S3I8T6/FMC_A2_R
- IC5 pad 36: /FMC_D7 -> /STM32H7S3I8T6/FMC_D7_R
- IC5 pad 37: /FMC_D6 -> /STM32H7S3I8T6/FMC_D6_R
- IC5 pad 38: /FMC_D5 -> /STM32H7S3I8T6/FMC_D5_R
- IC5 pad 39: /Interface_Headers/I2S1_MCK -> /STM32H7S3I8T6/PA3_I2S6_MCK
- IC5 pad 42: /Interface_Headers/I2S1_WS -> /STM32H7S3I8T6/PA4_I2S3_WS
- IC5 pad 43: /Interface_Headers/I2S1_CK -> /STM32H7S3I8T6/PA5
- IC5 pad 46: /FMC_A3 -> /STM32H7S3I8T6/FMC_A3_R
- IC5 pad 47: /FMC_A5 -> /STM32H7S3I8T6/FMC_A5_R
- IC5 pad 49: /FMC_NOE -> /STM32H7S3I8T6/FMC_NOE_R
- IC5 pad 50: /FMC_NWE -> /STM32H7S3I8T6/FMC_NWE_R
- IC5 pad 53: /Interface_Headers/I/O_HDR4 -> /STM32H7S3I8T6/PF11_ADC1_INP2
- IC5 pad 54: /FMC_A4 -> Net-(IC5-PE7)
- IC5 pad 55: /FMC_A12 -> Net-(IC5-PE8)
- IC5 pad 56: /Memory/FMC_BA0 -> Net-(IC5-PE9)
- IC5 pad 57: /Memory/FMC_BA1 -> Net-(IC5-PE10)
- IC5 pad 65: /Interface_Headers/I/O_HDR6 -> /STM32H7S3I8T6/PP4
- IC5 pad 7: /FMC_D12 -> /STM32H7S3I8T6/FMC_D12_R
- IC5 pad 70: /Interface_Headers/I/O_HDR5 -> /STM32H7S3I8T6/PO5
- IC5 pad 71: /Interface_Headers/QSPI_CLK -> /STM32H7S3I8T6/PO4_XSPIM_P1_CLK
- IC5 pad 72: /Interface_Headers/I/O_HDR7 -> /STM32H7S3I8T6/PP5
- IC5 pad 75: 3V3_BK4+ -> Net-(CN1-C3)
- IC5 pad 77: /Interface_Headers/I/O_HDR3 -> /STM32H7S3I8T6/PO2
- IC5 pad 8: /FMC_D13 -> /STM32H7S3I8T6/FMC_D13_R
- IC5 pad 81: 3V3_BK4+ -> Net-(CN1-C3)
- IC5 pad 82: /Interface_Headers/QSPI_CS -> /STM32H7S3I8T6/PO0_XSPIM_P1_NCS1
- IC5 pad 89: /FMC_NE1 -> /STM32H7S3I8T6/PD12
- IC5 pad 9: /FMC_D14 -> /STM32H7S3I8T6/FMC_D14_R
- IC5 pad 91: /Interface_Headers/I/O_HDR1 -> /Camera_Interface/CAMERA_SDA
- IC5 pad 92: /Interface_Headers/I/O_HDR2 -> /Camera_Interface/CAMERA_SCL
- IC5 pad 93: /Interface_Headers/SPI_CS -> /STM32H7S3I8T6/PB12_SPI2_NSS
- IC5 pad 94: /Interface_Headers/SPI_CLK -> /STM32H7S3I8T6/PB13_SPI2_SCK
- IC5 pad 95: /Interface_Headers/SPI_MISO -> /STM32H7S3I8T6/PB14_SPI2_MISO
- IC5 pad 96: /Interface_Headers/SPI_MOSI -> /STM32H7S3I8T6/PB15_SPI2_MOSI
- J27 pad 1: /Camera_Interface/STROBE_J -> /Camera_Interface/STROBE
- J27 pad 10: /Camera_Interface/DVDD -> 1V5_BK2+
- J27 pad 12: /DCMIPP_D9 -> /DCMIPP_D7
- J27 pad 14: /DCMIPP_D8 -> /DCMIPP_D6
- J27 pad 16: /DCMIPP_D7 -> /DCMIPP_D5
- J27 pad 17: /Camera_Interface/DCMIPP_PIXCLK -> /Camera_Interface/DCMIPP_PIXCLK_R
- J27 pad 18: /DCMIPP_D6 -> /Camera_Interface/DCMIPP_D6_R
- J27 pad 19: /DCMIPP_D2 -> /Camera_Interface/DCMIPP_D2_R
- J27 pad 20: /DCMIPP_D5 -> /Camera_Interface/DCMIPP_D5_R
- J27 pad 21: /DCMIPP_D3 -> /Camera_Interface/DCMIPP_D3_R
- J27 pad 22: /DCMIPP_D4 -> /Camera_Interface/DCMIPP_D4_R
- J27 pad 23: /DCMIPP_D1 -> unconnected-(J27-Pad23)
- J27 pad 24: /DCMIPP_D0 -> unconnected-(J27-Pad24)
- J27 pad 7: /Camera_Interface/DCMIPP_VSYNC -> /Camera_Interface/DCMIPP_VSYNC_R
- J27 pad 8: /Camera_Interface/PWDN -> /Camera_Interface/PWDN_R
- J27 pad 9: /Camera_Interface/DCMIPP_HSYNC -> /Camera_Interface/DCMIPP_HSYNC_R
- J3 pad 2: GND -> /Interface_Headers/SWCLK
- J3 pad 3: /Interface_Headers/UART2_TX/RX_R -> GND
- J3 pad 4: GND -> /Interface_Headers/SWO
- J3 pad 6: GND -> /Camera_Interface/RESETB
- LD1 pad 3: /Camera_Interface/CAMERA_SDA -> /Power_Management/SDA_STPMIC1
- LD1 pad 4: /Camera_Interface/CAMERA_SCL -> /Power_Management/SCL_STPMIC1
- R11 pad 2: /Camera_Interface/CAMERA_SDA -> /Power_Management/SDA_STPMIC1
- R21 pad 1: /STM32H7S3I8T6/PH0-OSC_IN -> Net-(Y1-OUTPUT)
- R21 pad 2: Net-(Y1-OUTPUT) -> /STM32H7S3I8T6/PH0-OSC_IN
- R6 pad 2: /Camera_Interface/CAMERA_SCL -> /Power_Management/SCL_STPMIC1
Routing:
- net 3V3_BK4+: track 146.7 -> 281.1 mm, vias 16 -> 26
- net /FMC_A6: track 39.3 -> 125.7 mm, vias 1 -> 2
- net /FMC_A7: track 40.1 -> 123.3 mm, vias 1 -> 2
- net /Memory/FMC_SDNWE: track 38.6 -> 112.8 mm, vias 1 -> 2
- net /Memory/FMC_SDNRAS: track 37.2 -> 107.6 mm, vias 1 -> 2
- net /Memory/FMC_SDNCAS: track 38.2 -> 103.5 mm, vias 1 -> 2
- net /Memory/FMC_SDNE0: track 39.0 -> 99.5 mm, vias 1 -> 2
- net /FMC_A8: track 44.3 -> 89.9 mm, vias 0 -> 2
- net /FMC_D9: track 29.8 -> 68.6 mm, vias 0 -> 4
- net /FMC_D8: track 49.4 -> 87.3 mm, vias 0 -> 3
- net /FMC_D15: track 11.4 -> 48.8 mm, vias 0 -> 2
- net /FMC_A0: track 15.0 -> 50.5 mm
- net /FMC_D12: track 10.5 -> 44.3 mm
- net /FMC_A5: track 14.8 -> 47.8 mm
- net /FMC_A10: track 41.5 -> 72.3 mm, vias 0 -> 2
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Other:
- board text added: "PONKEYn"
