File: STM32H7_Board.kicad_pcb (KiCad board)
At the start: 4 copper layers, 100 x 50 mm, 111 parts, among them CN1 100n, IC1 SDRAM_IS42S16320F-7TL, IC5 STM32H7S3I8T6 LQFP 176, J1 BTB_10132798-062100LF, J2 I2S_OR_LJ_OUT, J22 USB_C_Receptacle_USB2.0_16P, J27 Molex-52437-2471, J3 SWDB, J9 BTB_10132798-062100LF, Q1 MOSFET_SI2333DDS-T1-BE3, U2 NAND_MT29F2G16ABAEAWP-AITE, U7 USBLC6-2SC6, Y1 ECS-3225SMV-240-FP-TR

Commit message: Update
Parts:
- removed R7: 0R, Resistor_SMD:R_0805_2012Metric_1
- added C2: 1u, Capacitor_SMD:C_0805_2012Metric, B.Cu at (106.2, 99.1)
- added C3: 4u7, Capacitor_SMD:C_0805_2012Metric, B.Cu at (106.2, 96.9)
- added C5: 100n, Capacitor_SMD:C_0603_1608Metric, F.Cu at (157.5, 66.3)
- added C6: 100n, Capacitor_SMD:C_0603_1608Metric, F.Cu at (157.5, 61.8)
- added R2: 33R, Resistor_SMD:R_0603_1608Metric, F.Cu at (127.8, 84.6)
- added R3: 33R, Resistor_SMD:R_0603_1608Metric, B.Cu at (173.6, 79.9)
- added R4: 33R, Resistor_SMD:R_0603_1608Metric, F.Cu at (166.8, 67.8)
- added RN15: 33R, Resistor_SMD:R_Array_Convex_4x0402, F.Cu at (127.5, 92.2)
- RN11, RN12, RN13: moved to B.Cu
- moved RN13 35.2 mm to (171.3, 79.4), turned to -90 degrees
- moved RN12 29.1 mm to (175.9, 79.4), turned to -90 degrees
- moved RN11 25.1 mm to (178.7, 79.4), turned to -90 degrees
- moved C50 5.84 mm to (183.6, 76.7), turned to 0 degrees
- moved U3 5.62 mm to (101.2, 90.6)
- moved J27 5.13 mm to (173.8, 74.1)
- moved C1 3.95 mm to (108.0, 92.2), turned to -90 degrees
- moved C55 3.70 mm to (187.5, 76.7), turned to 0 degrees
- moved C102 1.65 mm to (155.7, 77.1)
- moved C111 0.93 mm to (134.8, 112.3)
- moved RN4 0.91 mm to (152.1, 77.2)
- moved C10 0.53 mm to (111.7, 91.7)
- moved C24 0.53 mm to (110.5, 95.1)
- moved L4 0.53 mm to (113.2, 94.9)
- moved C104 0.17 mm to (147.3, 77.1)
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Connections:
- net /Camera_Interface/DCMIPP_D2_R renamed /Camera_Interface/Y2_R
- net /Camera_Interface/DCMIPP_D3_R renamed /Camera_Interface/Y3_R
- net /Camera_Interface/DCMIPP_D4_R renamed /Camera_Interface/Y4_R
- net /Camera_Interface/DCMIPP_D5_R renamed /Camera_Interface/Y5_R
- net /Camera_Interface/DCMIPP_D6_R renamed /Camera_Interface/Y6_R
- net /Camera_Interface/DCMIPP_HSYNC renamed /Camera_Interface/HSYNC
- net /Camera_Interface/DCMIPP_HSYNC_R renamed /Camera_Interface/HSYNC_R
- net /Camera_Interface/DCMIPP_PIXCLK renamed /Camera_Interface/PCLK
- net /Camera_Interface/DCMIPP_PIXCLK_R renamed /Camera_Interface/PCLK_R
- net /Camera_Interface/DCMIPP_VSYNC renamed /Camera_Interface/VSYNC
- net /Camera_Interface/DCMIPP_VSYNC_R renamed /Camera_Interface/VSYNC_R
- net /Camera_Interface/PWDN renamed /Camera_Interface/CAM_PWDN
- net /Camera_Interface/PWDN_R renamed /Camera_Interface/CAM_PWDN_R
- C64 pad 2: /Camera_Interface/RESETB -> /Interface_Headers/NRST
- CN1 pad 5: Net-(CN1-C3) -> 1V8_LD5+
- CN1 pad 6: Net-(CN1-C3) -> 1V8_LD5+
- CN1 pad 7: 3V3_BK4+ -> 1V8_LD5+
- CN1 pad 8: 3V3_BK4+ -> 1V8_LD5+
- IC5 pad 101: /DCMIPP_D7 -> /STM32H7S3I8T6/DCMIPP_D7_R
- IC5 pad 103: /DCMIPP_D0 -> /STM32H7S3I8T6/DCMIPP_D0_R
- IC5 pad 104: /DCMIPP_D1 -> /STM32H7S3I8T6/DCMIPP_D1_R
- IC5 pad 105: /DCMIPP_D2 -> /STM32H7S3I8T6/DCMIPP_D2_R
- IC5 pad 106: /DCMIPP_D3 -> /STM32H7S3I8T6/DCMIPP_D3_R
- IC5 pad 21: Net-(IC5-PF9) -> /STM32H7S3I8T6/PF9_TIM14_CH1
- IC5 pad 25: /Camera_Interface/RESETB -> /Interface_Headers/NRST
- IC5 pad 43: /STM32H7S3I8T6/PA5 -> /Camera_Interface/RESETB
- IC5 pad 63: 3V3_BK4+ -> 1V8_LD5+
- IC5 pad 69: 3V3_BK4+ -> 1V8_LD5+
- IC5 pad 75: Net-(CN1-C3) -> 1V8_LD5+
- IC5 pad 81: Net-(CN1-C3) -> 1V8_LD5+
- J27 pad 12: /DCMIPP_D7 -> /Camera_Interface/Y9_R
- J27 pad 14: /DCMIPP_D6 -> /Camera_Interface/Y8_R
- J27 pad 16: /DCMIPP_D5 -> /Camera_Interface/Y7_R
- J3 pad 6: /Camera_Interface/RESETB -> /Interface_Headers/NRST
- J9 pad 7: /Camera_Interface/RESETB -> /Interface_Headers/NRST
- LD1 pad 1: /Camera_Interface/RESETB -> /Interface_Headers/NRST
- LD1 pad 19: unconnected-(LD1-LDO25IN-Pad19) -> PWR_D+
- LD1 pad 20: unconnected-(LD1-LDO5OUT-Pad20) -> 1V8_LD5+
- RN12 pad 1: /DCMIPP_D6 -> /Camera_Interface/Y8_R
- RN12 pad 2: /DCMIPP_D5 -> /Camera_Interface/Y7_R
- RN5 pad 4: /Camera_Interface/STROBE -> unconnected-(RN5-R4.1-Pad4)
- RN5 pad 5: Net-(IC5-PF9) -> unconnected-(RN5-R4.2-Pad5)
- U1 pad 1: /Camera_Interface/RESETB -> /Interface_Headers/NRST
- U1 pad 2: /Camera_Interface/RESETB -> /Interface_Headers/NRST
Routing:
- net 1V2_BK1+: track 35.7 -> 139.1 mm
- net 1V8_LD5+: track 0.00 -> 83.6 mm, vias 0 -> 5
- net /DCMIPP_D6: track 54.4 -> 0.00 mm
- net /Camera_Interface/CAMERA_SCL: track 8.73 -> 58.6 mm, vias 0 -> 2
- net /Camera_Interface/CAMERA_SDA: track 7.45 -> 57.3 mm, vias 0 -> 2
- net 3V3_BK4+: track 281.1 -> 320.5 mm, vias 26 -> 25
- net /DCMIPP_D4: track 53.0 -> 27.9 mm, vias 0 -> 1
- net /Interface_Headers/NRST: track 0.00 -> 22.1 mm, vias 0 -> 2
- net /DCMIPP_D5: track 3.60 -> 21.8 mm, vias 1 -> 0
- net /Power_Management/PONKEYN: track 17.4 -> 35.1 mm
- net /Power_Management/INTN: track 5.22 -> 22.2 mm, vias 0 -> 2
- net /DCMIPP_D7: track 28.3 -> 11.3 mm
- net /Camera_Interface/HSYNC: track 4.70 -> 20.9 mm, vias 1 -> 0
- net /DCMIPP_D0: track 32.8 -> 47.9 mm
- net GND: track 226.4 -> 240.6 mm, vias 91 -> 94
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Other:
- board text added: "PONKEY"
- board text removed: "PONKEYn"
