File: STM32H7_Board.kicad_pcb (KiCad board)
At the start: 4 copper layers, 100 x 50 mm, 118 parts, among them CN1 100n, IC1 SDRAM_IS42S16320F-7TL, IC5 STM32H7S3I8T6 LQFP 176, J1 BTB_10132798-062100LF, J2 I2S_OR_LJ_OUT, J22 USB_C_Receptacle_USB2.0_16P, J27 Molex-52437-2471, J3 SWDB, J9 BTB_10132798-062100LF, Q1 MOSFET_SI2333DDS-T1-BE3, U2 NAND_MT29F2G16ABAEAWP-AITE, U7 USBLC6-2SC6, Y1 ECS-3225SMV-240-FP-TR

Commit message: Update
Parts:
- added R10: 33R, Resistor_SMD:R_0603_1608Metric, B.Cu at (145.2, 93.9)
- added R7: 33R, Resistor_SMD:R_0603_1608Metric, B.Cu at (148.4, 104.1)
- added RN16: 33R, Resistor_SMD:R_Array_Convex_4x0402, B.Cu at (145.7, 96.2)
- RN10, RN9: moved to B.Cu
- moved RN10 16.5 mm to (145.8, 99.7), turned to 0 degrees
- moved RN9 16.4 mm to (145.7, 102.3)
Connections:
- IC5 pad 102: /STM32H7S3I8T6/PD15 -> /Interface_Headers/BTB20
- IC5 pad 109: /FMC_D4 -> /STM32H7S3I8T6/FMC_D4_R
- IC5 pad 110: /FMC_D3 -> /STM32H7S3I8T6/FMC_D3_R
- IC5 pad 111: /FMC_D2 -> /STM32H7S3I8T6/FMC_D2_R
- IC5 pad 112: /FMC_D1 -> /STM32H7S3I8T6/FMC_D1_R
- IC5 pad 113: /FMC_D0 -> /STM32H7S3I8T6/FMC_D0_R
- IC5 pad 121: /STM32H7S3I8T6/PC10_I2S3_CK -> /Interface_Headers/BTB6
- IC5 pad 122: /STM32H7S3I8T6/PC11_I2S3_SDI -> /Interface_Headers/BTB4
- IC5 pad 123: /STM32H7S3I8T6/PC12_I2S6_CK -> /Interface_Headers/BTB1
- IC5 pad 126: /Power_Management/WAKEUP -> /STM32H7S3I8T6/PD2
- IC5 pad 138: /Power_Management/PWRCTRL -> /STM32H7S3I8T6/PM2
- IC5 pad 139: /Power_Management/INTN -> /STM32H7S3I8T6/PM3
- IC5 pad 147: /STM32H7S3I8T6/PM9 -> /Power_Management/WAKEUP
- IC5 pad 149: /STM32H7S3I8T6/PM12 -> /Power_Management/PWRCTRL
- IC5 pad 150: /STM32H7S3I8T6/PM11 -> /Power_Management/INTN
- IC5 pad 71: /STM32H7S3I8T6/PO4_XSPIM_P1_CLK -> /Interface_Headers/BTB21
- IC5 pad 82: /STM32H7S3I8T6/PO0_XSPIM_P1_NCS1 -> /Interface_Headers/BTB26
- IC5 pad 93: /STM32H7S3I8T6/PB12_SPI2_NSS -> /Interface_Headers/BTB30
- IC5 pad 94: /STM32H7S3I8T6/PB13_SPI2_SCK -> /Interface_Headers/BTB29
- IC5 pad 95: /STM32H7S3I8T6/PB14_SPI2_MISO -> /Interface_Headers/BTB27
- IC5 pad 96: /STM32H7S3I8T6/PB15_SPI2_MOSI -> /Interface_Headers/BTB28
- J1 pad 1: unconnected-(J1-Pad1) -> /Interface_Headers/BTB1
- J1 pad 2: unconnected-(J1-Pad2) -> /Interface_Headers/BTB2
- J1 pad 20: unconnected-(J1-Pad20) -> /Interface_Headers/BTB20
- J1 pad 21: unconnected-(J1-Pad21) -> /Interface_Headers/BTB21
- J1 pad 22: unconnected-(J1-Pad22) -> /PP3_XSPIM_P1_IO3
- J1 pad 23: unconnected-(J1-Pad23) -> /PP2_XSPIM_P1_IO2
- J1 pad 24: unconnected-(J1-Pad24) -> /PP1_XSPIM_P1_IO1
- J1 pad 25: unconnected-(J1-Pad25) -> /PP0_XSPIM_P1_IO0
- J1 pad 26: unconnected-(J1-Pad26) -> /Interface_Headers/BTB26
- J1 pad 27: unconnected-(J1-Pad27) -> /Interface_Headers/BTB27
- J1 pad 28: unconnected-(J1-Pad28) -> /Interface_Headers/BTB28
- J1 pad 29: unconnected-(J1-Pad29) -> /Interface_Headers/BTB29
- J1 pad 3: unconnected-(J1-Pad3) -> /Interface_Headers/BTB3
- J1 pad 30: unconnected-(J1-Pad30) -> /Interface_Headers/BTB30
- J1 pad 31: unconnected-(J1-Pad31) -> GND
- J1 pad 32: unconnected-(J1-Pad32) -> GND
- J1 pad 33: unconnected-(J1-Pad33) -> GND
- J1 pad 34: unconnected-(J1-Pad34) -> GND
- J1 pad 35: unconnected-(J1-Pad35) -> GND
- J1 pad 36: unconnected-(J1-Pad36) -> GND
- J1 pad 37: unconnected-(J1-Pad37) -> GND
- J1 pad 38: unconnected-(J1-Pad38) -> GND
- J1 pad 39: unconnected-(J1-Pad39) -> GND
- J1 pad 4: unconnected-(J1-Pad4) -> /Interface_Headers/BTB4
- J1 pad 40: unconnected-(J1-Pad40) -> GND
- J1 pad 41: unconnected-(J1-Pad41) -> GND
- J1 pad 42: unconnected-(J1-Pad42) -> GND
- J1 pad 43: unconnected-(J1-Pad43) -> GND
- J1 pad 44: unconnected-(J1-Pad44) -> GND
- J1 pad 45: unconnected-(J1-Pad45) -> GND
- J1 pad 46: unconnected-(J1-Pad46) -> GND
- J1 pad 47: unconnected-(J1-Pad47) -> GND
- J1 pad 48: unconnected-(J1-Pad48) -> GND
- J1 pad 49: unconnected-(J1-Pad49) -> GND
- J1 pad 5: unconnected-(J1-Pad5) -> /Interface_Headers/BTB5
- J1 pad 50: unconnected-(J1-Pad50) -> GND
- J1 pad 51: unconnected-(J1-Pad51) -> GND
- J1 pad 52: unconnected-(J1-Pad52) -> GND
- J1 pad 53: unconnected-(J1-Pad53) -> GND
- J1 pad 54: unconnected-(J1-Pad54) -> GND
- J1 pad 55: unconnected-(J1-Pad55) -> GND
- J1 pad 56: unconnected-(J1-Pad56) -> GND
- J1 pad 57: unconnected-(J1-Pad57) -> GND
- J1 pad 58: unconnected-(J1-Pad58) -> GND
- J1 pad 59: unconnected-(J1-Pad59) -> GND
- J1 pad 6: unconnected-(J1-Pad6) -> /Interface_Headers/BTB6
- J1 pad 60: unconnected-(J1-Pad60) -> GND
- RN14 pad 1: /STM32H7S3I8T6/FMC_D8_R -> unconnected-(RN14-R1.1-Pad1)
- RN14 pad 8: /FMC_D8 -> unconnected-(RN14-R1.2-Pad8)
Routing:
- net /FMC_A6: track 125.7 -> 29.7 mm, vias 2 -> 1
- net /FMC_A7: track 123.3 -> 30.7 mm, vias 2 -> 1
- net /Memory/FMC_SDNWE: track 112.8 -> 21.7 mm, vias 2 -> 1
- net /Memory/FMC_SDNRAS: track 107.6 -> 19.8 mm, vias 2 -> 1
- net /FMC_D8: track 87.3 -> 0.00 mm, vias 3 -> 0
- net /Memory/FMC_SDNCAS: track 103.5 -> 18.9 mm, vias 2 -> 1
- net /Memory/FMC_SDNE0: track 99.5 -> 17.9 mm, vias 2 -> 1
- net /Memory/FMC_SDCKE0: track 41.8 -> 0.00 mm, vias 1 -> 0
- net GND: track 240.6 -> 274.3 mm, vias 94 -> 102
- net /Camera_Interface/RESETB: track 3.15 -> 33.1 mm, vias 1 -> 2
- net /Memory/FMC_NBL1: track 5.89 -> 34.6 mm, vias 0 -> 2
- net /FMC_D0: track 29.1 -> 49.7 mm, vias 2 -> 1
- net /FMC_D1: track 27.8 -> 48.1 mm, vias 1 -> 0
- net /FMC_D7: track 26.6 -> 46.7 mm, vias 0 -> 2
- net /FMC_D4: track 28.9 -> 49.0 mm, vias 1 -> 0
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
Commit message: Update
Parts:
- removed C15, C16, C18, C20, C48, C50, C55: 100n, Capacitor_SMD:C_0603_1608Metric
- removed R10: 33R, Resistor_SMD:R_0603_1608Metric
- removed R5: 4k7, Resistor_SMD:R_0805_2012Metric_1
- removed RN16: 33R, Resistor_SMD:R_Array_Convex_4x0402
- removed U2: NAND_MT29F2G16ABAEAWP-AITE, Personal_Project:NAND_MT29F2G16ABAEAWP-AITE_TSOP-I-48_18.4x12mm_P0.5mmNA
- added C7: 100n, Capacitor_SMD:C_0603_1608Metric, F.Cu at (212.9, 75.9)
- added IC2: SRAM_R1LP5256ESA-5SI#S1_TSOP28, Personal_Project:SRAM_R1LV5256ESA5SIS1_TSOP28, F.Cu at (182.1, 94.2)
- added R13: 4k7, Resistor_SMD:R_0805_2012Metric_1, F.Cu at (208.7, 76.1)
- IC1: value SDRAM_IS42S16320F-7TL -> NAND_MT29F1G08ABAEAWP-IT_E_TR; footprint Personal_Project:SDRAM_IS42S16320F-6TL -> Personal_Project:NAND_MT29F1G08ABAEAWP-IT_E_TR_SOP50P2000X120-48N; moved to B.Cu
- moved IC1 31.2 mm to (204.4, 111.4)
- moved J9 17.4 mm to (195.2, 93.8), turned to -90 degrees
- moved J27 7.84 mm to (181.7, 74.1)
- moved R3 7.47 mm to (181.1, 80.1)
- moved RN11 7.47 mm to (186.1, 79.6)
- moved RN12 7.47 mm to (183.3, 79.6)
- moved RN13 7.47 mm to (178.8, 79.6)
- moved RN9 6.70 mm to (145.8, 95.7), turned to 0 degrees
- moved RN10 0.95 mm to (145.8, 98.7)
- moved RN8 0.93 mm to (158.8, 79.1)
- moved R7 0.89 mm to (149.2, 103.7)
Connections:
- IC1 pad 1: 3V3_BK4+ -> unconnected-(IC1-NC_1-Pad1)
- IC1 pad 10: /FMC_D5 -> unconnected-(IC1-NC_7-Pad10)
- IC1 pad 11: /FMC_D6 -> unconnected-(IC1-NC_8-Pad11)
- IC1 pad 12: GND -> 3V3_BK4+
- IC1 pad 13: /FMC_D7 -> GND
- IC1 pad 14: 3V3_BK4+ -> unconnected-(IC1-NC_9-Pad14)
- IC1 pad 15: /Memory/FMC_NBL0 -> unconnected-(IC1-NC_10-Pad15)
- IC1 pad 16: /Memory/FMC_SDNWE -> /Memory/NAND_CLE
- IC1 pad 17: /Memory/FMC_SDNCAS -> /Memory/NAND_ALE
- IC1 pad 18: /Memory/FMC_SDNRAS -> /FMC_NWE
- IC1 pad 19: /Memory/FMC_SDNE0 -> /Memory/NAND_WP#
- IC1 pad 2: /FMC_D0 -> unconnected-(IC1-NC_2-Pad2)
- IC1 pad 20: /Memory/FMC_BA0 -> unconnected-(IC1-NC_11-Pad20)
- IC1 pad 21: /Memory/FMC_BA1 -> unconnected-(IC1-NC_12-Pad21)
- IC1 pad 22: /FMC_A10 -> unconnected-(IC1-NC_13-Pad22)
- IC1 pad 23: /FMC_A0 -> unconnected-(IC1-NC_14-Pad23)
- IC1 pad 24: /FMC_A1 -> unconnected-(IC1-NC_15-Pad24)
- IC1 pad 25: /FMC_A2 -> GND
- IC1 pad 26: /FMC_A3 -> unconnected-(IC1-NC_16-Pad26)
- IC1 pad 27: 3V3_BK4+ -> unconnected-(IC1-NC_17-Pad27)
- IC1 pad 28: GND -> unconnected-(IC1-NC_18-Pad28)
- IC1 pad 29: /FMC_A4 -> /FMC_D0
- IC1 pad 3: 3V3_BK4+ -> unconnected-(IC1-NC_3-Pad3)
- IC1 pad 30: /FMC_A5 -> /FMC_D1
- IC1 pad 31: /FMC_A6 -> /FMC_D2
- IC1 pad 32: /FMC_A7 -> /FMC_D3
- IC1 pad 33: /FMC_A8 -> unconnected-(IC1-NC_19-Pad33)
- IC1 pad 34: /FMC_A9 -> 3V3_BK4+
- IC1 pad 35: /FMC_A11 -> unconnected-(IC1-NC_20-Pad35)
- IC1 pad 36: /FMC_A12 -> GND
- IC1 pad 37: /Memory/FMC_SDCKE0 -> 3V3_BK4+
- IC1 pad 38: /Memory/FMC_SDCLK -> unconnected-(IC1-DNU_1-Pad38)
- IC1 pad 39: /Memory/FMC_NBL1 -> 3V3_BK4+
- IC1 pad 4: /FMC_D1 -> unconnected-(IC1-NC_4-Pad4)
- IC1 pad 41: GND -> /FMC_D4
- IC1 pad 42: /FMC_D8 -> /FMC_D5
- IC1 pad 43: 3V3_BK4+ -> /FMC_D6
- IC1 pad 44: /FMC_D9 -> /FMC_D7
- IC1 pad 45: /FMC_D10 -> unconnected-(IC1-NC_22-Pad45)
- IC1 pad 46: GND -> unconnected-(IC1-NC_23-Pad46)
- IC1 pad 47: /FMC_D11 -> unconnected-(IC1-DNU_2-Pad47)
- IC1 pad 48: /FMC_D12 -> GND
- IC1 pad 5: /FMC_D2 -> unconnected-(IC1-NC_5-Pad5)
- IC1 pad 6: GND -> unconnected-(IC1-NC_6-Pad6)
- IC1 pad 7: /FMC_D3 -> /Memory/NAND_R/B#
- IC1 pad 8: /FMC_D4 -> /FMC_NOE
- IC1 pad 9: 3V3_BK4+ -> /Memory/NAND_CE#
- IC5 pad 127: /STM32H7S3I8T6/FMC_SDNWE_R -> /Power_Management/INTN
- IC5 pad 128: /STM32H7S3I8T6/FMC_SDNRAS_R -> /STM32H7S3I8T6/PE12
- IC5 pad 129: /STM32H7S3I8T6/FMC_SDNCAS_R -> /Power_Management/PWRCTRL
- IC5 pad 130: /STM32H7S3I8T6/FMC_SDNE0_R -> /STM32H7S3I8T6/PE10
- IC5 pad 131: /STM32H7S3I8T6/FMC_SDCKE0_R -> /Power_Management/WAKEUP
- IC5 pad 147: /Power_Management/WAKEUP -> /STM32H7S3I8T6/PM9
- IC5 pad 149: /Power_Management/PWRCTRL -> /STM32H7S3I8T6/PM12
- IC5 pad 150: /Power_Management/INTN -> /STM32H7S3I8T6/PM11
- IC5 pad 162: /STM32H7S3I8T6/PF4 -> /STM32H7S3I8T6/FMC_A13_R
- IC5 pad 164: /STM32H7S3I8T6/PB4 -> /Camera_Interface/VSYNC
- IC5 pad 174: /Camera_Interface/VSYNC -> /STM32H7S3I8T6/PB7
- IC5 pad 2: /STM32H7S3I8T6/PC13 -> /Memory/NAND_WP#
- IC5 pad 28: /STM32H7S3I8T6/FMC_NBL1_R -> /STM32H7S3I8T6/PC0
- IC5 pad 45: /Memory/FMC_INT -> /Memory/NAND_R/B#
- IC5 pad 57: Net-(IC5-PE10) -> /STM32H7S3I8T6/PE10
- IC5 pad 83: /Memory/FMC_NBL0 -> /STM32H7S3I8T6/PD8
- IC5 pad 84: /Memory/FMC_SDCLK -> /STM32H7S3I8T6/PD9
- IC5 pad 89: /STM32H7S3I8T6/PD12 -> /Memory/SRAM_CS#
- RN10 pad 1: /STM32H7S3I8T6/FMC_SDNWE_R -> /STM32H7S3I8T6/FMC_A13_R
- RN10 pad 4: unconnected-(RN10-R4.1-Pad4) -> /STM32H7S3I8T6/FMC_D0_R
- RN10 pad 5: unconnected-(RN10-R4.2-Pad5) -> /FMC_D0
- RN10 pad 8: /Memory/FMC_SDNWE -> /FMC_A13
- RN14 pad 6: /Memory/FMC_NCE -> /Memory/NAND_CE#
- RN4 pad 3: /Memory/FMC_BA0 -> /FMC_A14
- RN4 pad 4: /Memory/FMC_BA1 -> unconnected-(RN4-R4.1-Pad4)
- RN4 pad 5: Net-(IC5-PE10) -> unconnected-(RN4-R4.2-Pad5)
- RN5 pad 1: /Memory/FMC_CLE -> unconnected-(RN5-R1.1-Pad1)
- RN5 pad 2: /Memory/FMC_ALE -> /Memory/NAND_CLE
- RN5 pad 3: /Camera_Interface/PCLK -> /Memory/NAND_ALE
- RN5 pad 4: unconnected-(RN5-R4.1-Pad4) -> /Camera_Interface/PCLK
- RN5 pad 5: unconnected-(RN5-R4.2-Pad5) -> Net-(IC5-PF8)
- RN5 pad 6: Net-(IC5-PF8) -> Net-(IC5-PF6)
- RN5 pad 7: Net-(IC5-PF6) -> Net-(IC5-PF5)
- RN5 pad 8: Net-(IC5-PF5) -> unconnected-(RN5-R1.2-Pad8)
- RN6 pad 1: /Memory/FMC_NBL1 -> unconnected-(RN6-R1.1-Pad1)
- RN6 pad 8: /STM32H7S3I8T6/FMC_NBL1_R -> unconnected-(RN6-R1.2-Pad8)
- RN9 pad 1: /STM32H7S3I8T6/FMC_SDCKE0_R -> /STM32H7S3I8T6/FMC_D1_R
- RN9 pad 2: /STM32H7S3I8T6/FMC_SDNE0_R -> /STM32H7S3I8T6/FMC_D2_R
- RN9 pad 3: /STM32H7S3I8T6/FMC_SDNCAS_R -> /STM32H7S3I8T6/FMC_D3_R
- RN9 pad 4: /STM32H7S3I8T6/FMC_SDNRAS_R -> /STM32H7S3I8T6/FMC_D4_R
- RN9 pad 5: /Memory/FMC_SDNRAS -> /FMC_D4
- RN9 pad 6: /Memory/FMC_SDNCAS -> /FMC_D3
- RN9 pad 7: /Memory/FMC_SDNE0 -> /FMC_D2
- RN9 pad 8: /Memory/FMC_SDCKE0 -> /FMC_D1
Routing:
- net /Memory/FMC_SDCLK: track 69.9 -> 0.00 mm, vias 2 -> 0
- net /Memory/FMC_BA1: track 63.1 -> 0.00 mm, vias 2 -> 0
- net /Memory/FMC_BA0: track 60.7 -> 0.00 mm, vias 2 -> 0
- net /Memory/NAND_CE#: track 0.00 -> 55.3 mm
- net /Memory/FMC_NCE: track 53.1 -> 0.00 mm
- net /FMC_A14: track 0.00 -> 52.9 mm
- net /FMC_D9: track 68.7 -> 19.7 mm, vias 4 -> 1
- net /Memory/FMC_NBL0: track 48.9 -> 0.00 mm
- net /FMC_A13: track 0.00 -> 46.0 mm, vias 0 -> 1
- net /FMC_A0: track 50.5 -> 5.95 mm
- net /DCMIPP_D2: track 52.3 -> 94.6 mm
- net /FMC_D5: track 47.5 -> 8.54 mm, vias 2 -> 1
- net /FMC_D7: track 46.7 -> 7.90 mm, vias 2 -> 1
- net /FMC_D6: track 46.7 -> 8.04 mm, vias 2 -> 1
- net /FMC_A8: track 87.8 -> 53.1 mm, vias 1 -> 0
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
Commit message: Update
Parts:
- added REF**: TSOP-II-54_22.2x10.16mm_P0.8mm, Package_SO:TSOP-II-54_22.2x10.16mm_P0.8mm, F.Cu at (226.2, 81.0)
- moved IC1 11.1 mm to (213.2, 104.8), turned to 180 degrees
Routing:
- net /FMC_D5: track 8.54 -> 46.4 mm, vias 1 -> 2
- net /FMC_A3: track 11.6 -> 48.0 mm, vias 0 -> 2
- net /FMC_D6: track 8.04 -> 42.7 mm, vias 1 -> 2
- net /FMC_A4: track 22.5 -> 56.8 mm, vias 0 -> 2
- net /FMC_A5: track 14.3 -> 48.2 mm, vias 0 -> 2
- net /FMC_A12: track 26.8 -> 54.1 mm, vias 0 -> 2
- net /FMC_D4: track 57.2 -> 43.1 mm
- net /FMC_D7: track 7.90 -> 20.4 mm, vias 1 -> 2
- net /FMC_NOE: track 0.00 -> 11.7 mm
- net /FMC_NWE: track 0.00 -> 11.5 mm
- net GND: track 270.1 -> 281.2 mm, vias 91 -> 92
- net /FMC_D2: track 56.3 -> 67.0 mm
- net /FMC_D0: track 58.7 -> 69.0 mm
- net /FMC_D1: track 57.9 -> 67.7 mm
- net /FMC_A2: track 9.82 -> 0.00 mm
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
Commit message: Update
Parts:
- removed C7: 100n, Capacitor_SMD:C_0603_1608Metric
- removed IC2: SRAM_R1LP5256ESA-5SI#S1_TSOP28, Personal_Project:SRAM_R1LV5256ESA5SIS1_TSOP28
- removed REF**: TSOP-II-54_22.2x10.16mm_P0.8mm, Package_SO:TSOP-II-54_22.2x10.16mm_P0.8mm
- added C11: 100n, Capacitor_SMD:C_0603_1608Metric, F.Cu at (177.7, 106.9)
- added C12: 100n, Capacitor_SMD:C_0603_1608Metric, F.Cu at (191.2, 92.9)
- added C13: 100n, Capacitor_SMD:C_0603_1608Metric, F.Cu at (174.3, 84.1)
- added C14: 100n, Capacitor_SMD:C_0603_1608Metric, F.Cu at (229.4, 60.0)
- added C15: 100n, Capacitor_SMD:C_0603_1608Metric, F.Cu at (229.4, 62.5)
- added C16: 100n, Capacitor_SMD:C_0603_1608Metric, F.Cu at (229.4, 65.0)
- added C18: 2u2, Capacitor_SMD:C_0603_1608Metric, F.Cu at (229.4, 67.5)
- added C20: 2u2, Capacitor_SMD:C_0603_1608Metric, F.Cu at (229.4, 70.0)
- added C8: 100n, Capacitor_SMD:C_0603_1608Metric, F.Cu at (191.0, 88.1)
- added RN16: 33R, Resistor_SMD:R_Array_Convex_4x0402, B.Cu at (145.8, 101.5)
- added SDRAM1: SDRAM_IS42S83200J-7TLI, Personal_Project:SDRAM_IS42S16320F-6TL, F.Cu at (182.7, 94.5)
- moved J9 0.80 mm to (196.0, 93.9)
- turned R3 to -90 degrees
Connections:
- net Net-(IC5-PE7) renamed /STM32H7S3I8T6/FMC_A4_R
- net Net-(IC5-PE8) renamed /STM32H7S3I8T6/FMC_A12_R
- net Net-(IC5-PE9) renamed /STM32H7S3I8T6/FMC_BA0_R
- net Net-(IC5-PF5) renamed /STM32H7S3I8T6/FMC_CLE_R
- net Net-(IC5-PF6) renamed /STM32H7S3I8T6/FMC_ALE_R
- IC5 pad 127: /Power_Management/INTN -> /STM32H7S3I8T6/PE11_FMC_SDNWE_R
- IC5 pad 128: /STM32H7S3I8T6/PE12 -> /STM32H7S3I8T6/PE12_FMC_SDNRAS_R
- IC5 pad 129: /Power_Management/PWRCTRL -> /STM32H7S3I8T6/PE13_FMC_SDNCAS_R
- IC5 pad 130: /STM32H7S3I8T6/PE10 -> /STM32H7S3I8T6/PE14_FMC_SDNE0_R
- IC5 pad 131: /Power_Management/WAKEUP -> /STM32H7S3I8T6/PE15_FMC_SDCKE0_R
- IC5 pad 162: /STM32H7S3I8T6/FMC_A13_R -> /STM32H7S3I8T6/PD12
- IC5 pad 57: /STM32H7S3I8T6/PE10 -> /STM32H7S3I8T6/FMC_BA1_R
- IC5 pad 83: /STM32H7S3I8T6/PD8 -> /Memory/SDRAM_DQMH
- IC5 pad 84: /STM32H7S3I8T6/PD9 -> /Memory/SDRAM_CLK
- IC5 pad 89: /Memory/SRAM_CS# -> /STM32H7S3I8T6/PD12
- RN10 pad 1: /STM32H7S3I8T6/FMC_A13_R -> /STM32H7S3I8T6/PE11_FMC_SDNWE_R
- RN10 pad 8: /FMC_A13 -> /Memory/SDRAM_~{WE}
- RN4 pad 3: /FMC_A14 -> /Memory/SDRAM_BA0
- RN4 pad 4: unconnected-(RN4-R4.1-Pad4) -> /Memory/SDRAM_BA1
- RN4 pad 5: unconnected-(RN4-R4.2-Pad5) -> /STM32H7S3I8T6/FMC_BA1_R
Routing:
- net /Memory/SDRAM_BA1: track 0.00 -> 61.8 mm, vias 0 -> 2
- net /Memory/SDRAM_BA0: track 0.00 -> 58.5 mm, vias 0 -> 2
- net /FMC_A14: track 53.4 -> 0.00 mm, vias 2 -> 0
- net /FMC_A13: track 46.3 -> 0.00 mm, vias 1 -> 0
- net /DCMIPP_D2: track 94.6 -> 52.3 mm
- net /FMC_NWE: track 11.5 -> 42.5 mm, vias 0 -> 2
- net /FMC_D11: track 34.7 -> 61.9 mm, vias 1 -> 2
- net /LCD_Interface/LCD_TE: track 22.4 -> 42.2 mm, vias 1 -> 2
- net /FMC_D6: track 42.7 -> 26.9 mm
- net /STM32H7S3I8T6/PE11_FMC_SDNWE_R: track 0.00 -> 14.6 mm, vias 0 -> 1
- net /STM32H7S3I8T6/PE15_FMC_SDCKE0_R: track 0.00 -> 14.5 mm, vias 0 -> 1
- net /STM32H7S3I8T6/PE14_FMC_SDNE0_R: track 0.00 -> 14.5 mm, vias 0 -> 1
- net /STM32H7S3I8T6/PE13_FMC_SDNCAS_R: track 0.00 -> 14.3 mm, vias 0 -> 1
- net /STM32H7S3I8T6/PE12_FMC_SDNRAS_R: track 0.00 -> 14.3 mm, vias 0 -> 1
- net /FMC_D2: track 67.0 -> 53.0 mm, vias 1 -> 2
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
Commit message: Update
Parts:
- removed C1: 1uF, Capacitor_SMD:C_0805_2012Metric
- removed C10, C4, C47, C54: 22u, Capacitor_SMD:C_0805_2012Metric
- removed C2: 1u, Capacitor_SMD:C_0805_2012Metric
- removed C21, C3, C45: 4u7, Capacitor_SMD:C_0805_2012Metric
- removed C23, C24, C25, C39: 10u, Capacitor_SMD:C_0805_2012Metric
- removed C29: 100n, Capacitor_SMD:C_0805_2012Metric
- removed C35: 10n, Capacitor_SMD:C_0805_2012Metric
- removed CN1: 100n, Resistor_SMD:R_Array_Concave_4x0603
- removed FB3: BLM31PG601SN1L, Resistor_SMD:R_1206_3216Metric_Pad1.30x1.75mm_HandSolder
- removed J27: Molex-52437-2471, Personal_Project:Molex-52437-2471
- removed L10, L11, L3, L4: 1u DFE252012P-1R0M=P2, Inductor_SMD:L_1008_2520Metric
- removed LD1: LDO_STPMIC1BPQR, Personal_Project:WFQFN-44L_QFN40P500X600X80-45N-D
- removed OS1: Oscillator_ECS-3225Q-33-240-BS-TR, Personal_Project:Oscillator_ECS327MVATX3CNTR
- removed R11, R8, R9: 2k2, Resistor_SMD:R_0805_2012Metric
- removed R12: 10k, Resistor_SMD:R_0805_2012Metric
- removed RN13: 33R, Resistor_SMD:R_Array_Convex_4x0402
- removed U3: ~, Personal_Project:Button_KMR231GLFS
- added C26: 22u, Capacitor_SMD:C_1210_3225Metric, F.Cu at (120.1, 85.0)
- added C7: 22u, Capacitor_SMD:C_1210_3225Metric, F.Cu at (119.0, 113.3)
- added G***: LOGO, Personal_Project:PCB_Logo, F.Cu at (185.6, 112.5)
- added L1: 2u2 NR4020S2R2MT, Personal_Project:L_NR4020S2R2MT, F.Cu at (121.8, 108.0)
- added L5: 2u2 NR4020S2R2MT, Personal_Project:L_NR4020S2R2MT, F.Cu at (121.8, 97.9)
- added R5: 806k, Resistor_SMD:R_0805_2012Metric, F.Cu at (120.5, 93.7)
- added SMPS1: SMPS_TPS62420DRCTG4, Package_SON:VSON-10-1EP_3x3mm_P0.5mm_EP1.65x2.4mm_ThermalVias, F.Cu at (119.5, 103.0)
- C17, C19, C46, C49, R2, RN15: moved to B.Cu
- C27: value 100n -> 33p
- C6: value 100n -> 10u; footprint Capacitor_SMD:C_0603_1608Metric -> Capacitor_SMD:C_0805_2012Metric
- R3, R7: value 33R -> 180k; footprint Resistor_SMD:R_0603_1608Metric -> Resistor_SMD:R_0805_2012Metric; moved to F.Cu
- R4: value 33R -> 180k; footprint Resistor_SMD:R_0603_1608Metric -> Resistor_SMD:R_0805_2012Metric
- R6: value 2k2 -> 33R; footprint Resistor_SMD:R_0805_2012Metric -> Resistor_SMD:R_0603_1608Metric
- moved C27 75.8 mm to (120.4, 91.5)
- moved R3 69.3 mm to (118.1, 109.2), turned to 90 degrees
- moved R4 62.8 mm to (117.2, 106.3), turned to 180 degrees
- moved C15 62.6 mm to (175.2, 93.7), turned to 90 degrees
- moved C14 61.9 mm to (175.2, 89.8), turned to 90 degrees
- moved C16 58.3 mm to (174.2, 83.8), turned to 180 degrees
- moved C6 57.5 mm to (114.0, 99.5)
- moved C46 55.6 mm to (168.0, 79.7), turned to 180 degrees
- moved C49 55.2 mm to (168.6, 76.7), turned to 90 degrees
- moved C17 49.7 mm to (166.8, 76.7)
- moved IC1 42.0 mm to (180.6, 78.4)
- moved R6 40.1 mm to (154.2, 80.9), turned to 0 degrees
- moved C19 39.2 mm to (193.2, 78.3), turned to 0 degrees
- moved RN12 38.9 mm to (145.1, 86.2)
- moved RN11 36.5 mm to (150.1, 85.3), turned to 180 degrees
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Connections:
- net /STM32H7S3I8T6/DCMIPP_D0_R renamed /STM32H7S3I8T6/PC6_PSSI_D0_R
- net /STM32H7S3I8T6/DCMIPP_D1_R renamed /STM32H7S3I8T6/PC7_PSSI_D1_R
- net /STM32H7S3I8T6/DCMIPP_D2_R renamed /STM32H7S3I8T6/PC8_PSSI_D2_R
- net /STM32H7S3I8T6/DCMIPP_D3_R renamed /STM32H7S3I8T6/PC9_PSSI_D3_R
- net /STM32H7S3I8T6/DCMIPP_D7_R renamed /STM32H7S3I8T6/PD14_PSSI_D7_R
- C101 pad 1: 3V3_BK4+ -> SMPS_OUT2_3V3+
- C102 pad 1: 3V3_BK4+ -> SMPS_OUT2_3V3+
- C103 pad 1: 3V3_BK4+ -> SMPS_OUT2_3V3+
- C104 pad 1: 1V2_BK1+ -> SMPS_OUT1_1V2+
- C105 pad 1: 3V3_BK4+ -> SMPS_OUT2_3V3+
- C108 pad 1: 3V3_BK4+ -> SMPS_OUT2_3V3+
- C109 pad 2: 3V3_BK4+ -> SMPS_OUT2_3V3+
- C11 pad 1: 3V3_BK4+ -> SMPS_OUT2_3V3+
- C111 pad 2: 3V3_BK4+ -> SMPS_OUT2_3V3+
- C114 pad 1: 3V3_BK4+ -> SMPS_OUT2_3V3+
- C115 pad 1: 3V3_BK4+ -> SMPS_OUT2_3V3+
- C12 pad 1: 3V3_BK4+ -> SMPS_OUT2_3V3+
- C120 pad 1: 3V3_BK4+ -> SMPS_OUT2_3V3+
- C121 pad 1: 3V3_BK4+ -> SMPS_OUT2_3V3+
- C122 pad 1: 3V3_BK4+ -> SMPS_OUT2_3V3+
- C13 pad 1: 3V3_BK4+ -> SMPS_OUT2_3V3+
- C14 pad 1: 3V3_BK4+ -> SMPS_OUT2_3V3+
- C15 pad 1: 3V3_BK4+ -> SMPS_OUT2_3V3+
- C16 pad 1: 3V3_BK4+ -> SMPS_OUT2_3V3+
- C17 pad 1: 3V3_BK4+ -> SMPS_OUT2_3V3+
- C18 pad 1: 3V3_BK4+ -> SMPS_OUT2_3V3+
- C19 pad 1: 3V3_BK4+ -> SMPS_OUT2_3V3+
- C20 pad 1: 3V3_BK4+ -> SMPS_OUT2_3V3+
- C22 pad 1: 1V2_BK1+ -> SMPS_OUT1_1V2+
- C27 pad 1: /Camera_Interface/AVDD -> /Power_Management/ADJ2
- C27 pad 2: GND -> SMPS_OUT2_3V3+
- C46 pad 1: 3V3_BK4+ -> SMPS_OUT2_3V3+
- C49 pad 1: 3V3_BK4+ -> SMPS_OUT2_3V3+
- C57 pad 1: 1V2_BK1+ -> SMPS_OUT1_1V2+
- C6 pad 1: /Camera_Interface/RESETB -> GND
- C6 pad 2: GND -> PWR_D+
- C8 pad 1: 3V3_BK4+ -> SMPS_OUT2_3V3+
- C86 pad 1: 3V3_BK4+ -> SMPS_OUT2_3V3+
- C88 pad 1: 3V3_BK4+ -> SMPS_OUT2_3V3+
- C9 pad 1: 1V2_BK1+ -> SMPS_OUT1_1V2+
- C90 pad 2: 3V3_BK4+ -> SMPS_OUT2_3V3+
- C91 pad 1: 3V3_BK4+ -> SMPS_OUT2_3V3+
- C93 pad 1: 3V3_BK4+ -> SMPS_OUT2_3V3+
- C95 pad 1: 3V3_BK4+ -> SMPS_OUT2_3V3+
- C98 pad 1: 3V3_BK4+ -> SMPS_OUT2_3V3+
- FB1 pad 1: 3V3_BK4+ -> SMPS_OUT2_3V3+
- IC1 pad 12: 3V3_BK4+ -> SMPS_OUT2_3V3+
- IC1 pad 34: 3V3_BK4+ -> SMPS_OUT2_3V3+
- IC1 pad 37: 3V3_BK4+ -> SMPS_OUT2_3V3+
- IC1 pad 39: 3V3_BK4+ -> SMPS_OUT2_3V3+
- IC5 pad 1: 3V3_BK4+ -> SMPS_OUT2_3V3+
- IC5 pad 100: 3V3_BK4+ -> SMPS_OUT2_3V3+
- IC5 pad 102: /Interface_Headers/BTB20 -> /STM32H7S3I8T6/PD15
- IC5 pad 107: 3V3_BK4+ -> SMPS_OUT2_3V3+
- IC5 pad 116: /STM32H7S3I8T6/PA15_I2S6_WS -> /Interface_Headers/BTB46
- IC5 pad 117: 1V2_BK1+ -> SMPS_OUT1_1V2+
- IC5 pad 119: 1V2_BK1+ -> SMPS_OUT1_1V2+
- IC5 pad 12: 3V3_BK4+ -> SMPS_OUT2_3V3+
- IC5 pad 120: 3V3_BK4+ -> SMPS_OUT2_3V3+
- IC5 pad 121: /Interface_Headers/BTB6 -> /Interface_Headers/BTB50
- IC5 pad 122: /Interface_Headers/BTB4 -> /Interface_Headers/BTB49
- IC5 pad 123: /Interface_Headers/BTB1 -> /Interface_Headers/BTB37
- IC5 pad 133: 3V3_BK4+ -> SMPS_OUT2_3V3+
- IC5 pad 134: /DCMIPP_D5 -> /Interface_Headers/BTB35
- IC5 pad 135: /Camera_Interface/HSYNC -> /Interface_Headers/BTB47
- IC5 pad 140: 3V3_BK4+ -> SMPS_OUT2_3V3+
- IC5 pad 141: 3V3_BK4+ -> SMPS_OUT2_3V3+
- IC5 pad 145: 3V3_BK4+ -> SMPS_OUT2_3V3+
- IC5 pad 148: 3V3_BK4+ -> SMPS_OUT2_3V3+
- IC5 pad 154: /STM32H7S3I8T6/FMC_NCE_R -> /Memory/NAND_CE#
- IC5 pad 157: 3V3_BK4+ -> SMPS_OUT2_3V3+
- IC5 pad 162: /STM32H7S3I8T6/PD12 -> /STM32H7S3I8T6/PF4
- IC5 pad 164: /Camera_Interface/VSYNC -> /Interface_Headers/BTB40
- IC5 pad 165: /STM32H7S3I8T6/PB5_I2S6_SDO -> /Interface_Headers/BTB44
- IC5 pad 166: 1V2_BK1+ -> SMPS_OUT1_1V2+
- IC5 pad 168: 1V2_BK1+ -> SMPS_OUT1_1V2+
- IC5 pad 169: 3V3_BK4+ -> SMPS_OUT2_3V3+
- IC5 pad 173: /STM32H7S3I8T6/PB6_UART5_TX -> /Interface_Headers/BTB38
- IC5 pad 174: /STM32H7S3I8T6/PB7 -> /Interface_Headers/BTB34
- IC5 pad 175: /Power_Management/SCL_STPMIC1 -> /Interface_Headers/BTB31
- IC5 pad 176: /Power_Management/SDA_STPMIC1 -> /Interface_Headers/BTB55
- IC5 pad 19: /STM32H7S3I8T6/PF7_UART7_TX -> /Interface_Headers/BTB53
- IC5 pad 20: Net-(IC5-PF8) -> /Interface_Headers/BTB32
- IC5 pad 22: /Interface_Headers/USR_BTN -> /STM32H7S3I8T6/PF10
- IC5 pad 27: 3V3_BK4+ -> SMPS_OUT2_3V3+
- IC5 pad 39: /STM32H7S3I8T6/PA3_I2S6_MCK -> /STM32H7S3I8T6/PA3_I2S6_MCK_R
- IC5 pad 41: 3V3_BK4+ -> SMPS_OUT2_3V3+
- IC5 pad 42: /STM32H7S3I8T6/PA4_I2S3_WS -> /STM32H7S3I8T6/PA4_I2S3_WS_R
- IC5 pad 43: /Camera_Interface/RESETB -> /STM32H7S3I8T6/PA5_I2S1_C_R
- IC5 pad 45: /Memory/NAND_R/B# -> /STM32H7S3I8T6/PA7_I2S6_SDO_R
- IC5 pad 5: 3V3_BK4+ -> SMPS_OUT2_3V3+
- IC5 pad 51: 3V3_BK4+ -> SMPS_OUT2_3V3+
- IC5 pad 53: /STM32H7S3I8T6/PF11_ADC1_INP2 -> /Interface_Headers/BTB22
- IC5 pad 58: 3V3_BK4+ -> SMPS_OUT2_3V3+
- IC5 pad 59: 1V2_BK1+ -> SMPS_OUT1_1V2+
- IC5 pad 61: 1V2_BK1+ -> SMPS_OUT1_1V2+
- IC5 pad 62: /Camera_Interface/CAM_PWDN -> /STM32H7S3I8T6/PO1
- IC5 pad 63: 1V8_LD5+ -> SMPS_OUT2_3V3+
- IC5 pad 66: /PP2_XSPIM_P1_IO2 -> /STM32H7S3I8T6/PP2
- IC5 pad 67: /PP3_XSPIM_P1_IO3 -> /STM32H7S3I8T6/PP3
- IC5 pad 69: 1V8_LD5+ -> SMPS_OUT2_3V3+
- IC5 pad 71: /Interface_Headers/BTB21 -> /Interface_Headers/BTB29
- IC5 pad 72: /STM32H7S3I8T6/PP5 -> /Interface_Headers/BTB28
- IC5 pad 73: /PP0_XSPIM_P1_IO0 -> /STM32H7S3I8T6/PP0
- IC5 pad 75: 1V8_LD5+ -> SMPS_OUT2_3V3+
- IC5 pad 76: /STM32H7S3I8T6/PP6 -> /Interface_Headers/BTB26
- IC5 pad 77: /STM32H7S3I8T6/PO2 -> /Interface_Headers/BTB25
- IC5 pad 78: /STM32H7S3I8T6/PP7 -> /Interface_Headers/BTB23
- IC5 pad 79: /PP1_XSPIM_P1_IO1 -> /STM32H7S3I8T6/PP1
- IC5 pad 81: 1V8_LD5+ -> SMPS_OUT2_3V3+
- IC5 pad 82: /Interface_Headers/BTB26 -> /STM32H7S3I8T6/PO0
- IC5 pad 83: /Memory/SDRAM_DQMH -> /STM32H7S3I8T6/PD8_FMC_NBL0_R
- IC5 pad 84: /Memory/SDRAM_CLK -> /STM32H7S3I8T6/PD9_FMC_SDCLK_R
- IC5 pad 85: /DCMIPP_D4 -> /Interface_Headers/BTB7
- IC5 pad 86: /DCMIPP_D6 -> /Interface_Headers/BTB8
- IC5 pad 87: 3V3_BK4+ -> SMPS_OUT2_3V3+
- IC5 pad 89: /STM32H7S3I8T6/PD12 -> /Interface_Headers/BTB43
- IC5 pad 90: /STM32H7S3I8T6/PD13 -> /Memory/NAND_R/B#
- IC5 pad 91: /Camera_Interface/CAMERA_SDA -> /Interface_Headers/BTB41
- IC5 pad 92: /Camera_Interface/CAMERA_SCL -> /STM32H7S3I8T6/PB11
- IC5 pad 93: /Interface_Headers/BTB30 -> /Interface_Headers/BTB1
- IC5 pad 94: /Interface_Headers/BTB29 -> /Interface_Headers/BTB2
- IC5 pad 95: /Interface_Headers/BTB27 -> /Interface_Headers/BTB4
- IC5 pad 96: /Interface_Headers/BTB28 -> /Interface_Headers/BTB5
- IC5 pad 97: 1V2_BK1+ -> SMPS_OUT1_1V2+
- IC5 pad 99: 1V2_BK1+ -> SMPS_OUT1_1V2+
- J1 pad 10: unconnected-(J1-Pad10) -> /Interface_Headers/BTB10
- J1 pad 11: unconnected-(J1-Pad11) -> /Interface_Headers/BTB11
- J1 pad 12: unconnected-(J1-Pad12) -> GND
- J1 pad 13: unconnected-(J1-Pad13) -> /Interface_Headers/BTB13
- J1 pad 14: unconnected-(J1-Pad14) -> /Interface_Headers/BTB14
- J1 pad 15: unconnected-(J1-Pad15) -> GND
- J1 pad 16: unconnected-(J1-Pad16) -> /Interface_Headers/BTB16
- J1 pad 17: unconnected-(J1-Pad17) -> /Interface_Headers/BTB17
- J1 pad 18: unconnected-(J1-Pad18) -> GND
- J1 pad 19: unconnected-(J1-Pad19) -> /Interface_Headers/BTB19
- J1 pad 21: /Interface_Headers/BTB21 -> GND
- J1 pad 22: /PP3_XSPIM_P1_IO3 -> /Interface_Headers/BTB22
- J1 pad 23: /PP2_XSPIM_P1_IO2 -> /Interface_Headers/BTB23
- J1 pad 24: /PP1_XSPIM_P1_IO1 -> GND
- J1 pad 25: /PP0_XSPIM_P1_IO0 -> /Interface_Headers/BTB25
- J1 pad 27: /Interface_Headers/BTB27 -> GND
- J1 pad 3: /Interface_Headers/BTB3 -> GND
- J1 pad 31: GND -> /Interface_Headers/BTB60
- J1 pad 32: GND -> /Interface_Headers/BTB59
- J1 pad 33: GND -> /Interface_Headers/BTB58
- J1 pad 35: GND -> /Interface_Headers/BTB56
- J1 pad 36: GND -> /Interface_Headers/BTB55
- J1 pad 38: GND -> /Interface_Headers/BTB53
- J1 pad 39: GND -> /Interface_Headers/BTB52
- J1 pad 41: GND -> /Interface_Headers/BTB50
- J1 pad 42: GND -> /Interface_Headers/BTB49
- J1 pad 44: GND -> /Interface_Headers/BTB47
- J1 pad 45: GND -> /Interface_Headers/BTB46
- J1 pad 47: GND -> /Interface_Headers/BTB44
- J1 pad 48: GND -> /Interface_Headers/BTB43
- J1 pad 50: GND -> /Interface_Headers/BTB41
- J1 pad 51: GND -> /Interface_Headers/BTB40
- J1 pad 53: GND -> /Interface_Headers/BTB38
- J1 pad 54: GND -> /Interface_Headers/BTB37
- J1 pad 56: GND -> /Interface_Headers/BTB35
- J1 pad 57: GND -> /Interface_Headers/BTB34
- J1 pad 59: GND -> /Interface_Headers/BTB32
- J1 pad 6: /Interface_Headers/BTB6 -> GND
- J1 pad 60: GND -> /Interface_Headers/BTB31
- J1 pad 7: unconnected-(J1-Pad7) -> /Interface_Headers/BTB7
- J1 pad 8: unconnected-(J1-Pad8) -> /Interface_Headers/BTB8
- J1 pad 9: unconnected-(J1-Pad9) -> GND
- J3 pad 1: GND -> USB_VBUS+
- OS3 pad 4: 3V3_BK4+ -> SMPS_OUT2_3V3+
- R13 pad 1: 3V3_BK4+ -> SMPS_OUT2_3V3+
- R2 pad 2: /DCMIPP_D7 -> /Interface_Headers/BTB10
- R3 pad 1: /Camera_Interface/Y9_R -> SMPS_OUT1_1V2+
- R3 pad 2: /DCMIPP_D7 -> /Power_Management/DEF_1
- R4 pad 1: /Camera_Interface/XCLK -> /Power_Management/DEF_1
- R4 pad 2: Net-(OS1-OUTPUT) -> GND
- R6 pad 1: 3V3_BK4+ -> /Interface_Headers/BTB30
- R6 pad 2: /Power_Management/SCL_STPMIC1 -> /STM32H7S3I8T6/PA7_I2S6_SDO_R
- R7 pad 1: /STM32H7S3I8T6/FMC_D8_R -> /Power_Management/ADJ2
- R7 pad 2: /FMC_D8 -> GND
- RN11 pad 1: /Camera_Interface/Y2_R -> unconnected-(RN11-R1.1-Pad1)
- RN11 pad 2: /Camera_Interface/Y5_R -> /Memory/SDRAM_DQMH
- RN11 pad 3: /Camera_Interface/Y3_R -> /Memory/SDRAM_CLK
- RN11 pad 4: /Camera_Interface/Y4_R -> unconnected-(RN11-R4.1-Pad4)
- RN11 pad 5: /DCMIPP_D2 -> unconnected-(RN11-R4.2-Pad5)
- RN11 pad 6: /DCMIPP_D1 -> /STM32H7S3I8T6/PD9_FMC_SDCLK_R
- RN11 pad 7: /DCMIPP_D3 -> /STM32H7S3I8T6/PD8_FMC_NBL0_R
- RN11 pad 8: /DCMIPP_D0 -> unconnected-(RN11-R1.2-Pad8)
- RN12 pad 1: /Camera_Interface/Y8_R -> /Interface_Headers/BTB17
- RN12 pad 2: /Camera_Interface/Y7_R -> /Interface_Headers/BTB19
- RN12 pad 3: /Camera_Interface/PCLK_R -> /Interface_Headers/BTB20
- RN12 pad 4: /Camera_Interface/Y6_R -> unconnected-(RN12-R4.1-Pad4)
- RN12 pad 5: /DCMIPP_D4 -> unconnected-(RN12-R4.2-Pad5)
- RN12 pad 6: /Camera_Interface/PCLK -> /STM32H7S3I8T6/PA5_I2S1_C_R
- RN12 pad 7: /DCMIPP_D5 -> /STM32H7S3I8T6/PA4_I2S3_WS_R
- RN12 pad 8: /DCMIPP_D6 -> /STM32H7S3I8T6/PA3_I2S6_MCK_R
- RN14 pad 1: unconnected-(RN14-R1.1-Pad1) -> /STM32H7S3I8T6/FMC_D8_R
- RN14 pad 3: /STM32H7S3I8T6/FMC_NCE_R -> unconnected-(RN14-R3.1-Pad3)
- RN14 pad 6: /Memory/NAND_CE# -> unconnected-(RN14-R3.2-Pad6)
- RN14 pad 8: unconnected-(RN14-R1.2-Pad8) -> /FMC_D8
- RN15 pad 5: /DCMIPP_D0 -> /Interface_Headers/BTB11
- RN15 pad 6: /DCMIPP_D1 -> /Interface_Headers/BTB13
- RN15 pad 7: /DCMIPP_D2 -> /Interface_Headers/BTB14
- RN15 pad 8: /DCMIPP_D3 -> /Interface_Headers/BTB16
- RN5 pad 4: /Camera_Interface/PCLK -> unconnected-(RN5-R4.1-Pad4)
- RN5 pad 5: Net-(IC5-PF8) -> unconnected-(RN5-R4.2-Pad5)
- SDRAM1 pad 1: 3V3_BK4+ -> SMPS_OUT2_3V3+
- SDRAM1 pad 14: 3V3_BK4+ -> SMPS_OUT2_3V3+
- SDRAM1 pad 27: 3V3_BK4+ -> SMPS_OUT2_3V3+
- SDRAM1 pad 3: 3V3_BK4+ -> SMPS_OUT2_3V3+
- SDRAM1 pad 43: 3V3_BK4+ -> SMPS_OUT2_3V3+
- SDRAM1 pad 49: 3V3_BK4+ -> SMPS_OUT2_3V3+
- SDRAM1 pad 9: 3V3_BK4+ -> SMPS_OUT2_3V3+
- Y1 pad 4: 3V3_BK4+ -> SMPS_OUT2_3V3+
Routing:
- net 3V3_BK4+: track 299.1 -> 0.00 mm, vias 19 -> 0
- net SMPS_OUT2_3V3+: track 0.00 -> 285.5 mm, vias 0 -> 18
- net 1V2_BK1+: track 139.9 -> 0.00 mm, vias 5 -> 0
- net SMPS_OUT1_1V2+: track 0.00 -> 107.8 mm, vias 0 -> 4
- net 1V8_LD5+: track 83.6 -> 0.00 mm, vias 5 -> 0
- net /FMC_D8: track 0.00 -> 71.6 mm, vias 0 -> 2
- net /Camera_Interface/CAMERA_SCL: track 66.3 -> 0.00 mm, vias 2 -> 0
- net /Camera_Interface/CAMERA_SDA: track 65.2 -> 0.00 mm, vias 2 -> 0
- net GND: track 288.7 -> 225.3 mm, vias 97 -> 164
- net /Memory/NAND_CLE: track 5.40 -> 65.1 mm, vias 0 -> 1
- net /Memory/NAND_ALE: track 5.45 -> 62.7 mm, vias 0 -> 1
- net /Memory/SDRAM_CKE: track 0.00 -> 53.9 mm, vias 0 -> 1
- net /Memory/NAND_CE#: track 55.3 -> 2.31 mm, vias 0 -> 1
- net /DCMIPP_D2: track 52.3 -> 0.00 mm, vias 1 -> 0
- net /DCMIPP_D3: track 51.8 -> 0.00 mm, vias 1 -> 0
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- added copper zone on F.Cu, net /Power_Management/SW1
- added copper zone on F.Cu, net /Power_Management/SW2
- added copper zone on F.Cu, net SMPS_OUT1_1V2+
- added copper zone on B.Cu, net SMPS_OUT2_3V3+
- added copper zone on F.Cu, net SMPS_OUT2_3V3+
- removed copper zone on B.Cu, net /Power_Management/VLX1
- removed copper zone on B.Cu, net /Power_Management/VLX3
- removed copper zone on B.Cu, net /Power_Management/VLX4
- removed copper zone on B.Cu, net 1V2_BK1+
- removed copper zone on B.Cu, net 2V8_BK3+
- removed copper zone on B.Cu, net 3V3_BK4+
- removed copper zone on B.Cu, net PWR_D+
Other:
- board text removed: "PONKEY"
