File: STM32H7_Board.kicad_pcb (KiCad board)
At the start: 4 copper layers, 100 x 50 mm, 95 parts, among them IC1 NAND_MT29F1G08ABAEAWP-IT_E_TR, IC5 STM32H7S3I8T6 LQFP 176, J1 BTB_10132798-062100LF, J2 I2S_OR_LJ_OUT, J22 USB_C_Receptacle_USB2.0_16P, J3 SWDB, J9 BTB_10132798-062100LF, Q1 MOSFET_SI2333DDS-T1-BE3, U7 USBLC6-2SC6, Y1 ECS-3225SMV-240-FP-TR

Commit message: Update
Routing:
- net GND: track 447.3 -> 467.0 mm, vias 353 -> 369
- net /Interface_Headers/NRST: track 223.9 -> 223.4 mm

Commit message: Pin typo fix
Parts:
- IC1: value NAND_MT29F1G08ABAEAWP-IT_E_TR -> NAND_MT29F2G08ABAGAWP-IT:G
Connections:
- U1 pad 2: /Interface_Headers/NRST -> GND
- U1 pad 3: GND -> /Interface_Headers/NRST
Routing:
- net GND: track 467.0 -> 474.9 mm, vias 369 -> 370
- net /Interface_Headers/NRST: track 223.4 -> 225.7 mm

Commit message: Update
Parts:
- removed R6: 33R, Resistor_SMD:R_0603_1608Metric
- removed RN12: 33R, Resistor_SMD:R_Array_Convex_4x0402
Connections:
- IC5 pad 39: /STM32H7S3I8T6/PA3_I2S6_MCK_R -> /Interface_Headers/BTB19
- IC5 pad 42: /STM32H7S3I8T6/PA4_I2S3_WS_R -> /Interface_Headers/BTB20
- IC5 pad 43: /STM32H7S3I8T6/PA5_I2S1_C_R -> /Interface_Headers/BTB22
- IC5 pad 45: /STM32H7S3I8T6/PA7_I2S6_SDO_R -> /Interface_Headers/BTB30
Routing:
- net /Interface_Headers/BTB19: track 27.0 -> 45.5 mm, vias 0 -> 1
- net /STM32H7S3I8T6/PA3_I2S6_MCK_R: track 17.7 -> 0.00 mm, vias 1 -> 0
- net /Interface_Headers/BTB20: track 29.4 -> 46.2 mm, vias 0 -> 1
- net /STM32H7S3I8T6/PA4_I2S3_WS_R: track 16.0 -> 0.00 mm, vias 1 -> 0
- net /Interface_Headers/BTB22: track 31.2 -> 46.5 mm, vias 0 -> 1
- net /STM32H7S3I8T6/PA5_I2S1_C_R: track 14.4 -> 0.00 mm, vias 1 -> 0
- net /Interface_Headers/BTB30: track 46.3 -> 51.2 mm, vias 0 -> 1
- net /STM32H7S3I8T6/PA7_I2S6_SDO_R: track 3.28 -> 0.00 mm, vias 1 -> 0
- net GND: track 474.9 -> 476.1 mm, vias 370 -> 371
- net /Interface_Headers/BTB31: track 26.2 -> 26.8 mm
