File: STM32H7S3I8T6.kicad_sch (KiCad schematic)
At the start: 43 parts, among them IC5 STM32H7S3I8T6 LQFP 176, J19 BOOT0_Jumper, Y1 Oscillator_ASE-50.000MHZ-L-R-T

Commit message: Update
Parts:
- C113, C116, C119, C86, C88, C90, C94, C97: footprint Capacitor_SMD:C_0805_2012Metric_Pad1.18x1.45mm_HandSolder -> Capacitor_SMD:C_0805_2012Metric
- FB5: renamed from FB3_BEAD(FCM1608KF-601T03)_600Ohm@100MHz1; value BLM21PG601SN1D_0805 -> BEAD(FCM1608KF-601T03)_600Ohm@100MHz1
- R20, R21, R22: footprint Resistor_SMD:R_0805_2012Metric_Pad1.20x1.40mm_HandSolder -> Resistor_SMD:R_0805_2012Metric_1
Connections:
- net AGND: no longer C100.1, C94.2, C96.1, C97.2
- net GND: now also C100.1, C94.2, C96.1, C97.2
- net PO0_XSPIM_P1_NCS1 renamed PO0
- net PO4_XSPIM_P1_CLK renamed PO4
- net PP0_XSPIM_P1_IO0 renamed PP0
- net PP1_XSPIM_P1_IO1 renamed PP1
- net PP2_XSPIM_P1_IO2 renamed PP2
- net PP3_XSPIM_P1_IO3 renamed PP3
- net USB_OTG_FS_DM renamed PM12
- net USB_OTG_FS_DP renamed PM11

Commit message: Update
Parts:
- FB5: footprint Capacitor_SMD:C_0805_2012Metric_Pad1.18x1.45mm_HandSolder -> Capacitor_SMD:C_0805_2012Metric
Connections:
- net AGND is gone; now on net GND: IC5.32 (VSSA), IC5.33 (VREFM)
- net GND: now also C22.2, IC5.118 (VSS_14)
- net SMPS_GND: no longer C22.2, IC5.118 (VSS_14)
Changed lines of the file:
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@@
 			)
 		)
-		(property "Value" "SMPS_GND"
+		(property "Value" "GND"
 			(at 306.578 129.032 0)
 			(effects
@@
 	)
 	(symbol
-		(lib_id "power:GND")
-		(at 149.86 175.26 270)
-		(unit 1)
-		(exclude_from_sim no)
-		(in_bom yes)
-		(on_board yes)
-		(dnp no)
-		(property "Reference" "#PWR0192"
-			(at 143.51 175.26 0)
-			(effects
-				(font
-					(size 1.27 1.27)
-				)
-				(hide yes)
-			)
-		)
-		(property "Value" "AGND"
-			(at 151.384 177.8 90)
-			(effects
-				(font
-					(size 1.27 1.27)
-				)
-				(justify right)
-			)
-		)
-		(property "Footprint" ""
-			(at 149.86 175.26 0)
-			(effects
-				(font
-					(size 1.27 1.27)
-				)
-				(hide yes)
-			)
-		)
-		(property "Datasheet" ""
-			(at 149.86 175.26 0)
-			(effects
-				(font
-					(size 1.27 1.27)
-				)
-				(hide yes)
-			)
-		)
-		(property "Description" "Power symbol creates a global label with name \"GND\" , ground"
-			(at 149.86 175.26 0)
-			(effects
-				(font
-					(size 1.27 1.27)
-				)
-				(hide yes)
-			)
-		)
-		(pin "1"
-		)
-		(instances
-			(project "STM32H7_Board"
-				(path "/9b48e30a-b912-4658-a133-1a15707d5b7d/c1266206-99aa-4330-9c51-1a1fe13fdf97"
-					(reference "#PWR0192")
-					(unit 1)
-				)
-			)
-		)
-	)
-	(symbol
 		(lib_id "Device:C")
 		(at 265.43 36.83 0)
@@
 	(symbol
 		(lib_id "power:GND")
+		(at 149.86 175.26 270)
+		(mirror x)
+		(unit 1)
+		(exclude_from_sim no)
+		(in_bom yes)
+		(on_board yes)
+		(dnp no)
+		(fields_autoplaced yes)
+		(property "Reference" "#PWR01"
+			(at 143.51 175.26 0)
+			(effects
+				(font
+					(size 1.27 1.27)
+				)
+				(hide yes)
+			)
+		)
+		(property "Value" "GND"
+			(at 144.78 175.26 0)
+			(effects
+				(font
+					(size 1.27 1.27)
+				)
+				(hide yes)
+			)
+		)
+		(property "Footprint" ""
+			(at 149.86 175.26 0)
+			(effects
+				(font
+					(size 1.27 1.27)
+				)
+				(hide yes)
+			)
+		)
+		(property "Datasheet" ""
+			(at 149.86 175.26 0)
+			(effects
+				(font
+					(size 1.27 1.27)
+				)
+				(hide yes)
+			)
+		)
+		(property "Description" "Power symbol creates a global label with name \"GND\" , ground"
+			(at 149.86 175.26 0)
+			(effects
+				(font
+					(size 1.27 1.27)
+				)
+				(hide yes)
+			)
+		)
+		(pin "1"
+		)
+		(instances
+			(project "STM32H7_Board"
+				(path "/9b48e30a-b912-4658-a133-1a15707d5b7d/c1266206-99aa-4330-9c51-1a1fe13fdf97"
+					(reference "#PWR01")
+					(unit 1)
+				)
+			)
+		)
+	)
+	(symbol
+		(lib_id "power:GND")
 		(at 271.78 232.41 0)
 		(mirror y)
@@
 			)
 		)
-		(property "Footprint" "Capacitor_SMD:C_0805_2012Metric_Pad1.18x1.45mm_HandSolder"
+		(property "Footprint" "Capacitor_SMD:C_0805_2012Metric"
 			(at 293.37 32.258 90)
 			(effects

Commit message: Update
Parts:
- removed C113: 100n, Capacitor_SMD:C_0805_2012Metric, symbol Device:C
- removed C116: 1u, Capacitor_SMD:C_0805_2012Metric, symbol Device:C
- removed C119: 4u7, Capacitor_SMD:C_0805_2012Metric, symbol Device:C
- removed FB5: BEAD(FCM1608KF-601T03)_600Ohm@100MHz1, Capacitor_SMD:C_0805_2012Metric, symbol Device:FerriteBead
Connections:
- net 1V8_LD3+ is gone; now on net 3V3_BK3+: C106.1, C107.1, C110.1, C112.1, IC5.63 (VDDXSPI1_1), IC5.69 (VDDXSPI1_2), IC5.75 (VDDXSPI1_3), IC5.81 (VDDXSPI1_4)
- net SMPS_GND is gone; now on net GND: C104.2, C57.2, C9.2, IC5.167 (VSS_16), IC5.60 (VSS_6), IC5.98 (VSS_12)
- net USB_OTG_HS_VBUS_FR is gone; now on net 3V3_BK3+: IC5.140 (VDD50USB)
- net VDD33USB is gone; now on net 3V3_BK3+: C111.2, IC5.141 (VDD33USB)
Other:
- note added: "USB regulator supply input"

Commit message: Update
Parts:
- Y1: value Oscillator_ASE-50.000MHZ-L-R-T -> ECS-3225SMV-240-FP-TR
Other:
- note added: "ECS-3225SMV-240-FP-TR"
Changed lines of the file:
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@@
 		)
 	)
+	(text "ECS-3225SMV-240-FP-TR"
+		(exclude_from_sim no)
+		(at 37.338 140.462 0)
+		(effects
+			(font
+				(size 1 1)
+			)
+		)
+	)
 	(text "Connect VCAPS together"
 		(exclude_from_sim no)
@@
 			)
 		)
-		(property "Value" "Oscillator_ASE-50.000MHZ-L-R-T"
+		(property "Value" "ECS-3225SMV-240-FP-TR"
 			(at 52.07 147.32 0)
 			(effects

Commit message: Update
Parts:
- removed C100: 100n, Capacitor_SMD:C_0805_2012Metric, symbol Device:C
- removed C96: 1u, Capacitor_SMD:C_0805_2012Metric, symbol Device:C
Connections:
- net PE2 is gone; now on net FMC_D11: IC5.172 (PE2)
- net SDMMC1_D0 is gone; now on net DCMIPP_D2: IC5.105 (PC8)
- net SDMMC1_D1 is gone; now on net DCMIPP_D3: IC5.106 (PC9)
- net DCMIPP_D2: no longer IC5.170 (PE0)
- net DCMIPP_D3: no longer IC5.171 (PE1)
- net FMC_D10: now also IC5.171 (PE1); no longer IC5.92 (PB11)
- net FMC_D11: no longer IC5.91 (PB10)
- net FMC_D9: now also IC5.170 (PE0); no longer IC5.93 (PB12)
- net 3V3_BK3+ renamed 3V3_BK4+
- net BK1+ renamed 1V2_BK1+
- net DCMIPP_PIXCLK renamed PF8_DCMIPP_PIXCLK
- net FMC_INT renamed PD13
- net PA13_SWDIO renamed PA13_DEBUG_JTMS-SWDIO
- net PA14_SWCLK renamed PA14_DEBUG_JTCK-SWCLK
- net PA15_I2S1_WS renamed PA15_I2S6_WS
- net PA4_I2S6_WS renamed PA4_I2S1_WS
- net PA5_I2S6_CK renamed PA5_I2S1_CK
- net PA7_I2S6_SDO renamed PA7_FMC_INT
- net PB0_I2S1_CK renamed PB0_GFXTIM_TE
- net PB13_UART5_TX/RX renamed PB13_SPI2_SCK
- net PB14_USART1_TX/RX renamed PB14_SPI2_MISO
- net PB15 renamed PB15_SPI2_MOSI
- net PB3_SWO renamed PB3_DEBUG_JTDO-SWO
- net PB5 renamed PB5_I2S6_SDO
- net PB6_I2C1_SCL renamed PB6_UART5_TX
- net PF11 renamed PF11_ADC1_INP2
- net PF7_SPI5_SCK renamed PF7_UART7_TX
- net PF9_SPI5_MOSI renamed PF9_TIM14_CH1
- net PM0 renamed PM0_UCPD1_CC1
- net PM1 renamed PM1_UCPD1_CC2
- net PM14_SPI5_MISO renamed PM14
- net PO0 renamed PO0_XSPIM_P1_NCS1
- net PO4 renamed PO4_XSPIM_P1_CLK
- net PP0 renamed PP0_XSPIM_P1_IO0
- net PP1 renamed PP1_XSPIM_P1_IO1
- net PP2 renamed PP2_XSPIM_P1_IO2
- net PP3 renamed PP3_XSPIM_P1_IO3
- net SDMMC1_CK renamed PC12_I2S6_CK
- net SDMMC1_CKIN renamed PB8_I2C1_SCL
- net SDMMC1_CMD renamed PD2
- net SDMMC1_D2 renamed PC10
- net SDMMC1_D3 renamed PC11
- new net PB10_I2C2_SCL: IC5.91 (PB10)
- new net PB11_I2C2_SDA: IC5.92 (PB11)
- new net PB12_SPI2_NSS: IC5.93 (PB12)
Other:
- note removed: "Bank Address 0 (BA0)"
- note removed: "Connect VCAPS together"
- note removed: "SDRAM1"
- moved on the sheet: C102, C106, C107, C110, C112, C95

Commit message: Update
Parts:
- removed C106, C107, C110, C112: 100n, Capacitor_SMD:C_0805_2012Metric, symbol Device:C
- removed J19: BOOT0_Jumper, Connector_PinHeader_2.54mm:PinHeader_1x03_P2.54mm_Vertical, symbol Connector_Generic:Conn_01x03
- removed R22: 1k, Resistor_SMD:R_0805_2012Metric_1, symbol Device:R
- added CN1: 100n, Resistor_SMD:R_Array_Concave_4x0603, symbol Personal_Projects:C_Network04
- added RN1, RN10, RN14, RN2, RN3, RN4, RN5, RN6, RN7, RN8, RN9: 33R, Resistor_SMD:R_Array_Convex_4x0402, symbol Device:R_Pack04
- R21: value 22R -> 51R
Connections:
- net 3V3_BK4+: now also CN1.5 (C4), CN1.6 (C3), CN1.7 (C2), CN1.8 (C1)
- net FMC_A0: now also RN6.2 (R2.1); no longer IC5.29 (PC1)
- net FMC_A1: now also RN6.3 (R3.1); no longer IC5.30 (PC2)
- net FMC_A10: now also RN3.7 (R2.2); no longer IC5.160 (PF2)
- net FMC_A11: now also RN3.8 (R1.2); no longer IC5.161 (PF3)
- net FMC_A12: now also RN4.2 (R2.1); no longer IC5.55 (PE8)
- net FMC_A2: now also RN6.4 (R4.1); no longer IC5.31 (PC3)
- net FMC_A3: now also RN8.1 (R1.1); no longer IC5.46 (PC4)
- net FMC_A4: now also RN4.1 (R1.1); no longer IC5.54 (PE7)
- net FMC_A5: now also RN8.2 (R2.1); no longer IC5.47 (PC5)
- net FMC_A6: now also RN10.6 (R3.2); no longer IC5.124 (PD0)
- net FMC_A7: now also RN10.7 (R2.2); no longer IC5.125 (PD1)
- net FMC_A8: now also RN3.5 (R4.2); no longer IC5.158 (PF0)
- net FMC_A9: now also RN3.6 (R3.2); no longer IC5.159 (PF1)
- net FMC_ALE: now also RN5.2 (R2.1); no longer IC5.18 (PF6)
- net FMC_BA0: now also RN4.3 (R3.1); no longer IC5.56 (PE9)
- net FMC_BA1: now also RN4.4 (R4.1); no longer IC5.57 (PE10)
- net FMC_CLE: now also RN5.1 (R1.1); no longer IC5.17 (PF5)
- net FMC_D10: now also RN2.7 (R2.2); no longer IC5.171 (PE1)
- net FMC_D11: now also RN2.8 (R1.2); no longer IC5.172 (PE2)
- net FMC_D12: now also RN1.1 (R1.1); no longer IC5.7 (PE3)
- net FMC_D13: now also RN1.2 (R2.1); no longer IC5.8 (PE4)
- net FMC_D14: now also RN1.3 (R3.1); no longer IC5.9 (PE5)
- net FMC_D15: now also RN1.4 (R4.1); no longer IC5.10 (PE6)
- net FMC_D5: now also RN7.3 (R3.1); no longer IC5.38 (PA2)
- net FMC_D6: now also RN7.2 (R2.1); no longer IC5.37 (PA1)
- net FMC_D7: now also RN7.1 (R1.1); no longer IC5.36 (PA0)
- net FMC_D8: now also RN14.8 (R1.2); no longer IC5.156 (PD7)
- net FMC_D9: now also RN2.6 (R3.2); no longer IC5.170 (PE0)
- net FMC_NBL1: now also RN6.1 (R1.1); no longer IC5.28 (PC0)
- net FMC_NCE: now also RN14.6 (R3.2); no longer IC5.154 (PD5)
- net FMC_NOE: now also RN8.3 (R3.1); no longer IC5.49 (PB1)
- net FMC_NWE: now also RN8.4 (R4.1); no longer IC5.50 (PB2)
- net FMC_SDCKE0: now also RN9.8 (R1.2); no longer IC5.131 (PE15)
- net FMC_SDNCAS: now also RN9.6 (R3.2); no longer IC5.129 (PE13)
- net FMC_SDNE0: now also RN9.7 (R2.2); no longer IC5.130 (PE14)
- net FMC_SDNRAS: now also RN9.5 (R4.2); no longer IC5.128 (PE12)
- net FMC_SDNWE: now also RN10.8 (R1.2); no longer IC5.127 (PE11)
- net GND: now also CN1.1 (common), CN1.2 (common), CN1.3 (common), CN1.4 (common)
- net PF8_DCMIPP_PIXCLK: now also RN5.3 (R3.1); no longer IC5.20 (PF8)
- net PF9_TIM14_CH1: now also RN5.4 (R4.1); no longer IC5.21 (PF9)
- net PH0-OSC_IN: now also R21.2; no longer R21.1
- net at Y1.3 (OUTPUT): now also R21.1; no longer R21.2
- net DCMIPP_D9 renamed PD15
- net FMC_NE1 renamed PD12
- net PA4_I2S1_WS renamed PA4_I2S3_WS
- net PA5_I2S1_CK renamed PA5
- net PB4_I2S1_SDI renamed PB4
- net PC10 renamed PC10_I2S3_CK
- net PC11 renamed PC11_I2S3_SDI
- net PD6 renamed PD6_FMC_NE3_R
- net PD6_FMC_NE3_R: now also RN14.2 (R2.1)
- net PF4_DCMIPP_D8 renamed PF4
- new net: IC5.172 (PE2), RN2.1 (R1.1)
- new net: IC5.171 (PE1), RN2.2 (R2.1)
- new net: IC5.170 (PE0), RN2.3 (R3.1)
- new net: IC5.158 (PF0), RN3.4 (R4.1)
- new net: IC5.159 (PF1), RN3.3 (R3.1)
- new net: IC5.160 (PF2), RN3.2 (R2.1)
- new net: IC5.161 (PF3), RN3.1 (R1.1)
- new net: IC5.17 (PF5), RN5.8 (R1.2)
- new net: IC5.18 (PF6), RN5.7 (R2.2)
- new net: IC5.20 (PF8), RN5.6 (R3.2)
- new net: IC5.21 (PF9), RN5.5 (R4.2)
- new net: IC5.54 (PE7), RN4.8 (R1.2)
- new net: IC5.55 (PE8), RN4.7 (R2.2)
- new net: IC5.56 (PE9), RN4.6 (R3.2)
- new net: IC5.57 (PE10), RN4.5 (R4.2)
- new net FMC_A0_R: IC5.29 (PC1), RN6.7 (R2.2)
- new net FMC_A1_R: IC5.30 (PC2), RN6.6 (R3.2)
- new net FMC_A2_R: IC5.31 (PC3), RN6.5 (R4.2)
- new net FMC_A3_R: IC5.46 (PC4), RN8.8 (R1.2)
- new net FMC_A5_R: IC5.47 (PC5), RN8.7 (R2.2)
- new net FMC_A6_R: IC5.124 (PD0), RN10.3 (R3.1)
- new net FMC_A7_R: IC5.125 (PD1), RN10.2 (R2.1)
- new net FMC_D12_R: IC5.7 (PE3), RN1.8 (R1.2)
- new net FMC_D13_R: IC5.8 (PE4), RN1.7 (R2.2)
- new net FMC_D14_R: IC5.9 (PE5), RN1.6 (R3.2)
- new net FMC_D15_R: IC5.10 (PE6), RN1.5 (R4.2)
- new net FMC_D5_R: IC5.38 (PA2), RN7.6 (R3.2)
- new net FMC_D6_R: IC5.37 (PA1), RN7.7 (R2.2)
- new net FMC_D7_R: IC5.36 (PA0), RN7.8 (R1.2)
- new net FMC_D8_R: IC5.156 (PD7), RN14.1 (R1.1)
- new net FMC_NBL1_R: IC5.28 (PC0), RN6.8 (R1.2)
- new net FMC_NCE_R: IC5.154 (PD5), RN14.3 (R3.1)
- new net FMC_NOE_R: IC5.49 (PB1), RN8.6 (R3.2)
- new net FMC_NWE_R: IC5.50 (PB2), RN8.5 (R4.2)
- new net FMC_SDCKE0_R: IC5.131 (PE15), RN9.1 (R1.1)
- new net FMC_SDNCAS_R: IC5.129 (PE13), RN9.3 (R3.1)
- new net FMC_SDNE0_R: IC5.130 (PE14), RN9.2 (R2.1)
- new net FMC_SDNRAS_R: IC5.128 (PE12), RN9.4 (R4.1)
- new net FMC_SDNWE_R: IC5.127 (PE11), RN10.1 (R1.1)
- new net PD6_FMC_NE3: RN14.7 (R2.2)
- no-connect marks 5 -> 13
Other:
- note removed: "Place it as close as possible to the oscillator's output pin"
- note removed: "SMPS Input Capacitor (Data Sheet)"
- moved on the sheet: C101, C102, C103, C105, C88, C91, C93, C94, C95, C97, C98, FB1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

Commit message: Update
Parts:
- added C5: 100n, Capacitor_SMD:C_0603_1608Metric, symbol Device:C
- added R2: 33R, Resistor_SMD:R_0603_1608Metric, symbol Device:R
- added RN15: 33R, Resistor_SMD:R_Array_Convex_4x0402, symbol Device:R_Pack04
Connections:
- net 3V3_BK4+: no longer CN1.5 (C4), CN1.6 (C3), CN1.7 (C2), CN1.8 (C1), IC5.63 (VDDXSPI1_1), IC5.69 (VDDXSPI1_2), IC5.75 (VDDXSPI1_3), IC5.81 (VDDXSPI1_4)
- net DCMIPP_D0: now also RN15.5 (R4.2); no longer IC5.103 (PC6)
- net DCMIPP_D1: now also RN15.6 (R3.2); no longer IC5.104 (PC7)
- net DCMIPP_D2: now also RN15.7 (R2.2); no longer IC5.105 (PC8)
- net DCMIPP_D3: now also RN15.8 (R1.2); no longer IC5.106 (PC9)
- net DCMIPP_D7: now also R2.2; no longer IC5.101 (PD14)
- net GND: now also C5.1
- net NRST: now also C5.2
- net PF9_TIM14_CH1: now also IC5.21 (PF9); no longer RN5.4 (R4.1)
- net at RN5.5 (R4.2): no longer IC5.21 (PF9)
- new net 1V8_LD5+: CN1.5 (C4), CN1.6 (C3), CN1.7 (C2), CN1.8 (C1), IC5.63 (VDDXSPI1_1), IC5.69 (VDDXSPI1_2), IC5.75 (VDDXSPI1_3), IC5.81 (VDDXSPI1_4)
- new net DCMIPP_D0_R: IC5.103 (PC6), RN15.4 (R4.1)
- new net DCMIPP_D1_R: IC5.104 (PC7), RN15.3 (R3.1)
- new net DCMIPP_D2_R: IC5.105 (PC8), RN15.2 (R2.1)
- new net DCMIPP_D3_R: IC5.106 (PC9), RN15.1 (R1.1)
- new net DCMIPP_D7_R: IC5.101 (PD14), R2.1
- no-connect marks 13 -> 15
Other:
- moved on the sheet: C121, C122

Commit message: Update
Parts:
- added R10, R7: 33R, Resistor_SMD:R_0603_1608Metric, symbol Device:R
- added RN16: 33R, Resistor_SMD:R_Array_Convex_4x0402, symbol Device:R_Pack04
Connections:
- net FMC_D0: now also RN16.8 (R1.2); no longer IC5.113 (PA12)
- net FMC_D1: now also RN16.7 (R2.2); no longer IC5.112 (PA11)
- net FMC_D2: now also RN16.6 (R3.2); no longer IC5.111 (PA10)
- net FMC_D3: now also RN16.5 (R4.2); no longer IC5.110 (PA9)
- net FMC_D4: now also R10.2; no longer IC5.109 (PA8)
- net FMC_D8: now also R7.2; no longer RN14.8 (R1.2)
- net FMC_D8_R: now also R7.1; no longer RN14.1 (R1.1)
- new net FMC_D0_R: IC5.113 (PA12), RN16.1 (R1.1)
- new net FMC_D1_R: IC5.112 (PA11), RN16.2 (R2.1)
- new net FMC_D2_R: IC5.111 (PA10), RN16.3 (R3.1)
- new net FMC_D3_R: IC5.110 (PA9), RN16.4 (R4.1)
- new net FMC_D4_R: IC5.109 (PA8), R10.1
- no-connect marks 15 -> 17
Other:
- moved on the sheet: RN14
