File: STM32H7S3I8T6.kicad_sch (KiCad schematic)
At the start: 49 parts, among them CN1 100n, IC5 STM32H7S3I8T6 LQFP 176, Y1 ECS-3225SMV-240-FP-TR

Commit message: Update
Parts:
- removed R10: 33R, Resistor_SMD:R_0603_1608Metric, symbol Device:R
- removed RN16: 33R, Resistor_SMD:R_Array_Convex_4x0402, symbol Device:R_Pack04
Connections:
- net FMC_SDCKE0 is gone; now on net FMC_D1: RN9.8 (R1.2)
- net FMC_SDNCAS is gone; now on net FMC_D3: RN9.6 (R3.2)
- net FMC_SDNE0 is gone; now on net FMC_D2: RN9.7 (R2.2)
- net FMC_SDNRAS is gone; now on net FMC_D4: RN9.5 (R4.2)
- net PB4 is gone; now on net DCMIPP_VSYNC: IC5.164 (PB4)
- net PF4 is gone; now on net FMC_A13_R: IC5.162 (PF4)
- net DCMIPP_VSYNC: no longer IC5.174 (PB7)
- net FMC_ALE: now also RN5.3 (R3.1); no longer RN5.2 (R2.1)
- net FMC_CLE: now also RN5.2 (R2.1); no longer RN5.1 (R1.1)
- net FMC_D0: now also RN10.5 (R4.2)
- net FMC_D0_R: now also RN10.4 (R4.1)
- net FMC_D1_R: now also RN9.1 (R1.1)
- net FMC_D2_R: now also RN9.2 (R2.1)
- net FMC_D3_R: now also RN9.3 (R3.1)
- net FMC_D4_R: now also RN9.4 (R4.1)
- net PF8_DCMIPP_PIXCLK: now also RN5.4 (R4.1); no longer RN5.3 (R3.1)
- net at IC5.17 (PF5): now also RN5.7 (R2.2); no longer RN5.8 (R1.2)
- net at IC5.18 (PF6): now also RN5.6 (R3.2); no longer RN5.7 (R2.2)
- net at IC5.20 (PF8): now also RN5.5 (R4.2); no longer RN5.6 (R3.2)
- net at RN4.5 (R4.2): no longer IC5.57 (PE10)
- net FMC_BA0 renamed FMC_A14
- net FMC_BA1: no longer names the net of RN4.4 (R4.1)
- net FMC_NBL0 renamed PD8
- net FMC_NBL1: no longer names the net of RN6.1 (R1.1)
- net FMC_NBL1_R: no longer names the net of RN6.8 (R1.2)
- net FMC_NBL1_R: no longer IC5.28 (PC0)
- net FMC_SDCKE0_R renamed PE15
- net PE15: no longer RN9.1 (R1.1)
- net FMC_SDCLK renamed PD9
- net FMC_SDNCAS_R renamed PE13
- net PE13: no longer RN9.3 (R3.1)
- net FMC_SDNE0_R renamed PE14
- net PE14: no longer RN9.2 (R2.1)
- net FMC_SDNRAS_R renamed PE12
- net PE12: no longer RN9.4 (R4.1)
- net FMC_SDNWE renamed FMC_A13
- net FMC_SDNWE_R renamed FMC_A13_R
- net FMC_A13_R: no longer IC5.127 (PE11)
- net PD12 renamed PD12_FMC_NE1
- new net PB7: IC5.174 (PB7)
- new net PC0: IC5.28 (PC0)
- new net PE10: IC5.57 (PE10)
- new net PE11: IC5.127 (PE11)
- no-connect marks 17 -> 19
Other:
- moved on the sheet: RN10, RN4, RN5, RN6

Commit message: Update
Parts:
- added RN16: 33R, Resistor_SMD:R_Array_Convex_4x0402, symbol Device:R_Pack04
Connections:
- net PE10 is gone; now on net FMC_BA1_R: IC5.57 (PE10)
- net PE11 is gone; now on net PE11_FMC_SDNWE_R: IC5.127 (PE11)
- net FMC_CLE_R: now reaches IC5.17 (PF5), RN5.7 (R2.2)
- net FMC_ALE_R: now reaches IC5.18 (PF6), RN5.6 (R3.2)
- net FMC_A4_R: now reaches IC5.54 (PE7), RN4.8 (R1.2)
- net FMC_A12_R: now reaches IC5.55 (PE8), RN4.7 (R2.2)
- net FMC_BA0_R: now reaches IC5.56 (PE9), RN4.6 (R3.2)
- net FMC_BA1: now reaches RN4.4 (R4.1)
- net FMC_BA1_R: now reaches RN4.5 (R4.2)
- net FMC_A13 renamed PE11_FMC_SDNWE
- net FMC_A13_R renamed PE11_FMC_SDNWE_R
- net PE11_FMC_SDNWE_R: no longer IC5.162 (PF4)
- net FMC_A14 renamed FMC_BA0
- net PD12_FMC_NE1 renamed PD12
- net PD8 renamed PD8_FMC_NBL0
- net PD9 renamed FMC_SDCLK
- net PE12 renamed PE12_FMC_SDNRAS_R
- net PE12_FMC_SDNRAS_R: now also RN16.4 (R4.1)
- net PE13 renamed PE13_FMC_SDNCAS_R
- net PE13_FMC_SDNCAS_R: now also RN16.3 (R3.1)
- net PE14 renamed PE14_FMC_SDNE0_R
- net PE14_FMC_SDNE0_R: now also RN16.2 (R2.1)
- net PE15 renamed PE15_FMC_SDCKE0_R
- net PE15_FMC_SDCKE0_R: now also RN16.1 (R1.1)
- new net PE12_FMC_SDNRAS: RN16.5 (R4.2)
- new net PE13_FMC_SDNCAS: RN16.6 (R3.2)
- new net PE14_FMC_SDNE0: RN16.7 (R2.2)
- new net PE15_FMC_SDCKE0: RN16.8 (R1.2)
- new net PF4: IC5.162 (PF4)
- no-connect marks 19 -> 17

Commit message: Update
Parts:
- removed CN1: 100n, Resistor_SMD:R_Array_Concave_4x0603, symbol Personal_Projects:C_Network04
- removed R7: 33R, Resistor_SMD:R_0603_1608Metric, symbol Device:R
- added R6: 33R, Resistor_SMD:R_0603_1608Metric, symbol Device:R
- added RN11, RN12: 33R, Resistor_SMD:R_Array_Convex_4x0402, symbol Device:R_Pack04
Connections:
- net 3V3_BK4+ is gone; now on net SMPS_OUT2_3V3+: C101.1, C102.1, C103.1, C105.1, C108.1, C109.2, C111.2, C114.1, C115.1, C120.1, C121.1, C122.1, C86.1, C88.1, C90.2, C91.1, C93.1, C95.1, C98.1, FB1.1, IC5.1 (VBAT), IC5.100 (VDD_8), IC5.107 (VDD_9), IC5.12 (VDD_2), IC5.120 (VDD_10), IC5.133 (VDD_11), IC5.140 (VDD50USB), IC5.141 (VDD33USB), IC5.145 (DVDD), IC5.148 (VDD_12), IC5.157 (VDD_13), IC5.169 (VDD_14), IC5.27 (VDD_3), IC5.41 (VDD_4), IC5.5 (VDD_1), IC5.51 (VDD_5), IC5.58 (VDD_6), IC5.87 (VDD_7), OS3.4 (VDD), Y1.4 (VDD)
- net FMC_D8: now also RN14.8 (R1.2)
- net FMC_D8_R: now also RN14.1 (R1.1)
- net FMC_NCE: now also IC5.154 (PD5); no longer RN14.6 (R3.2)
- net PA3_I2S6_MCK: now also RN12.1 (R1.1); no longer IC5.39 (PA3)
- net PA4_I2S3_WS: now also RN12.2 (R2.1); no longer IC5.42 (PA4)
- net PD8_FMC_NBL0: now also RN11.2 (R2.1); no longer IC5.83 (PD8)
- net at RN5.5 (R4.2): no longer IC5.20 (PF8)
- net 1V2_BK1+ renamed SMPS_OUT1_1V2+
- net 1V8_LD5+ renamed SMPS_OUT2_3V3+
- net DCMIPP_D0 renamed PC6_PSSI_D0
- net DCMIPP_D0_R renamed PC6_PSSI_D0_R
- net DCMIPP_D1 renamed PC7_PSSI_D1
- net DCMIPP_D1_R renamed PC7_PSSI_D1_R
- net DCMIPP_D2 renamed PC8_PSSI_D2
- net DCMIPP_D2_R renamed PC8_PSSI_D2_R
- net DCMIPP_D3 renamed PC9_PSSI_D3
- net DCMIPP_D3_R renamed PC9_PSSI_D3_R
- net DCMIPP_D4 renamed PD10_PSSI_D4
- net DCMIPP_D5 renamed PD3_PSSI_D5
- net DCMIPP_D6 renamed PD11_PSSI_D6
- net DCMIPP_D7 renamed PD14_PSSI_D7
- net DCMIPP_D7_R renamed PD14_PSSI_D7_R
- net DCMIPP_HSYNC renamed PD4_PSSI_DE
- net DCMIPP_VSYNC renamed PB4_I2S1_SDI
- net FMC_NCE_R: no longer names the net of RN14.3 (R3.1)
- net FMC_NCE_R: no longer IC5.154 (PD5)
- net FMC_SDCLK renamed PD9_FMC_SDCLK_R
- net PD9_FMC_SDCLK_R: now also RN11.6 (R3.2)
- net PA5 renamed PA5_I2S1_C_R
- net PA5_I2S1_C_R: now also RN12.6 (R3.2)
- net PA7_FMC_INT renamed PA7_I2S6_SDO_R
- net PA7_I2S6_SDO_R: now also R6.2
- net PB10_I2C2_SCL renamed PB10_SPI2_SCK
- net PB11_I2C2_SDA renamed PB11
- net PB13_SPI2_SCK renamed PB13_UART5_TX
- net PB5_I2S6_SDO renamed PB5_SPI3_MOSI
- net PB6_UART5_TX renamed PB6_LPUART1_TX
- net PB7 renamed PB7_PSSI_RDY
- net PC10_I2S3_CK renamed PC10_SPI3_SCK
- net PC11_I2S3_SDI renamed PC11_SPI3_MISO
- net PD13 renamed PD13_FMC_INT
- net PF8_DCMIPP_PIXCLK: no longer names the net of RN5.4 (R4.1)
- net PO0_XSPIM_P1_NCS1 renamed PO0
- net PO4_XSPIM_P1_CLK renamed PO4
- net PP0_XSPIM_P1_IO0 renamed PP0
- net PP1_XSPIM_P1_IO1 renamed PP1
- net PP2_XSPIM_P1_IO2 renamed PP2
- net PP3_XSPIM_P1_IO3 renamed PP3
- new net PA3_I2S6_MCK_R: IC5.39 (PA3), RN12.8 (R1.2)
- new net PA4_I2S3_WS_R: IC5.42 (PA4), RN12.7 (R2.2)
- new net PA5_I2S1_CK: RN12.3 (R3.1)
- new net PA7_I2S6_SDO: R6.1
- new net PD8_FMC_NBL0_R: IC5.83 (PD8), RN11.7 (R2.2)
- new net PD9_FMC_SDCLK: RN11.3 (R3.1)
- new net PF8_PSSI_PDCK: IC5.20 (PF8)
- no-connect marks 17 -> 25
Other:
- moved on the sheet: C114, RN5

Commit message: Update
Connections:
- net FMC_D11_R: now reaches IC5.172 (PE2), RN2.1 (R1.1)
- net FMC_D10_R: now reaches IC5.171 (PE1), RN2.2 (R2.1)
- net FMC_D9_R: now reaches IC5.170 (PE0), RN2.3 (R3.1)
- net FMC_A8_R: now reaches IC5.158 (PF0), RN3.4 (R4.1)
- net FMC_A9_R: now reaches IC5.159 (PF1), RN3.3 (R3.1)
- net FMC_A10_R: now reaches IC5.160 (PF2), RN3.2 (R2.1)
- net FMC_A11_R: now reaches IC5.161 (PF3), RN3.1 (R1.1)
Changed lines of the file:
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@@
+		)
+	)
+	(label "FMC_D10_R"
+		(at 175.26 67.31 270)
+		(fields_autoplaced yes)
+		(effects
+			(font
+				(size 1.27 1.27)
+			)
+			(justify right bottom)
 		)
 	)
@@
 		)
 	)
+	(label "FMC_A8_R"
+		(at 208.28 72.39 270)
+		(fields_autoplaced yes)
+		(effects
+			(font
+				(size 1.27 1.27)
+			)
+			(justify right bottom)
+		)
+	)
 	(label "PB9_I2C1_SDA"
 		(at 151.13 55.88 270)
@@
 		)
 	)
+	(label "FMC_A9_R"
+		(at 205.74 72.39 270)
+		(fields_autoplaced yes)
+		(effects
+			(font
+				(size 1.27 1.27)
+			)
+			(justify right bottom)
+		)
+	)
 	(label "PC8_PSSI_D2_R"
 		(at 306.07 165.1 180)
@@
 		)
 	)
+	(label "FMC_A10_R"
+		(at 203.2 72.39 270)
+		(fields_autoplaced yes)
+		(effects
+			(font
+				(size 1.27 1.27)
+			)
+			(justify right bottom)
+		)
+	)
 	(label "PP2"
 		(at 215.9 248.92 90)
@@
 		)
 	)
+	(label "FMC_A11_R"
+		(at 200.66 72.39 270)
+		(fields_autoplaced yes)
+		(effects
+			(font
+				(size 1.27 1.27)
+			)
+			(justify right bottom)
+		)
+	)
 	(label "PA6_TIM13_CH1"
 		(at 130.81 210.82 0)
@@
 		(fields_autoplaced yes)
 		(effects
+			(font
+				(size 1.27 1.27)
+			)
+			(justify right bottom)
+		)
+	)
+	(label "FMC_D11_R"
+		(at 172.72 67.31 270)
+		(fields_autoplaced yes)
+		(effects
+			(font
+				(size 1.27 1.27)
+			)
+			(justify right bottom)
+		)
+	)
+	(label "FMC_D9_R"
+		(at 177.8 67.31 270)
+		(fields_autoplaced yes)
+		(effects

Commit message: Update
Parts:
- added RN13: 33R, Resistor_SMD:R_Array_Convex_4x0402, symbol Device:R_Pack04
Connections:
- net FMC_NCE: now also RN13.7 (R2.2); no longer IC5.154 (PD5)
- net PB0_GFXTIM_TE: now also RN13.8 (R1.2); no longer IC5.48 (PB0)
- net PC13: now also RN13.6 (R3.2); no longer IC5.2 (PC13)
- new net FMC_NCE_R: IC5.154 (PD5), RN13.2 (R2.1)
- new net PB0_GFXTIM_TE_R: IC5.48 (PB0), RN13.1 (R1.1)
- new net PC13_R: IC5.2 (PC13), RN13.3 (R3.1)
- no-connect marks 25 -> 27
Other:
- moved on the sheet: RN12

Commit message: Update
Parts:
- removed R2: 33R, Resistor_SMD:R_0603_1608Metric, symbol Device:R
- removed RN15: 33R, Resistor_SMD:R_Array_Convex_4x0402, symbol Device:R_Pack04
Connections:
- net PC6_PSSI_D0_R is gone; now on net PC6_PSSI_D0: IC5.103 (PC6)
- net PC7_PSSI_D1_R is gone; now on net PC7_PSSI_D1: IC5.104 (PC7)
- net PC8_PSSI_D2_R is gone; now on net PC8_PSSI_D2: IC5.105 (PC8)
- net PC9_PSSI_D3_R is gone; now on net PC9_PSSI_D3: IC5.106 (PC9)
- net PD14_PSSI_D7_R is gone; now on net PD14_PSSI_D7: IC5.101 (PD14)
- net FMC_A0: now also RN6.1 (R1.1); no longer RN6.2 (R2.1)
- net FMC_A0_R: now also RN6.8 (R1.2); no longer RN6.7 (R2.2)
- net FMC_ALE: now also RN5.4 (R4.1); no longer RN5.3 (R3.1)
- net FMC_ALE_R: now also RN5.5 (R4.2); no longer RN5.6 (R3.2)
- net FMC_D9: now also RN2.5 (R4.2); no longer RN2.6 (R3.2)
- net FMC_D9_R: now also RN2.4 (R4.1); no longer RN2.3 (R3.1)
- net PA4_I2S3_WS: now also RN12.3 (R3.1); no longer RN12.2 (R2.1)
- net PA4_I2S3_WS_R: now also RN12.6 (R3.2); no longer RN12.7 (R2.2)
- net PA5_I2S1_CK: now also RN12.4 (R4.1); no longer RN12.3 (R3.1)
- net PA5_I2S1_C_R: now also RN12.5 (R4.2); no longer RN12.6 (R3.2)
- net PD8_FMC_NBL0: now also RN11.1 (R1.1); no longer RN11.2 (R2.1)
- net PD8_FMC_NBL0_R: now also RN11.8 (R1.2); no longer RN11.7 (R2.2)
Other:
- note removed: "ALLOW FOR THE POSSIBILITYY OF BOTH SMPS AND LDO"
- note removed: "BOOT0 Switch HIGH enables UART or I2C too allow programminng of the MCU 0 Boot from the user flash memory at x0800 0000 1 Boot from the bootloader"
- note removed: "Connect OTG_HS_SO through a jumper as a debug pin or a general GPIO ------------------ -------------------------"
- note removed: "ECS-3225SMV-240-FP-TR"
- note removed: "If a fourth VCAP pin is available on the package, it must be connected to the other VCAP pins, but no additional capacitor is required."
- note removed: "VBAT: optional external power supply for backup domain"
- moved on the sheet: C102, C105, C111, C115

Commit message: Pin typo fix
Connections:
- net PA4_I2S3_WS renamed PA4_I2S1_WS
- net PA4_I2S3_WS_R renamed PA4_I2S1_WS_R
Changed lines of the file:
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@@
 		)
 	)
-	(label "PA4_I2S3_WS_R"
+	(label "PA4_I2S1_WS_R"
 		(at 137.16 200.66 0)
 		(fields_autoplaced yes)
@@
 		)
 	)
-	(label "PA4_I2S3_WS"
+	(label "PA4_I2S1_WS"
 		(at 68.58 207.01 0)
 		(fields_autoplaced yes)
@@
 		)
 	)
-	(hierarchical_label "PA4_I2S3_WS"
+	(hierarchical_label "PA4_I2S1_WS"
 		(shape output)
 		(at 68.58 207.01 180)

Commit message: Update
Other:
- note removed: "Direct SMPS supply (LDO off)"
- note removed: "The external Octo and HexaSPI power supply (VDDXSPI1, VDDXSPI2) is 1.8 V"
- note removed: "VCAP: digital core domain supply"
- note removed: "VDD33USB: USB regulator supply output for USB interface"
- note removed: "VDD50USB: external power supply for USB regulator"
- note removed: "VDD: external power supply for I/Os and system analog blocks such as reset, power management and oscillators"
- note removed: "VDDA: external analog power supply for ADCs and voltage reference buffers"
- note removed: "VDDLDO: external power supply for voltage regulator"
- note removed: "VDDSMPS: external power supply for the SMPS step-down converter"
- note removed: "VFBSMPS: step-down converter sense feedback"
- note removed: "VLXSMPS: step-down converter supply output"
- note removed: "VREF+: external reference voltage for ADC."
- note removed: "VSS: common ground for all supplies except for step-down converter and analog peripherals"
- note removed: "VSSA: separate analog and reference voltage ground"
- note removed: "VSSSMPS: separate step-down converter ground"
- note removed: "enabled by USBREGEN bit in the PWR control register 2 (PWR_CSR2),"
- company: (none) -> Peter Hancak
- title: (none) -> STM32H7S3 Board
Changed lines of the file:
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@@
 	(generator_version "8.0")
 	(paper "A3")
+	(title_block
+		(title "STM32H7S3 Board")
+		(date "2026-03-17")
+		(rev "B")
+		(company "Peter Hancak")
+	)
 	(junction
 		(at 337.82 127)
@@
 		)
 	)
-	(text "VDD50USB: external power supply for USB regulator"
-		(exclude_from_sim no)
-		(at 254 113.03 90)
-		(effects
-			(font
-				(size 1 1)
-			)
-		)
-	)
-	(text "VDDA: external analog power supply \nfor ADCs and voltage reference buffers"
-		(exclude_from_sim no)
-		(at 181.61 184.15 0)
-		(effects
-			(font
-				(size 1 1)
-			)
-		)
-	)
 	(text "PH1-OSC_OUT pin must be left HI-Z"
 		(exclude_from_sim no)
@@
 		)
 	)
-	(text "VSSSMPS: separate step-down converter ground"
-		(exclude_from_sim no)
-		(at 189.23 127 0)
-		(effects
-			(font
-				(size 1 1)
-			)
-		)
-	)
 	(text "600Ohm at 100MHz"
 		(exclude_from_sim no)
@@
 		)
 	)
-	(text "VDD33USB: USB regulator supply output for USB interface"
-		(exclude_from_sim no)
-		(at 251.46 115.57 90)
-		(effects
-			(font
-				(size 1 1)
-			)
-		)
-	)
-	(text "The external Octo and HexaSPI \npower supply (VDDXSPI1, VDDXSPI2) \nis 1.8 V"
-		(exclude_from_sim no)
-		(at 299.466 246.888 0)
-		(effects
-			(font
-				(size 1 1)
-			)
-			(justify left)
-		)
-	)
-	(text "VREF+: external reference voltage for ADC."
-		(exclude_from_sim no)
-		(at 184.15 177.8 0)
-		(effects
-			(font
-				(size 1 1)
-			)
-		)
-	)
 	(text "OSC32_OUT pin must be left HI-Z"
 		(exclude_from_sim no)
@@
 		)
 	)
-	(text "VDDLDO: external power supply for voltage regulator"
-		(exclude_from_sim no)
-		(at 180.34 110.49 90)
-		(effects
-			(font
-				(size 1 1)
-			)
-		)
-	)
-	(text "enabled by USBREGEN bit in the PWR \ncontrol register 2 (PWR_CSR2),"
-		(exclude_from_sim no)
-		(at 295.148 19.812 0)
-		(effects
-			(font
-				(size 1 1)
-			)
-		)
-	)
-	(text "VLXSMPS: step-down converter supply output"
-		(exclude_from_sim no)
-		(at 186.69 129.54 0)
-		(effects
-			(font
-				(size 1 1)
-			)
-		)
-	)
 	(text "PIN1 NC = Oscillation"
 		(exclude_from_sim no)
@@
 		)
 	)
-	(text "VDDSMPS: external power supply for the SMPS step-down converter"
-		(exclude_from_sim no)
-		(at 195.58 132.08 0)
-		(effects
-			(font
-				(size 1 1)
-			)
-		)
-	)
-	(text "VCAP: digital core domain supply"
-		(exclude_from_sim no)
-		(at 187.96 101.6 90)
-		(effects
-			(font
-				(size 1 1)
-			)
-		)
-	)
-	(text "VSSA: separate analog and reference voltage ground"
-		(exclude_from_sim no)
-		(at 186.69 175.26 0)
-		(effects
-			(font
-				(size 1 1)
-			)
-		)
-	)
-	(text "Direct SMPS supply (LDO off)"
-		(exclude_from_sim no)
-		(at 372.11 194.31 0)
-		(effects
-			(font
-				(size 1 1)
-			)
-			(justify left)
-		)
-	)
-	(text "VSS: common ground for all supplies except \nfor step-down converter and analog\nperipherals"
-		(exclude_from_sim no)
-		(at 248.92 184.15 0)
-		(effects
-			(font
-				(size 1 1)
-			)
-		)
-	)
-	(text "VDD: external power supply for I/Os and \nsystem analog blocks such as reset, power\nmanagement and oscillators"
-		(exclude_from_sim no)
-		(at 187.96 163.83 0)
-		(effects
-			(font
-				(size 1 1)
-			)
-		)
-	)
 	(text "VDDxspi1,VDDxspi2: external power supply for \ndedicated I/Os (Octo SPI and Hexa Deca\nSPI memories)"
 		(exclude_from_sim no)
@@
 		(effects
 			(font
-				(size 1 1)
-			)
-		)
-	)
-	(text "VFBSMPS: step-down converter sense feedback"
-		(exclude_from_sim no)
-		(at 187.96 134.62 0)
-		(effects
-			(font
