File: STM32H7_Board.kicad_sch (KiCad schematic)
At the start: 0 parts

Commit message: Update
Connections:
- no-connect marks 1 -> 13
Other:
- sheet Camera_SDCard_Interface renamed Camera_Interface
- sheet Camera_Interface ports: added none; removed SDMMC1_CK, SDMMC1_CKIN, SDMMC1_CMD, SDMMC1_D0, SDMMC1_D1, SDMMC1_D2, SDMMC1_D3
- sheet Interface_Headers ports: added I/O_HDR0, I/O_HDR1, I/O_HDR2, I/O_HDR3, I/O_HDR4, I/O_HDR5, I/O_HDR6, I/O_HDR7, I/O_HDR8, I/O_HDR9, RST_BTN, SDMMC1_CK, SDMMC1_CMD, SDMMC1_D0, SDMMC1_D1, SDMMC1_D2, SDMMC1_D3, USR_BTN; removed QSPI_CLK, QSPI_CS0, QSPI_IO0, QSPI_IO1, QSPI_IO2, QSPI_IO3
- sheet Power_Management ports: added RST_PWR; removed none
- sheet STM32H7S3I8T6 ports: added PM11, PM12, PO0, PO4, PP0, PP1, PP2, PP3; removed PO0_XSPIM_P1_NCS1, PO4_XSPIM_P1_CLK, PP0_XSPIM_P1_IO0, PP1_XSPIM_P1_IO1, PP2_XSPIM_P1_IO2, PP3_XSPIM_P1_IO3, USB_OTG_FS_DM, USB_OTG_FS_DP

Commit message: Update
Other:
- sheet Interface_Headers ports: added USB_DI_D2+, USB_DI_D2-; removed USB_D2+_DI, USB_D2-_DI

Commit message: Update
Other:
- sheet Interface_Headers ports: added QSPI_CLK, QSPI_CS, QSPI_D0, QSPI_D1, QSPI_D2, QSPI_D3; removed SDMMC1_CK, SDMMC1_CMD, SDMMC1_D0, SDMMC1_D1, SDMMC1_D2, SDMMC1_D3
- sheet STM32H7S3I8T6 ports: added PA13_DEBUG_JTMS-SWDIO, PA14_DEBUG_JTCK-SWCLK, PA15_I2S6_WS, PA4_I2S1_WS, PA5_I2S1_CK, PA7_FMC_INT, PB0_GFXTIM_TE, PB10_I2C2_SCL, PB11_I2C2_SDA, PB12_SPI2_NSS, PB13_SPI2_SCK, PB14_SPI2_MISO, PB15_SPI2_MOSI, PB3_DEBUG_JTDO-SWO, PB5_I2S6_SDO, PB6_UART5_TX, PB8_I2C1_SCL, PC10, PC11, PC12_I2S6_CK, PD13, PD2, PF11_ADC1_INP2, PF7_UART7_TX, PF8_DCMIPP_PIXCLK, PF9_TIM14_CH1, PM0_UCPD1_CC1, PM14, PM1_UCPD1_CC2, PO0_XSPIM_P1_NCS1, PO4_XSPIM_P1_CLK, PP0_XSPIM_P1_IO0, PP1_XSPIM_P1_IO1, PP2_XSPIM_P1_IO2, PP3_XSPIM_P1_IO3; removed DCMIPP_PIXCLK, FMC_INT, PA13_SWDIO, PA14_SWCLK, PA15_I2S1_WS, PA4_I2S6_WS, PA5_I2S6_CK, PA7_I2S6_SDO, PB0_I2S1_CK, PB13_UART5_TX/RX, PB14_USART1_TX/RX, PB15, PB3_SWO, PB5, PB6_I2C1_SCL, PE2, PF11, PF7_SPI5_SCK, PF9_SPI5_MOSI, PM0, PM1, PM14_SPI5_MISO, PO0, PO4, PP0, PP1, PP2, PP3, SDMMC1_CK, SDMMC1_CKIN, SDMMC1_CMD, SDMMC1_D0, SDMMC1_D1, SDMMC1_D2, SDMMC1_D3

Commit message: Update
Connections:
- no-connect marks 13 -> 14
Other:
- sheet Camera_Interface ports: added none; removed DCMIPP_D0, DCMIPP_D1
- sheet Power_Management ports: added none; removed PONKEYN
- sheet STM32H7S3I8T6 ports: added BOOT0, PA4_I2S3_WS, PA5, PB4, PC10_I2S3_CK, PC11_I2S3_SDI, PD12, PD15, PD6_FMC_NE3, PF4; removed DCMIPP_D9, FMC_NE1, PA4_I2S1_WS, PA5_I2S1_CK, PB4_I2S1_SDI, PC10, PC11, PD6, PF4_DCMIPP_D8
- note added: "FMC Bus length matching within ±150 mil (3.8 mm) across the entire bus"
- note added: "Length Match"

Commit message: Update
Connections:
- no-connect marks 14 -> 16
Other:
- sheet Camera_Interface ports: added CAM_PWDN, HSYNC, PCLK, VSYNC, Y2, Y3, Y4, Y5, Y6, Y7, Y8, Y9; removed DCMIPP_D2, DCMIPP_D3, DCMIPP_D4, DCMIPP_D5, DCMIPP_D6, DCMIPP_D7, DCMIPP_D8, DCMIPP_D9, DCMIPP_HSYNC, DCMIPP_PIXCLK, DCMIPP_VSYNC, PWDN
Changed lines of the file:
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@@
 	)
 	(junction
-		(at 297.18 198.12)
-		(diameter 0)
-		(color 0 0 0 0)
-	)
-	(junction
 		(at 292.1 107.95)
 		(diameter 0)
@@
 	)
 	(no_connect
+		(at 245.11 68.58)
+	)
+	(no_connect
 		(at 245.11 213.36)
 	)
@@
 	)
 	(no_connect
+		(at 317.5 68.58)
+	)
+	(no_connect
 		(at 245.11 215.9)
 	)
@@
 		)
 	)
-	(wire
-		(pts
-			(xy 297.18 63.5) (xy 297.18 198.12)
-		)
-		(stroke
-			(width 0)
-			(type default)
-		)
-	)
 	(bus
 		(pts
@@
 	(wire
 		(pts
-			(xy 297.18 63.5) (xy 317.5 63.5)
-		)
-		(stroke
-			(width 0)
-			(type default)
-		)
-	)
-	(wire
-		(pts
 			(xy 245.11 58.42) (xy 317.5 58.42)
 		)
@@
 	(wire
 		(pts
-			(xy 245.11 243.84) (xy 274.32 243.84)
-		)
-		(stroke
-			(width 0)
-			(type default)
-		)
-	)
-	(wire
-		(pts
 			(xy 245.11 160.02) (xy 264.16 160.02)
 		)
@@
 		)
 	)
-	(wire
-		(pts
-			(xy 245.11 68.58) (xy 317.5 68.58)
-		)
-		(stroke
-			(width 0)
-			(type default)
-		)
-	)
 	(bus
 		(pts
@@
 		)
 	)
-	(wire
-		(pts
-			(xy 245.11 177.8) (xy 317.5 177.8)
-		)
-		(stroke
-			(width 0)
-			(type default)
-		)
-	)
 	(bus
 		(pts
@@
 		)
 	)
-	(wire
-		(pts
-			(xy 245.11 246.38) (xy 276.86 246.38)
-		)
-		(stroke
-			(width 0)
-			(type default)
-		)
-	)
 	(bus
 		(pts
@@
 	(wire
 		(pts
+			(xy 245.11 177.8) (xy 317.5 177.8)
+		)
+		(stroke
+			(width 0)
+			(type default)
+		)
+	)
+	(wire
+		(pts
 			(xy 190.5 81.28) (xy 179.07 81.28)
 		)
@@
 	(wire
 		(pts
+			(xy 245.11 63.5) (xy 317.5 63.5)
+		)
+		(stroke
+			(width 0)
+			(type default)
+		)
+	)
+	(wire
+		(pts
 			(xy 302.26 157.48) (xy 317.5 157.48)
 		)
@@
 		)
 	)
+	(wire
+		(pts
+			(xy 245.11 243.84) (xy 274.32 243.84)
+		)
+		(stroke
+			(width 0)
+			(type default)
+		)
+	)
 	(bus
 		(pts
@@
 		)
 	)
+	(wire
+		(pts
+			(xy 245.11 246.38) (xy 276.86 246.38)
+		)
+		(stroke
+			(width 0)
+			(type default)
+		)
+	)
 	(bus
 		(pts
@@
 		)
 	)
+	(text_box "NOTES:\n- Camera RST connected to MCU GPIO PA5 43\n- MCU RST connected to STPMIC1\n- STPIMIC1 activates RST\n- STPMIC1 has own powerdown button "
+		(exclude_from_sim no)
+		(at 62.865 259.08 0)
+		(size 69.85 26.035)
+		(stroke
+			(width 0)
+			(type dash)
+		)
+		(fill
+			(type none)
+		)
+		(effects
+			(font
+				(size 1 1)
+			)
+			(justify left top)
+		)
+	)
 	(text_box "NOTES:\nVoltages: 5, 3.3, 2.8, 1.8, 1.5V\n\n1. Micro USB B because the PCB will not be\nfunctioning as a host (no external drive)\nMatched Net Lengths [Tolerance = 2mm]\nImpedance Constraint [Min = 85.00 Max = 95.00 ]\n\nTypical Current Consumption (based on ST's data sheets):\n- Run Mode (Vcore = 1.15V, 480 MHz):\n  Approximately 260-300 mA at full speed with all peripherals enabled.\n- Low Power Run (LP mode, 24 MHz, Vcore = 0.9V):\n  Typically around 15-20 mA.\n- Standby Mode (RTC enabled, backup RAM powered):\n   1-2 µA, depending on the specific settings.\n\nCamera Connection\n- The camera is based on 2.8V I/O voltage\n- This should still work with 3.3V based MCU (3.3V * 0.7 = 2.31<2.8)\n- The pins on the camera could be damaged by the 3.3V\n  (STM32 used these voltage levels in their design)\n\nDisplay Interface\n1. NOR Flash Mode (Recommended)\n✅ Best choice for parallel LCDs with built-in controllers.\n✅ Supports direct memory-mapped access (write commands and data directly).\n✅ Fast random access (suitable for sending commands/pixels).\n❌ Not for framebuffers (use external SDRAM for full-screen buffering).\n🔹 Use NOR mode if your display requires an 8080/6800 bus (e.g., ILI9341, SSD1963).\n\n📌 Setup Example:\n\nMemory Type: NOR\nMemory Width: 8-bit or 16-bit\nChip Select (NE1, NE2, etc.): Connect to LCD\nTiming Configuration: Match LCD controller's datasheet"
 		(exclude_from_sim no)
@@
 	(text "Length Match"
 		(exclude_from_sim no)
-		(at 281.432 44.196 0)
+		(at 281.94 44.45 0)
 		(effects
 			(font
@@
 			)
 		)
-		(pin "DCMIPP_PIXCLK" bidirectional
-			(at 317.5 55.88 180)
+		(pin "CAMERA_SCL" bidirectional
+			(at 317.5 76.2 180)
 			(effects
 				(font
@@
 			)
 		)
-		(pin "DCMIPP_D3" bidirectional
-			(at 317.5 30.48 180)
+		(pin "RESETB" bidirectional
+			(at 317.5 63.5 180)
 			(effects
 				(font
@@
 			)
 		)
-		(pin "DCMIPP_D5" bidirectional
-			(at 317.5 35.56 180)
+		(pin "CAMERA_SDA" bidirectional
+			(at 317.5 73.66 180)
 			(effects
 				(font
@@
 			)
 		)
-		(pin "PWDN" bidirectional
-			(at 317.5 66.04 180)
+		(pin "STROBE" bidirectional
+			(at 317.5 68.58 180)
 			(effects
 				(font
@@
 			)
 		)
-		(pin "DCMIPP_D4" bidirectional
-			(at 317.5 33.02 180)
+		(pin "Y7" bidirectional
+			(at 317.5 40.64 180)
 			(effects
 				(font
@@
 			)
 		)
-		(pin "DCMIPP_D2" bidirectional
-			(at 317.5 27.94 180)
+		(pin "Y8" bidirectional
+			(at 317.5 43.18 180)
 			(effects
 				(font
@@
 			)
 		)
-		(pin "DCMIPP_D6" bidirectional
-			(at 317.5 38.1 180)
+		(pin "HSYNC" bidirectional
+			(at 317.5 58.42 180)
 			(effects
 				(font
@@
 			)
 		)
-		(pin "DCMIPP_D7" bidirectional
-			(at 317.5 40.64 180)
+		(pin "VSYNC" bidirectional
+			(at 317.5 60.96 180)
 			(effects
 				(font
@@
 			)
 		)
-		(pin "DCMIPP_D8" bidirectional
-			(at 317.5 43.18 180)
+		(pin "CAM_PWDN" bidirectional
+			(at 317.5 66.04 180)
 			(effects
 				(font
@@
 			)
 		)
-		(pin "DCMIPP_D9" bidirectional
+		(pin "Y9" bidirectional
 			(at 317.5 45.72 180)
 			(effects
@@
 			)
 		)
-		(pin "CAMERA_SCL" bidirectional
-			(at 317.5 76.2 180)
+		(pin "Y6" bidirectional
+			(at 317.5 38.1 180)
 			(effects
 				(font
@@
 			)
 		)
-		(pin "RESETB" bidirectional
-			(at 317.5 63.5 180)
+		(pin "Y5" bidirectional
+			(at 317.5 35.56 180)
 			(effects
 				(font
@@
 			)
 		)
-		(pin "DCMIPP_HSYNC" bidirectional
-			(at 317.5 58.42 180)
+		(pin "PCLK" bidirectional
+			(at 317.5 55.88 180)
 			(effects
 				(font
@@
 			)
 		)
-		(pin "DCMIPP_VSYNC" bidirectional
-			(at 317.5 60.96 180)
+		(pin "Y2" bidirectional
+			(at 317.5 27.94 180)
 			(effects
 				(font
@@
 			)
 		)
-		(pin "CAMERA_SDA" bidirectional
-			(at 317.5 73.66 180)
+		(pin "Y3" bidirectional
+			(at 317.5 30.48 180)
 			(effects
 				(font
@@
 			)
 		)
-		(pin "STROBE" bidirectional
-			(at 317.5 68.58 180)
+		(pin "Y4" bidirectional
+			(at 317.5 33.02 180)
 			(effects
 				(font
@@
 		)
 		(pin "PA5" bidirectional
-			(at 245.11 177.8 0)
+			(at 245.11 63.5 0)
 			(effects
 				(font
@@
 		)
 		(pin "BOOT0" input
-			(at 245.11 140.97 0)
+			(at 245.11 177.8 0)
 			(effects
 				(font

Commit message: Update
Connections:
- no-connect marks 16 -> 19
Other:
- sheet Interface_Headers ports: added BTB1, BTB2, BTB20, BTB21, BTB22, BTB23, BTB24, BTB25, BTB26, BTB27, BTB28, BTB29, BTB3, BTB30, BTB4, BTB5, BTB6; removed I2C_SCL_HDR, I2C_SDA_HDR, I2S1_CK, I2S1_MCK, I2S1_SDI/O, I2S1_WS, I2S2_CK, I2S2_MCK, I2S2_SDI/O, I2S2_WS, I/O_HDR0, I/O_HDR1, I/O_HDR2, I/O_HDR3, I/O_HDR4, I/O_HDR5, I/O_HDR6, I/O_HDR7, I/O_HDR8, I/O_HDR9, QSPI_CLK, QSPI_CS, QSPI_D0, QSPI_D1, QSPI_D2, QSPI_D3, SPI_CLK, SPI_CS, SPI_MISO, SPI_MOSI, UART1_TX/RX, UART2_TX/RX

Commit message: Update
Connections:
- no-connect marks 19 -> 17
Other:
- sheet Memory ports: added NAND_ALE, NAND_CE#, NAND_CLE, NAND_D0, NAND_D1, NAND_D2, NAND_D3, NAND_D4, NAND_D5, NAND_D6, NAND_D7, NAND_RE#, NAND_R/B#, NAND_WE#, NAND_WP#, SRAM_A0, SRAM_A1, SRAM_A10, SRAM_A11, SRAM_A12, SRAM_A13, SRAM_A14, SRAM_A2, SRAM_A3, SRAM_A4, SRAM_A5, SRAM_A6, SRAM_A7, SRAM_A8, SRAM_A9, SRAM_CS#, SRAM_D0, SRAM_D1, SRAM_D2, SRAM_D3, SRAM_D4, SRAM_D5, SRAM_D6, SRAM_D7, SRAM_OE#, SRAM_WE#; removed FMC_A0, FMC_A1, FMC_A10, FMC_A11, FMC_A12, FMC_A2, FMC_A3, FMC_A4, FMC_A5, FMC_A6, FMC_A7, FMC_A8, FMC_A9, FMC_ALE, FMC_BA0, FMC_BA1, FMC_CLE, FMC_D0, FMC_D1, FMC_D10, FMC_D11, FMC_D12, FMC_D13, FMC_D14, FMC_D15, FMC_D2, FMC_D3, FMC_D4, FMC_D5, FMC_D6, FMC_D7, FMC_D8, FMC_D9, FMC_INT, FMC_NBL0, FMC_NBL1, FMC_NCE, FMC_NOE, FMC_NWE, FMC_SDCKE0, FMC_SDCLK, FMC_SDNCAS, FMC_SDNE0, FMC_SDNRAS, FMC_SDNWE
- sheet STM32H7S3I8T6 ports: added FMC_A13, FMC_A14, PB7, PC0, PD12_FMC_NE1, PD8, PD9, PE10, PE11, PE12, PE13, PE14, PE15; removed FMC_BA0, FMC_BA1, FMC_NBL0, FMC_NBL1, FMC_SDCKE0, FMC_SDCLK, FMC_SDNCAS, FMC_SDNE0, FMC_SDNRAS, FMC_SDNWE, PB4, PD12, PF4

Commit message: Update
Other:
- sheet Memory ports: added SDRAM_A0, SDRAM_A1, SDRAM_A10, SDRAM_A11, SDRAM_A12, SDRAM_A2, SDRAM_A3, SDRAM_A4, SDRAM_A5, SDRAM_A6, SDRAM_A7, SDRAM_A8, SDRAM_A9, SDRAM_BA0, SDRAM_BA1, SDRAM_CKE, SDRAM_CLK, SDRAM_DQ0, SDRAM_DQ1, SDRAM_DQ2, SDRAM_DQ3, SDRAM_DQ4, SDRAM_DQ5, SDRAM_DQ6, SDRAM_DQ7, SDRAM_DQMH, SDRAM_~{CAS}, SDRAM_~{CS}, SDRAM_~{RAS}, SDRAM_~{WE}; removed SRAM_A0, SRAM_A1, SRAM_A10, SRAM_A11, SRAM_A12, SRAM_A13, SRAM_A14, SRAM_A2, SRAM_A3, SRAM_A4, SRAM_A5, SRAM_A6, SRAM_A7, SRAM_A8, SRAM_A9, SRAM_CS#, SRAM_D0, SRAM_D1, SRAM_D2, SRAM_D3, SRAM_D4, SRAM_D5, SRAM_D6, SRAM_D7, SRAM_OE#, SRAM_WE#
