File: STM32H7_Board.kicad_sch (KiCad schematic)
At the start: 0 parts

Commit message: Update
Changed lines of the file:
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@@
 		)
 		(property "Value" "SMPS_OUT2_3V3+"
-			(at 294.894 153.162 0)
+			(at 302.26 157.734 90)
 			(effects
 				(font
