File: STM32H7_Board.kicad_sch (KiCad schematic)
At the start: 0 parts

Commit message: Update
Other:
- added sheet Notes (Notes.kicad_sch)
- sheet Power_Management ports: added RST_LOCAL; removed RST_PWR
