File: LCD_Camera_Interface.kicad_sch (KiCad schematic)
At the start: 15 parts, among them J1 SD_Molex_502570-0893, J27 Molex-52437-2471, J28 Camera_STROBE, J32 1.5V_Option_Header

Commit message: Update
Parts:
- removed C6: 100n, Capacitor_SMD:C_0805_2012Metric, symbol Device:C
- removed C8: 1u, Capacitor_SMD:C_0805_2012Metric, symbol Device:C
- removed EMI1: EMI_EMIF06-MSD02N16, Personal_Project:EMI_EMIF06MSD02N16, symbol Personal_Projects:EMI_EMIF06-MSD02N16
- removed J1: SD_Molex_502570-0893, Personal_Project:SD_Molex_502570-0893, symbol Personal_Projects:SD_Molex_502570-0893
- removed R5: 10k, Resistor_SMD:R_0805_2012Metric_Pad1.20x1.40mm_HandSolder, symbol Device:R
- removed R8: 100R, Resistor_SMD:R_0805_2012Metric_Pad1.20x1.40mm_HandSolder, symbol Device:R
- added H1, H2, H3, H4: MountingHole_Pad, MountingHole:MountingHole_3.2mm_M3_Pad, symbol Mechanical:MountingHole_Pad
- R7: footprint Resistor_SMD:R_0805_2012Metric_Pad1.20x1.40mm_HandSolder -> Resistor_SMD:R_0805_2012Metric_1
Connections:
- net GND: now also H1.1, H2.1, H3.1, H4.1
- no-connect marks 6 -> 1
Other:
- note removed: "DET Card detection pin Decided to use only ESD protection diode with the voltage decreasing on the MCU down to 1.8V at card detection. ESD protection should have less than 1pF to be used at high speed."
- note removed: "SDMMC1_CKIN signal not used - To be used in combination with level translator"
- note removed: "To be optionally adjusted to 1V8"
- moved on the sheet: C27, C29, C35, FB3, J27, J28, J32, OS1, R7

Commit message: Update
Connections:
- net 2V8_LD5+ renamed 2V8_BK3+
Changed lines of the file:
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@@
 			)
 		)
-		(property "Value" "2V8_LD5+"
+		(property "Value" "2V8_BK3+"
 			(at 269.24 96.266 0)
 			(effects
@@
 			)
 		)
-		(property "Value" "2V8_LD5+"
+		(property "Value" "2V8_BK3+"
 			(at 299.72 117.856 0)
 			(effects
@@
 			)
 		)
-		(property "Value" "2V8_LD5+"
+		(property "Value" "2V8_BK3+"
 			(at 295.91 144.526 0)
 			(effects

Commit message: Update
Parts:
- removed J28: Camera_STROBE, Connector_PinHeader_2.54mm:PinHeader_1x02_P2.54mm_Vertical, symbol Connector_Generic:Conn_01x02
- removed J32: 1.5V_Option_Header, Connector_PinHeader_2.54mm:PinHeader_1x02_P2.54mm_Vertical, symbol Connector_Generic:Conn_01x02
- added R8, R9: 2k2, Resistor_SMD:R_0805_2012Metric, symbol Device:R
- added RN11, RN12, RN13: 33R, Resistor_SMD:R_Array_Convex_4x0402, symbol Device:R_Pack04
Connections:
- net DVDD is gone; now on net 1V5_BK2+: J27.10
- net STROBE_J is gone; now on net STROBE: J27.1
- net 2V8_BK3+: now also R8.1, R9.1
- net CAMERA_SCL: now also R9.2
- net CAMERA_SDA: now also R8.2
- net DCMIPP_D2: now also RN11.8 (R1.2); no longer J27.19
- net DCMIPP_D3: now also RN11.6 (R3.2); no longer J27.21
- net DCMIPP_D4: now also RN11.5 (R4.2); no longer J27.22
- net DCMIPP_D5: now also RN11.7 (R2.2); no longer J27.20
- net DCMIPP_D6: now also RN12.5 (R4.2); no longer J27.18
- net DCMIPP_D7: now also RN12.2 (R2.1), RN12.7 (R2.2)
- net DCMIPP_D8: now also RN12.1 (R1.1), RN12.8 (R1.2)
- net DCMIPP_HSYNC: now also RN13.5 (R4.2); no longer J27.9
- net DCMIPP_PIXCLK: now also RN12.6 (R3.2); no longer J27.17
- net DCMIPP_VSYNC: now also RN13.7 (R2.2); no longer J27.7
- net PWDN: now also RN13.6 (R3.2); no longer J27.8
- net DCMIPP_D0: no longer names the net of J27.24
- net DCMIPP_D1: no longer names the net of J27.23
- new net DCMIPP_D2_R: J27.19, RN11.1 (R1.1)
- new net DCMIPP_D3_R: J27.21, RN11.3 (R3.1)
- new net DCMIPP_D4_R: J27.22, RN11.4 (R4.1)
- new net DCMIPP_D5_R: J27.20, RN11.2 (R2.1)
- new net DCMIPP_D6_R: J27.18, RN12.4 (R4.1)
- new net DCMIPP_HSYNC_R: J27.9, RN13.4 (R4.1)
- new net DCMIPP_PIXCLK_R: J27.17, RN12.3 (R3.1)
- new net DCMIPP_VSYNC_R: J27.7, RN13.2 (R2.1)
- new net PWDN_R: J27.8, RN13.3 (R3.1)
- no-connect marks 1 -> 5
Other:
- moved on the sheet: C27, C29, C35, FB3, J27, OS1, R7

Commit message: Update
Parts:
- removed R7: 0R, Resistor_SMD:R_0805_2012Metric_1, symbol Device:R
- added C6: 100n, Capacitor_SMD:C_0603_1608Metric, symbol Device:C
- added R3, R4: 33R, Resistor_SMD:R_0603_1608Metric, symbol Device:R
Connections:
- net GND: now also C6.2
- net RESETB: now also C6.1
- net XCLK: now also R4.1
- net at OS1.3 (OUTPUT): now also R4.2
- net DCMIPP_D2 renamed Y2
- net DCMIPP_D2_R renamed Y2_R
- net DCMIPP_D3 renamed Y3
- net DCMIPP_D3_R renamed Y3_R
- net DCMIPP_D4 renamed Y4
- net DCMIPP_D4_R renamed Y4_R
- net DCMIPP_D5 renamed Y5
- net DCMIPP_D5_R renamed Y5_R
- net DCMIPP_D6 renamed Y6
- net DCMIPP_D6_R renamed Y6_R
- net DCMIPP_D7 renamed Y7_R
- net Y7_R: no longer RN12.7 (R2.2)
- net DCMIPP_D8 renamed Y8_R
- net Y8_R: no longer RN12.8 (R1.2)
- net DCMIPP_D9 renamed Y9_R
- net Y9_R: now also R3.1
- net DCMIPP_HSYNC renamed HSYNC
- net DCMIPP_HSYNC_R renamed HSYNC_R
- net DCMIPP_PIXCLK renamed PCLK
- net DCMIPP_PIXCLK_R renamed PCLK_R
- net DCMIPP_VSYNC renamed VSYNC
- net DCMIPP_VSYNC_R renamed VSYNC_R
- net PWDN renamed CAM_PWDN
- net PWDN_R renamed CAM_PWDN_R
- new net Y7: RN12.7 (R2.2)
- new net Y8: RN12.8 (R1.2)
- new net Y9: R3.2

Commit message: Update
Parts:
- removed H1, H2, H3, H4: MountingHole_Pad, MountingHole:MountingHole_3.2mm_M3_Pad, symbol Mechanical:MountingHole_Pad
