File: Interface_Headers.kicad_sch (KiCad schematic)
At the start: 36 parts, among them J10 SWDB, J11 UART1_HDR, J22 USB_C_Receptacle_USB2.0_16P, J3 UART2_HDR, J7 I2C1_Headers, J9 User Button Jumper, U7 USBLC6-2SC6

Commit message: Update
Parts:
- removed H5, H6, H7, H8: MountingHole_Pad, MountingHole:MountingHole_3.2mm_M3_Pad, symbol Mechanical:MountingHole_Pad
- added J4: I/O_HDR1, Connector_PinHeader_2.54mm:PinHeader_2x10_P2.54mm_Horizontal, symbol Connector_Generic:Conn_02x10_Odd_Even
Connections:
- net GND: now also J4.1 (Pin_1), J4.11 (Pin_11), J4.13 (Pin_13), J4.15 (Pin_15), J4.17 (Pin_17), J4.19 (Pin_19), J4.3 (Pin_3), J4.5 (Pin_5), J4.7 (Pin_7), J4.9 (Pin_9)
- net +3.3V renamed 3V3_BK4+
- net QSPI_CLK renamed SDMMC1_CK
- net QSPI_CS0 renamed SDMMC1_CMD
- net QSPI_IO0 renamed SDMMC1_D0
- net QSPI_IO1 renamed SDMMC1_D1
- net QSPI_IO2 renamed SDMMC1_D2
- net QSPI_IO3 renamed SDMMC1_D3
- new net I/O_HDR0: J4.2 (Pin_2)
- new net I/O_HDR1: J4.4 (Pin_4)
- new net I/O_HDR2: J4.6 (Pin_6)
- new net I/O_HDR3: J4.8 (Pin_8)
- new net I/O_HDR4: J4.10 (Pin_10)
- new net I/O_HDR5: J4.12 (Pin_12)
- new net I/O_HDR6: J4.14 (Pin_14)
- new net I/O_HDR7: J4.16 (Pin_16)
- new net I/O_HDR8: J4.18 (Pin_18)
- new net I/O_HDR9: J4.20 (Pin_20)
Other:
- note added: "USB HS Matched Net Lengths [Tolerance = 2mm] Impedance Constraint 90 Ohm [Min = 85.00 Max = 95.00 ]"
- note removed: "------Maybe add diode on the 5V power"
- note removed: "Matched Net Lengths [Tolerance = 2mm] Impedance Constraint [Min = 85.00 Max = 95.00 ]"

Commit message: Update
Parts:
- removed J9: User Button Jumper, Connector_PinHeader_2.54mm:PinHeader_1x02_P2.54mm_Vertical, symbol Connector_Generic:Conn_01x02
- J11, J3, J7: footprint Connector_PinHeader_2.54mm:PinHeader_2x03_P2.54mm_Horizontal -> Personal_Project:PinHeader_2x03_P2.54mm_Horizontal_Court
Connections:
- net USR_BTN_J is gone; now on net USR_BTN: C65.2, U8.1, U8.2
- net USB_D2+: now also U7.6 (I/O1); no longer U7.4 (I/O2)
- net USB_D2-: now also U7.4 (I/O2); no longer U7.6 (I/O1)
- net USB_D2+_DI renamed USB_DI_D2-
- net USB_D2-_DI renamed USB_DI_D2+
Other:
- note removed: "Decide onn user button location ---------------"
- moved on the sheet: U7

Commit message: Update
Connections:
- net UART1_TX/RX_R: now reaches J11.3 (Pin_3), R4.2
- net UART2_TX/RX_R: now reaches J3.3 (Pin_3), R3.2
Other:
- moved on the sheet: R3, R4
Changed lines of the file:
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@@
 	(wire
 		(pts
-			(xy 327.66 53.34) (xy 309.88 53.34)
+			(xy 309.88 53.34) (xy 292.1 53.34)
 		)
 		(stroke
@@
 	(wire
 		(pts
-			(xy 335.28 80.01) (xy 344.17 80.01)
+			(xy 316.23 80.01) (xy 344.17 80.01)
 		)
 		(stroke
@@
 	(wire
 		(pts
-			(xy 327.66 80.01) (xy 309.88 80.01)
+			(xy 308.61 80.01) (xy 290.83 80.01)
 		)
 		(stroke
@@
 	(wire
 		(pts
-			(xy 335.28 53.34) (xy 344.17 53.34)
+			(xy 317.5 53.34) (xy 344.17 53.34)
 		)
 		(stroke
@@
 		)
 	)
+	(label "UART2_TX{slash}RX_R"
+		(at 322.58 80.01 0)
+		(fields_autoplaced yes)
+		(effects
+			(font
+				(size 1.27 1.27)
+			)
+			(justify left bottom)
+		)
+	)
 	(label "I{slash}O_HDR4"
 		(at 144.78 119.38 180)
@@
 		)
 	)
+	(label "UART1_TX{slash}RX_R"
+		(at 322.58 53.34 0)
+		(fields_autoplaced yes)
+		(effects
+			(font
+				(size 1.27 1.27)
+			)
+			(justify left bottom)
+		)
+	)
 	(label "USB_VBUS+"
 		(at 152.4 173.99 0)
@@
 	)
 	(label "UART2_TX{slash}RX"
-		(at 309.88 80.01 0)
+		(at 290.83 80.01 0)
 		(fields_autoplaced yes)
 		(effects
@@
 	)
 	(label "UART1_TX{slash}RX"
-		(at 309.88 53.34 0)
+		(at 292.1 53.34 0)
 		(fields_autoplaced yes)
 		(effects
@@
 	(hierarchical_label "UART1_TX{slash}RX"
 		(shape input)
-		(at 309.88 53.34 180)
+		(at 292.1 53.34 180)
 		(fields_autoplaced yes)
 		(effects
@@
 	(hierarchical_label "UART2_TX{slash}RX"
 		(shape input)
-		(at 309.88 80.01 180)
+		(at 290.83 80.01 180)
 		(fields_autoplaced yes)
 		(effects
@@
 	(symbol
 		(lib_id "Device:R")
-		(at 331.47 53.34 90)
+		(at 313.69 53.34 90)
 		(unit 1)
 		(exclude_from_sim no)
@@
 		(dnp no)
 		(property "Reference" "R4"
-			(at 326.644 52.324 90)
+			(at 308.864 52.324 90)
 			(effects
 				(font
@@
 		)
 		(property "Value" "33R"
-			(at 336.804 52.324 90)
+			(at 319.024 52.324 90)
 			(effects
 				(font
@@
 		)
 		(property "Footprint" "Resistor_SMD:R_0805_2012Metric"
-			(at 331.47 55.118 90)
+			(at 313.69 55.118 90)
 			(effects
 				(font
@@
 		)
 		(property "Datasheet" "~"
-			(at 331.47 53.34 0)
+			(at 313.69 53.34 0)
 			(effects
 				(font
@@
 		)
 		(property "Description" "Resistor"
-			(at 331.47 53.34 0)
+			(at 313.69 53.34 0)
 			(effects
 				(font
@@
 	(symbol
 		(lib_id "Device:R")
-		(at 331.47 80.01 90)
+		(at 312.42 80.01 90)
 		(unit 1)
 		(exclude_from_sim no)
@@
 		(dnp no)
 		(property "Reference" "R3"
-			(at 326.644 78.994 90)
+			(at 307.594 78.994 90)
 			(effects
 				(font
@@
 		)
 		(property "Value" "33R"
-			(at 336.804 78.994 90)
+			(at 317.754 78.994 90)
 			(effects
 				(font
@@
 		)
 		(property "Footprint" "Resistor_SMD:R_0805_2012Metric"
-			(at 331.47 81.788 90)
+			(at 312.42 81.788 90)
 			(effects
 				(font
@@
 		)
 		(property "Datasheet" "~"
-			(at 331.47 80.01 0)
+			(at 312.42 80.01 0)
 			(effects
 				(font
@@
 		)
 		(property "Description" "Resistor"
-			(at 331.47 80.01 0)
+			(at 312.42 80.01 0)
 			(effects
 				(font

Commit message: Update
Parts:
- removed C12, C26, C28, C31, C32, C56: 100n, Capacitor_SMD:C_0805_2012Metric, symbol Device:C
- removed C34: 4u7, Capacitor_SMD:C_0805_2012Metric, symbol Device:C
- removed FB2: 2508051217Y3 0805 (2012 Metric), Inductor_SMD:L_0805_2012Metric, symbol Device:FerriteBead
- removed FB4: Part # MI0805K601R-10, Capacitor_SMD:C_0805_2012Metric, symbol Device:FerriteBead
- added J1: BTB_10132798-062100LF, Personal_Project:BTB_AMPHENOL_10132798-062100LF, symbol Personal_Projects:BTB_10132798-062100LF
Connections:
- net SDMMC1_CK renamed QSPI_CLK
- net SDMMC1_CMD renamed QSPI_CS
- net SDMMC1_D0 renamed QSPI_D0
- net SDMMC1_D1 renamed QSPI_D1
- net SDMMC1_D2 renamed QSPI_D2
- net SDMMC1_D3 renamed QSPI_D3
Other:
- note removed: "600 Ohms @ 100 MHz"

Commit message: Update
Parts:
- removed DI1: Diode_PESD5V0U2BT-Q, Package_TO_SOT_SMD:SOT-23, symbol Personal_Projects:Diode_PESD5V0U2BT-Q
- removed FPC1: FPC_0545482072, Personal_Project:FPC_0545482072, symbol Personal_Projects:FPC_0545482072
- removed FPC2, FPC5, FPC6: FPC_0545481072, Personal_Project:FPC_0545481072, symbol Personal_Projects:FPC_0545481072
- removed J10: SWDB, Connector_PinHeader_2.54mm:PinHeader_2x04_P2.54mm_Horizontal, symbol Connector_Generic:Conn_02x04_Odd_Even
- removed J11: UART1_HDR, Personal_Project:PinHeader_2x03_P2.54mm_Horizontal_Court, symbol Connector_Generic:Conn_02x03_Odd_Even
- removed J3: UART2_HDR, Personal_Project:PinHeader_2x03_P2.54mm_Horizontal_Court, symbol Connector_Generic:Conn_02x03_Odd_Even
- removed J4: I/O_HDR1, Connector_PinHeader_2.54mm:PinHeader_2x10_P2.54mm_Horizontal, symbol Connector_Generic:Conn_02x10_Odd_Even
- removed J7: I2C1_Headers, Personal_Project:PinHeader_2x03_P2.54mm_Horizontal_Court, symbol Connector_Generic:Conn_02x03_Odd_Even
- removed R13, R2: 10k, Resistor_SMD:R_0805_2012Metric, symbol Device:R
- removed R3, R4: 33R, Resistor_SMD:R_0805_2012Metric, symbol Device:R
- added J3: SWDB, Connector_PinHeader_2.54mm:PinHeader_2x04_P2.54mm_Horizontal, symbol Connector_Generic:Conn_02x04_Odd_Even
Connections:
- net GND: now also J3.1 (Pin_1), J3.3 (Pin_3), J3.5 (Pin_5), J3.7 (Pin_7)
- net NRST: now also J3.6 (Pin_6)
- net SWCLK: now also J3.2 (Pin_2)
- net SWDIO: now also J3.8 (Pin_8)
- net SWO: now also J3.4 (Pin_4)
Other:
- note removed: "Place ESD close to the header"
- moved on the sheet: J1, J22, R15, R16, U7, Z3

Commit message: Update
Connections:
- net GND: now also J1.31, J1.32, J1.33, J1.34, J1.35, J1.36, J1.37, J1.38, J1.39, J1.40, J1.41, J1.42, J1.43, J1.44, J1.45, J1.46, J1.47, J1.48, J1.49, J1.50, J1.51, J1.52, J1.53, J1.54, J1.55, J1.56, J1.57, J1.58, J1.59, J1.60
- net BTB1: now reaches J1.1
- net BTB2: now reaches J1.2
- net BTB20: now reaches J1.20
- net BTB21: now reaches J1.21
- net BTB22: now reaches J1.22
- net BTB23: now reaches J1.23
- net BTB24: now reaches J1.24
- net BTB25: now reaches J1.25
- net BTB26: now reaches J1.26
- net BTB27: now reaches J1.27
- net BTB28: now reaches J1.28
- net BTB29: now reaches J1.29
- net BTB3: now reaches J1.3
- net BTB30: now reaches J1.30
- net BTB4: now reaches J1.4
- net BTB5: now reaches J1.5
- net BTB6: now reaches J1.6

Commit message: Update
Parts:
- added H1, H2, H3, H4: MountingHole_Pad, MountingHole:MountingHole_3.2mm_M3_Pad, symbol Mechanical:MountingHole_Pad
Connections:
- net GND: now also H1.1, H2.1, H3.1, H4.1; no longer J1.31, J1.32, J1.33, J1.34, J1.35, J1.36, J1.37, J1.38, J1.39, J1.40, J1.41, J1.42, J1.43, J1.44, J1.45, J1.46, J1.47, J1.48, J1.49, J1.50, J1.51, J1.52, J1.53, J1.54, J1.55, J1.56, J1.57, J1.58, J1.59, J1.60, J3.1 (Pin_1)
- net USB_VBUS+: now also J3.1 (Pin_1)
- net BTB10: now reaches J1.10
- net BTB11: now reaches J1.11
- net BTB12: now reaches J1.12
- net BTB13: now reaches J1.13
- net BTB14: now reaches J1.14
- net BTB15: now reaches J1.15
- net BTB16: now reaches J1.16
- net BTB17: now reaches J1.17
- net BTB18: now reaches J1.18
- net BTB19: now reaches J1.19
- net BTB7: now reaches J1.7
- net BTB8: now reaches J1.8
- net BTB9: now reaches J1.9
- new net BTB31: J1.60
- new net BTB32: J1.59
- new net BTB33: J1.58
- new net BTB34: J1.57
- new net BTB35: J1.56
- new net BTB36: J1.55
- new net BTB37: J1.54
- new net BTB38: J1.53
- new net BTB39: J1.52
- new net BTB40: J1.51
- new net BTB41: J1.50
- new net BTB42: J1.49
- new net BTB43: J1.48
- new net BTB44: J1.47
- new net BTB45: J1.46
- new net BTB46: J1.45
- new net BTB47: J1.44
- new net BTB48: J1.43
- new net BTB49: J1.42
- new net BTB50: J1.41
- new net BTB51: J1.40
- new net BTB52: J1.39
- new net BTB53: J1.38
- new net BTB54: J1.37
- new net BTB55: J1.36
- new net BTB56: J1.35
- new net BTB57: J1.34
- new net BTB58: J1.33
- new net BTB59: J1.32
- new net BTB60: J1.31
Other:
- moved on the sheet: J3

Commit message: Update
Parts:
- removed C65: 1uF, Capacitor_SMD:C_0805_2012Metric, symbol Device:C
- removed U1, U8: ~, Personal_Project:Button_KMR231GLFS, symbol Personal_Projects:Button_KMR231GLFS
- added U2: ~, Personal_Project:Button_SKSCLCE010, symbol Personal_Projects:BTN_SKSCLCE010
Connections:
- net GND: now also U2.1, U2.3
- net RST_BTN: now also U2.2, U2.4
Other:
- moved on the sheet: C64
