File: Interface_Headers.kicad_sch (KiCad schematic)
At the start: 13 parts, among them J1 BTB_10132798-062100LF, J22 USB_C_Receptacle_USB2.0_16P, J3 SWDB, U7 USBLC6-2SC6

Commit message: Update
Parts:
- removed C64: 1uF, Capacitor_SMD:C_0805_2012Metric, symbol Device:C
- removed U2: ~, Personal_Project:Button_SKSCLCE010, symbol Personal_Projects:BTN_SKSCLCE010
- removed Z3: Diode_BZX84C6V2-7-F, Personal_Project:Diode_BZX84C6V2_SOT96P240X110-3N, symbol Personal_Projects:Diode_BZX84C6V2-7-F
- added C1: 1uF, Capacitor_SMD:C_0805_2012Metric, symbol Device:C
- added R9: 10k, Resistor_SMD:R_0805_2012Metric_1, symbol Device:R
- added U1: ~, Personal_Project:Button_SKSCLCE010, symbol Personal_Projects:BTN_SKSCLCE010
Connections:
- net GND: now also J1.SH1, J1.SH2, J3.1 (Pin_1), C1.1, U1.1, U1.3
- net RST_BTN: now also C1.2, R9.1, U1.2, U1.4
- net USB_VBUS+: no longer J3.1 (Pin_1)
- new net SMPS_OUT2_3V3+: R9.2
Other:
- moved on the sheet: H1, H2, H3, H4, J3
