File: Power_Management.kicad_sch (KiCad schematic)
At the start: 38 parts, among them J2 I2S_OR_LJ_OUT, Q1 MOSFET_SI2333DDS-T1-BE3

Commit message: Update
Parts:
- C1, C10, C11, C13, C21, C23, C24, C25, C39, C4, C42, C43, C44, C45, C47, C51, C53, C54, C62, C63, C66, C67, C68: footprint Capacitor_SMD:C_0805_2012Metric_Pad1.18x1.45mm_HandSolder -> Capacitor_SMD:C_0805_2012Metric
Connections:
- net LDO3IN is gone; now on net PWR_D+: C42.1, LD1.13 (LDO3IN)
- net VREFDDR+ renamed VREFDDR
Other:
- note added: "VREFDDR: VOUT2 / 2 (BUCK2)"
- note removed: "VOUT2 / 2 (BUCK2)"

Commit message: Update
Parts:
- removed C1: 10u, Capacitor_SMD:C_0805_2012Metric, symbol Device:C
- removed C11, C13, C68: 4u7, Capacitor_SMD:C_0805_2012Metric, symbol Device:C
- removed C43: 1u, Capacitor_SMD:C_0805_2012Metric, symbol Device:C
- removed C62: 22u, Capacitor_SMD:C_0805_2012Metric, symbol Device:C
- removed L2: 1u DFE252012P-1R0M=P2, Inductor_SMD:L_1008_2520Metric, symbol Device:L
Connections:
- net LD4+: no longer names the net of LD1.39 (LDO4OUT)
- net LD6+: no longer names the net of LD1.21 (LDO6OUT)
- net VBUSOTG: no longer names the net of LD1.35 (VBUSOTG)
- net VREFDDR: no longer names the net of LD1.16 (VREFDDR)
- no-connect marks 2 -> 8
Other:
- note added: "LD4: 3.3V (fixed), 50mA"
- note added: "LDO6: 0.9 to 3.3V, 150mA"
- note removed: "0.9 to 3.3V, 150mA"
- note removed: "3.3V (fixed), 50mA"

Commit message: Update
Parts:
- removed C63: 4u7, Capacitor_SMD:C_0805_2012Metric, symbol Device:C
Connections:
- no-connect marks 8 -> 9
Changed lines of the file:
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@@
 	)
 	(junction
-		(at 265.43 132.08)
-		(diameter 0)
-		(color 0 0 0 0)
-	)
-	(junction
 		(at 345.44 66.04)
 		(diameter 0)
@@
 	)
 	(no_connect
+		(at 265.43 132.08)
+	)
+	(no_connect
 		(at 226.06 86.36)
 	)
@@
 	(wire
 		(pts
-			(xy 265.43 143.51) (xy 265.43 146.05)
-		)
-		(stroke
-			(width 0)
-			(type default)
-		)
-	)
-	(wire
-		(pts
 			(xy 157.48 95.25) (xy 173.99 95.25)
 		)
@@
 	(wire
 		(pts
-			(xy 265.43 132.08) (xy 276.86 132.08)
-		)
-		(stroke
-			(width 0)
-			(type default)
-		)
-	)
-	(wire
-		(pts
 			(xy 73.66 152.4) (xy 90.17 152.4)
 		)
@@
 	(wire
 		(pts
-			(xy 265.43 132.08) (xy 265.43 135.89)
-		)
-		(stroke
-			(width 0)
-			(type default)
-		)
-	)
-	(wire
-		(pts
 			(xy 214.63 149.86) (xy 214.63 177.8)
 		)
@@
 	(text "1.7 to 3.3V, 350mA"
 		(exclude_from_sim no)
-		(at 273.05 137.16 0)
+		(at 248.92 133.858 0)
 		(effects
 			(font
@@
 	)
 	(symbol
-		(lib_id "power:+3.3V")
-		(at 276.86 132.08 270)
-		(unit 1)
-		(exclude_from_sim no)
-		(in_bom yes)
-		(on_board yes)
-		(dnp no)
-		(property "Reference" "#PWR083"
-			(at 273.05 132.08 0)
-			(effects
-				(font
-					(size 1.27 1.27)
-				)
-				(hide yes)
-			)
-		)
-		(property "Value" "LD1+"
-			(at 281.178 133.858 90)
-			(effects
-				(font
-					(size 1.27 1.27)
-				)
-			)
-		)
-		(property "Footprint" ""
-			(at 276.86 132.08 0)
-			(effects
-				(font
-					(size 1.27 1.27)
-				)
-				(hide yes)
-			)
-		)
-		(property "Datasheet" ""
-			(at 276.86 132.08 0)
-			(effects
-				(font
-					(size 1.27 1.27)
-				)
-				(hide yes)
-			)
-		)
-		(property "Description" "Power symbol creates a global label with name \"+3.3V\""
-			(at 276.86 132.08 0)
-			(effects
-				(font
-					(size 1.27 1.27)
-				)
-				(hide yes)
-			)
-		)
-		(pin "1"
-		)
-		(instances
-			(project "STM32H7_Board"
-				(path "/9b48e30a-b912-4658-a133-1a15707d5b7d/9f177927-57f0-4f81-8b01-253cb2102d0e"
-					(reference "#PWR083")
-					(unit 1)
-				)
-			)
-		)
-	)
-	(symbol
 		(lib_id "power:GND")
 		(at 124.46 262.89 270)
@@
 	)
 	(symbol
-		(lib_id "power:GND")
-		(at 265.43 146.05 0)
-		(unit 1)
-		(exclude_from_sim no)
-		(in_bom yes)
-		(on_board yes)
-		(dnp no)
-		(property "Reference" "#PWR0106"
-			(at 265.43 152.4 0)
-			(effects
-				(font
-					(size 1.27 1.27)
-				)
-				(hide yes)
-			)
-		)
-		(property "Value" "GND"
-			(at 262.89 149.098 90)
-			(effects
-				(font
-					(size 1.27 1.27)
-				)
-				(justify left)
-				(hide yes)
-			)
-		)
-		(property "Footprint" ""
-			(at 265.43 146.05 0)
-			(effects
-				(font
-					(size 1.27 1.27)
-				)
-				(hide yes)
-			)
-		)
-		(property "Datasheet" ""
-			(at 265.43 146.05 0)
-			(effects
-				(font
-					(size 1.27 1.27)
-				)
-				(hide yes)
-			)
-		)
-		(property "Description" "Power symbol creates a global label with name \"GND\" , ground"
-			(at 265.43 146.05 0)
-			(effects
-				(font
-					(size 1.27 1.27)
-				)
-				(hide yes)
-			)
-		)
-		(pin "1"
-		)
-		(instances
-			(project "STM32H7_Board"
-				(path "/9b48e30a-b912-4658-a133-1a15707d5b7d/9f177927-57f0-4f81-8b01-253cb2102d0e"
-					(reference "#PWR0106")
-					(unit 1)
-				)
-			)
-		)
-	)
-	(symbol
 		(lib_id "Device:C")
 		(at 132.08 184.15 0)
@@
 					(unit 1)
 				)
-			)
-		)
-	)
-	(symbol
-		(lib_id "Device:C")
-		(at 265.43 139.7 0)
-		(unit 1)
-		(exclude_from_sim no)
-		(in_bom yes)
-		(on_board yes)
-		(dnp no)
-		(property "Reference" "C63"
-			(at 267.208 137.668 90)
-			(effects
-				(font
-					(size 1.27 1.27)
-				)
-				(justify left)
-			)
-		)
-		(property "Value" "4u7"
-			(at 267.208 145.034 90)
-			(effects
-				(font
-					(size 1.27 1.27)
-				)
-				(justify left)
-			)
-		)
-		(property "Footprint" "Capacitor_SMD:C_0805_2012Metric"
-			(at 266.3952 143.51 0)
-			(effects
-				(font
-					(size 1.27 1.27)
-				)
-				(hide yes)
-			)
-		)
-		(property "Datasheet" "~"
-			(at 265.43 139.7 0)
-			(effects
-				(font
-					(size 1.27 1.27)
-				)
-				(hide yes)
-			)
-		)
-		(property "Description" "Unpolarized capacitor"
-			(at 265.43 139.7 0)
-			(effects
-				(font
-					(size 1.27 1.27)
-				)
-				(hide yes)
-			)
-		)
-		(pin "1"
-		)
-		(pin "2"
-		)
-		(instances
-			(project "STM32H7_Board"
-				(path "/9b48e30a-b912-4658-a133-1a15707d5b7d/9f177927-57f0-4f81-8b01-253cb2102d0e"
-					(reference "C63")
-					(unit 1)
-				)

Commit message: Update
Parts:
- removed C42, C51: 10u, Capacitor_SMD:C_0805_2012Metric, symbol Device:C
- removed C44, C66: 1u, Capacitor_SMD:C_0805_2012Metric, symbol Device:C
- removed C53, C67: 4u7, Capacitor_SMD:C_0805_2012Metric, symbol Device:C
Connections:
- net 3V3_BK4+: now also LD1.42 (VIO), R11.1, R12.1, R6.1
- net PWR_D+: no longer LD1.13 (LDO3IN), LD1.19 (LDO25IN), LD1.22 (LDO16IN)
- net 1V8_LD3+: no longer names the net of LD1.14 (LDO3OUT)
- net 2V8_LD5+: no longer names the net of LD1.20 (LDO5OUT)
- removed net 3V3_BK3+: C47.1, L3.2, LD1.31 (VOUT3), LD1.42 (VIO), R11.1, R12.1, R6.1
- net 3V3_LD2+: no longer names the net of LD1.18 (LDO2OUT)
- net BK1+ renamed 1V2_BK1+
- net LD1+: no longer names the net of LD1.23 (LDO1OUT)
- new net 2V8_BK3+: C47.1, L3.2, LD1.31 (VOUT3)
- no-connect marks 9 -> 15
Other:
- note added: "LDO1: 1.7 to 3.3V, 350mA"
- note added: "LDO2: 1.7 to 3.3V, 350mA"
- note added: "LDO3: 1.7 to 3.3V, 100mA"
- note added: "LDO5: 1.7 to 3.9V, 350mA"
- note removed: "1.7 to 3.3V, 100mA"
- note removed: "1.7 to 3.3V, 350mA"
- note removed: "1.7 to 3.9V, 350mA"

Commit message: Update
Parts:
- added C1: 1uF, Capacitor_SMD:C_0805_2012Metric, symbol Device:C
- added U3: ~, Personal_Project:Button_KMR231GLFS, symbol Personal_Projects:Button_KMR231GLFS
Connections:
- net GND: now also C1.1, U3.3, U3.4, U3.5 (GND)
- net PONKEYN: now also C1.2, U3.1, U3.2

Commit message: Update
Parts:
- added C2: 1u, Capacitor_SMD:C_0805_2012Metric, symbol Device:C
- added C3: 4u7, Capacitor_SMD:C_0805_2012Metric, symbol Device:C
Connections:
- net GND: now also C2.2, C3.2
- net PWR_D+: now also LD1.19 (LDO25IN), C2.1
- net 1V8_LD5+: now reaches LD1.20 (LDO5OUT)
- net 1V8_LD5+: now also C3.1
- no-connect marks 15 -> 13
Other:
- note added: "LDO5: Set to 1V8 with the option of 3V3 Powers the XSPI"
- moved on the sheet: C1, U3

Commit message: Update
Parts:
- removed C1: 1uF, Capacitor_SMD:C_0805_2012Metric, symbol Device:C
- removed C10, C4, C47, C54: 22u, Capacitor_SMD:C_0805_2012Metric, symbol Device:C
- removed C2: 1u, Capacitor_SMD:C_0805_2012Metric, symbol Device:C
- removed C21, C3, C45: 4u7, Capacitor_SMD:C_0805_2012Metric, symbol Device:C
- removed C23, C24, C25, C39: 10u, Capacitor_SMD:C_0805_2012Metric, symbol Device:C
- removed L10, L11, L3, L4: 1u DFE252012P-1R0M=P2, Inductor_SMD:L_1008_2520Metric, symbol Device:L
- removed LD1: LDO_STPMIC1BPQR, Personal_Project:WFQFN-44L_QFN40P500X600X80-45N-D, symbol Personal_Projects:LDO_STPMIC1BPQR
- removed R11, R6: 2k2, Resistor_SMD:R_0805_2012Metric, symbol Device:R
- removed R12: 10k, Resistor_SMD:R_0805_2012Metric, symbol Device:R
- removed U3: ~, Personal_Project:Button_KMR231GLFS, symbol Personal_Projects:Button_KMR231GLFS
- added C26, C7: 22u, Capacitor_SMD:C_1210_3225Metric, symbol Device:C
- added C27: 33p, Capacitor_SMD:C_0805_2012Metric, symbol Device:C
- added C6: 10u, Capacitor_SMD:C_0805_2012Metric, symbol Device:C
- added L1, L5: 2u2 NR4020S2R2MT, Personal_Project:L_NR4020S2R2MT, symbol Device:L
- added R3, R4, R7: 180k, Resistor_SMD:R_0805_2012Metric, symbol Device:R
- added R5: 806k, Resistor_SMD:R_0805_2012Metric, symbol Device:R
- added SMPS1: SMPS_TPS62420DRCTG4, Package_SON:VSON-10-1EP_3x3mm_P0.5mm_EP1.65x2.4mm_ThermalVias, symbol Personal_Projects:SMPS_TPS62420DRCTG4
Connections:
- net GND: now also C26.1, C6.1, C7.1, R4.2, R7.2, SMPS1.11 (PAD), SMPS1.8 (GND)
- net PWR_D+: now also C6.2, SMPS1.2 (MODE_DATA), SMPS1.3 (VIN), SMPS1.7 (EN1), SMPS1.9 (EN2)
- new net ADJ2: C27.1, R5.2, R7.1, SMPS1.1 (ADJ2)
- new net DEF_1: R3.2, R4.1, SMPS1.5 (DEF_1)
- new net SMPS_OUT1_1V2+: C7.2, L1.2, R3.1, SMPS1.4 (FB1)
- new net SMPS_OUT2_3V3+: C26.2, C27.2, L5.2, R5.1
- new net SW1: L1.1, SMPS1.6 (SW1)
- new net SW2: L5.1, SMPS1.10 (SW2)
- no-connect marks 13 -> 0
Other:
- note added: "Power saver mode enabled for both"
- note added: "SMPS OUT1: 600mA"
- note added: "SMPS OUT2: 1000mA"
- note added: "VIN: 2.5V to 6.0V"
- note removed: "(VIN from 2.8V to 5.5V DC)"
- note removed: "0.6 to 3.9V, 2000mA"
- note removed: "0.725 to 1.5V, 1500mA"
- note removed: "1 to 1.5V, 1000mA"
- note removed: "1 to 3.4V, 500mA"
- note removed: "BK1 - STM32H7S3I8T6 VCORE dependding on VOS BK2 - Camera DVDD 1V5 BK3 - STM32H7S3I8T6 I/O VDD 3V3 BK4 - LCD, SDRAM, NAND 3V3, SD Detect Switch pull-up LDO1 LDO2 - SD Card 3V3 (Adjustable to 1V8) LDO3 - VDDXSPI 1V8 Supply on the MCU LDO4 LDO5 - Camera 2V8 LDO6"
- note removed: "LD4: 3.3V (fixed), 50mA"
- note removed: "LDO1: 1.7 to 3.3V, 350mA"
- note removed: "LDO2: 1.7 to 3.3V, 350mA"
- note removed: "LDO3: 1.7 to 3.3V, 100mA"
- note removed: "LDO5: 1.7 to 3.9V, 350mA"
- note removed: "LDO5: Set to 1V8 with the option of 3V3 Powers the XSPI"
- note removed: "LDO6: 0.9 to 3.3V, 150mA"
- note removed: "Power input switch"
- note removed: "Power output switch"
- note removed: "Reserved for MCU Core"
- note removed: "VREFDDR: VOUT2 / 2 (BUCK2)"
- note removed: "Vout_BK3 provides 3V3"

Commit message: Update
Other:
- moved on the sheet: D1, J2, JST1, Q1, R1, Z1
