File: Power_Management.kicad_sch (KiCad schematic)
At the start: 17 parts, among them J2 I2S_OR_LJ_OUT, Q1 MOSFET_SI2333DDS-T1-BE3

Commit message: Update
Other:
- company: (none) -> Peter Hancak
- title: (none) -> STM32H7S3 Board
Changed lines of the file:
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@@
 	(generator_version "8.0")
 	(paper "A3")
+	(title_block
+		(title "STM32H7S3 Board")
+		(date "2026-03-17")
+		(rev "B")
+		(company "Peter Hancak")
+	)
 	(junction
 		(at 142.24 91.44)

Commit message: Update
Parts:
- L5: value 2u2 NR4020S2R2MT -> 3u3 CPN4020H3R3MT
Changed lines of the file:
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@@
 			)
 		)
-		(property "Value" "2u2 NR4020S2R2MT"
+		(property "Value" "3u3 CPN4020H3R3MT"
 			(at 255.778 136.652 90)
 			(effects

Commit message: Update
Parts:
- SMPS1: value SMPS_TPS62420DRCTG4 -> SMPS_TPS62420DRCT
Changed lines of the file:
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@@
 		(dnp no)
 		(property "Reference" "SMPS1"
-			(at 208.28 81.534 0)
+			(at 210.058 81.534 0)
 			(effects
 				(font
@@
 			)
 		)
-		(property "Value" "SMPS_TPS62420DRCTG4"
+		(property "Value" "SMPS_TPS62420DRCT"
 			(at 218.44 84.836 0)
 			(effects
