File: Power_Management.kicad_sch (KiCad schematic)
At the start: 17 parts, among them J2 I2S_OR_LJ_OUT, Q1 MOSFET_SI2333DDS-T1-BE3

Commit message: Update
Parts:
- removed C6: 10u, Capacitor_SMD:C_0805_2012Metric, symbol Device:C
- removed D1: SMAJ6.0A, Personal_Project:DO-214AC-2, symbol Personal_Projects:DIODE_SMAJ6.0A
- removed J2: I2S_OR_LJ_OUT, Connector_PinHeader_2.54mm:PinHeader_1x03_P2.54mm_Vertical, symbol Connector_Generic:Conn_01x03
- removed JST1: JST_S3B-XH-2.54, Personal_Project:JST_S3B-XH-SHDRRA3W64P0X250_1X3_990X1150X610P, symbol Personal_Projects:JST_S3B-XH-A-1_LF_SN
- removed Q1: MOSFET_SI2333DDS-T1-BE3, Personal_Project:MOSFET_ SI2333DDS_SOT_DS-T1-BE3_VIS, symbol Personal_Projects:MOSFET_SI2333DDS-T1-BE3
- removed R1: 100k, Resistor_SMD:R_0805_2012Metric, symbol Device:R
- removed SMPS1: SMPS_TPS62420DRCT, Package_SON:VSON-10-1EP_3x3mm_P0.5mm_EP1.65x2.4mm_ThermalVias, symbol Personal_Projects:SMPS_TPS62420DRCTG4
- removed Z1: Diode_BZX84C6V2-7-F, Personal_Project:Diode_BZX84C6V2_SOT96P240X110-3N, symbol Personal_Projects:Diode_BZX84C6V2-7-F
- added C21, C29: 10u, Capacitor_SMD:C_0603_1608Metric, symbol Device:C
- added C35: 100n, Capacitor_SMD:C_0805_2012Metric, symbol Device:C
- added C67: 3n3, Capacitor_SMD:C_0603_1608Metric, symbol Device:C
- added D2: SMAJ6.0A, Personal_Projects:DO-214AC-2, symbol Personal_Projects:DIODE_SMAJ6.0A
- added D5: SS34-E3/57T, Diode_SMD:D_SMA, symbol Diode:SS34
- added EF1: EFUSE_TPS259531DSGR, Personal_Projects:EF_TPS259531DSGR, symbol Personal_Components:EFUSE_TPS259531DSGR
- added ID2: ID_LM66100DCKR, Personal_Projects:ID_LM66100DCKR, symbol Personal_Components:ID_LM66100DCKR
- added JST2: JST_S3B-XH-2.54, Personal_Projects:JST_S3B-XH-SHDRRA3W64P0X250_1X3_990X1150X610P, symbol Personal_Projects:JST_S3B-XH-A-1_LF_SN
- added R38, R52: 1M, Resistor_SMD:R_0603_1608Metric, symbol Device:R
- added R43: 383k, Resistor_SMD:R_0603_1608Metric, symbol Device:R
- added R51: 487R, Resistor_SMD:R_0603_1608Metric, symbol Device:R
- added SMPS1: SMPS_TPS62420DRCTG4, Package_SON:VSON-10-1EP_3x3mm_P0.5mm_EP1.65x2.4mm, symbol Personal_Components:SMPS_TPS62420DRCTG4
- added TP13, TP14, TP15, TP17: TestPoint, TestPoint:TestPoint_Pad_1.5x1.5mm, symbol Connector:TestPoint
- added U4: SN74LVC1G07DBVR, Package_TO_SOT_SMD:SOT-23-5, symbol 74xGxx:74LVC1G07
Connections:
- net ADJ2: now also SMPS1.1 (ADJ2)
- net DEF_1: now also SMPS1.5 (DEF_1)
- net GND: now also C21.2, C29.2, C35.2, C67.1, D2.2 (A), EF1.8 (GND), EF1.9 (GND__1), ID2.2 (GND), ID2.3 (*CE), ID2.5 (ST), JST2.2 (PWR-), R43.2, R51.2, SMPS1.11 (PAD), SMPS1.8 (GND), U4.3 (GND)
- net PWR+: now also D2.1 (K), ID2.1 (VIN), JST2.1 (PWR+), TP14.1
- net PWR+_PP: now also D5.1 (K), EF1.3 (IN), EF1.4 (IN__1), ID2.6 (VOUT), R38.1, TP13.1
- net RST_PWR: now also C35.1, JST2.3 (RST), U4.2
- net SMPS_OUT1_1V2+: now also SMPS1.4 (FB1), TP17.1
- net SMPS_OUT2_3V3+: now also TP15.1, U4.5 (VCC)
- net SW1: now also SMPS1.6 (SW1)
- net SW2: now also SMPS1.10 (SW2)
- net USB_VBUS+: now also D5.2 (A)
- new net: EF1.7 (ILM), R51.1
- new net DVDT_1: C67.2, EF1.1 (DVDT)
- new net EN/UVLO_1: EF1.2 (EN/UVLO), R38.2, R43.1
- new net PWR+_EF: C21.1, C29.1, EF1.5 (OUT), R52.1, SMPS1.2 (MODE_DATA), SMPS1.3 (VIN)
- new net RST_LOCAL: U4.4
- new net ~{FLT}: EF1.6 (~{FLT}), R52.2, SMPS1.7 (EN1), SMPS1.9 (EN2)
- no-connect marks 0 -> 1
Other:
- note added: "FLT 6V MAX"
- note added: "IN 1.5A MAX"
- note added: "IN 5A MAX"
- note added: "Power can be sourced from USB or Power connector"
- note added: "TPS259531DSGR OUTPUT VOLTAGE CLAMP: 5.7 V (typ) UNDERVOLTAGE LOCKOUT: Vsupply = VUVLO * (R1 + R2) / R2 ACTIVE CURRENT LIMITING: RILM = 2000/(ILIMIT - 0.04), for 4A RILM = 495Ohms"
- note removed: "Overvoltage protection for the PMOSFET VGS (VGS max is 8V)"
- note removed: "Polarity Protection"
- moved on the sheet: C26, C27, C7, L1, L5, R3, R4, R5, R7
